Commit message: wrong masses in urdf models fixed

File: shadow_robot/sr_hand/model/shadowhand_motor.urdf (robot description, URDF)
Before this commit: robot shadowhand, 25 links, 24 joints
Links:
- link ffdistal: mass 0.008 -> 0.010
- link ffmiddle: mass 0.008 -> 0.012
- link ffproximal: mass 0.008 -> 0.014
- link lfdistal: mass 0.008 -> 0.010
- link lfmetacarpal: mass 0.008 -> 0.075
- link lfmiddle: mass 0.008 -> 0.012
- link lfproximal: mass 0.008 -> 0.014
- link mfdistal: mass 0.008 -> 0.010
- link mfmiddle: mass 0.008 -> 0.012
- link mfproximal: mass 0.008 -> 0.014
- link palm: mass 0.08 -> 0.3
- link rfdistal: mass 0.008 -> 0.010
- link rfmiddle: mass 0.008 -> 0.012
- link rfproximal: mass 0.008 -> 0.014
- link shadow_forearm: geometry collision cylinder length=0.180 radius=0.06; visual mesh filename=package://sr_hand/model/meshes/forearm.mesh
- link thbase: mass 0.008 -> 0.010
- link thdistal: mass 0.008 -> 0.016
- link thhub: mass 0.008 -> 0.002
- link thmiddle: mass 0.008 -> 0.016
- link thproximal: mass 0.008 -> 0.016
- link wrist: mass 0.08 -> 0.3

File: shadow_robot/sr_hand/model/shadowhand_muscle.urdf (robot description, URDF)
Before this commit: robot shadowhand, 25 links, 24 joints
Links:
- link ffdistal: mass 0.008 -> 0.010
- link ffmiddle: mass 0.008 -> 0.012
- link ffproximal: mass 0.008 -> 0.014
- link lfdistal: mass 0.008 -> 0.010
- link lfmetacarpal: mass 0.008 -> 0.075
- link lfmiddle: mass 0.008 -> 0.012
- link lfproximal: mass 0.008 -> 0.014
- link mfdistal: mass 0.008 -> 0.010
- link mfmiddle: mass 0.008 -> 0.012
- link mfproximal: mass 0.008 -> 0.014
- link palm: mass 0.08 -> 0.3
- link rfdistal: mass 0.008 -> 0.010
- link rfmiddle: mass 0.008 -> 0.012
- link rfproximal: mass 0.008 -> 0.014
- link thbase: mass 0.008 -> 0.010
- link thdistal: mass 0.008 -> 0.016
- link thhub: mass 0.008 -> 0.002
- link thmiddle: mass 0.008 -> 0.016
- link thproximal: mass 0.008 -> 0.016
- link wrist: mass 0.08 -> 0.3

Commit message: Added packages for the video1394 acquisition, corrected few things on control_gui and hacked the cyberglove remapper to prevent the thumb problems (shut down THJ4 and THJ5)

File: shadow_robot/sr_hand/model/shadowhand_motor.urdf (robot description, URDF)
Before this commit: robot shadowhand, 25 links, 24 joints
Links:
- link shadow_forearm: geometry collision cylinder length=0.180 radius=0.06; visual mesh filename=package://sr_hand/model/meshes/forearm.mesh
