Commit message: the hand and the arm are viewable in gazebo. An empty_world.launch is in the gazebo folder to launch gazebo with the good param. For the arm urdf model, the base weight is set to 1000kg, not to fall when it spawns

File: shadow_robot/sr_hand/model/sr_arm_motor.urdf (robot description, URDF)
Before this commit: robot shadow_arm, 5 links, 4 joints
Links:
- link shadowarm_base: mass 0.5 -> 1000

File: shadow_robot/sr_hand/model/sr_arm_muscle.urdf (robot description, URDF)
Before this commit: robot shadow_arm, 5 links, 4 joints
Links:
- link shadowarm_base: mass 0.5 -> 1000

Commit message: Gazebo: starting the simulation paused, then bending the Elbow, so as not to start in the floor, then starting the physics (as suggested here http://answers.ros.org/question/857/set-revolute-joint-start-angle)
Still need to see if it's possible not to include gazebo as a dependency.

File: shadow_robot/sr_hand/model/sr_arm_motor.urdf (robot description, URDF)
Before this commit: robot sr_arm_motor, 6 links, 5 joints
Links:
- removed link world
Joints:
- removed joint base_fix
