Commit message: hand controller tuned (a bit) and small model bugs fixed. the joints are still not stiff at all...

File: shadow_robot/sr_hand/model/hand_urdf/finger/distal/distal.transmission.xacro (robot description, xacro)
@@ -5,5 +5,5 @@
        xmlns:xacro="http://ros.org/wiki/xacro">
   <xacro:macro name="distal_transmission">
-    <transmission type="SimpleTransmission" name="${link_prefix}distal_transmission">
+    <transmission type="pr2_mechanism_model/SimpleTransmission" name="${link_prefix}distal_transmission">
       <actuator name="${joint_prefix}J1" />
       <joint name="${joint_prefix}J1" />

File: shadow_robot/sr_hand/model/hand_urdf/finger/distal/distal.urdf.xacro (robot description, xacro)
@@ -33,4 +33,5 @@
       <limit lower="0" upper="${M_PI/2}" effort="10"
       velocity="1.0" />
+      <dynamics damping="3.5"/>
     </joint>
     <xacro:distal_transmission />

File: shadow_robot/sr_hand/model/hand_urdf/finger/knuckle/knuckle.transmission.xacro (robot description, xacro)
@@ -5,5 +5,5 @@
        xmlns:xacro="http://ros.org/wiki/xacro">
   <xacro:macro name="knuckle_transmission">
-    <transmission type="SimpleTransmission" name="${link_prefix}knuckle_transmission">
+    <transmission type="pr2_mechanism_model/SimpleTransmission" name="${link_prefix}knuckle_transmission">
       <actuator name="${joint_prefix}J4" />
       <joint name="${joint_prefix}J4" />

File: shadow_robot/sr_hand/model/hand_urdf/finger/knuckle/knuckle.urdf.xacro (robot description, xacro)
@@ -35,4 +35,5 @@
       <limit lower="-0.43633231299858238" upper="0.43633231299858238"
       effort="10" velocity="1.0"/>
+      <dynamics damping="3.5"/>
     </joint>
     <xacro:knuckle_transmission />

File: shadow_robot/sr_hand/model/hand_urdf/finger/lfmetacarpal/lfmetacarpal.transmission.xacro (robot description, xacro)
@@ -5,5 +5,5 @@
        xmlns:xacro="http://ros.org/wiki/xacro">
   <xacro:macro name="lfmetacarpal_transmission">
-    <transmission type="SimpleTransmission" name="lfmetacarpal_transmission">
+    <transmission type="pr2_mechanism_model/SimpleTransmission" name="lfmetacarpal_transmission">
       <actuator name="LFJ5" />
       <joint name="LFJ5" />

File: shadow_robot/sr_hand/model/hand_urdf/finger/lfmetacarpal/lfmetacarpal.urdf.xacro (robot description, xacro)
@@ -33,4 +33,5 @@
       <limit lower="0" upper="0.69813170079773179" effort="10"
       velocity="1.0" />
+      <dynamics damping="3.5"/>
     </joint>
     <xacro:lfmetacarpal_transmission />

File: shadow_robot/sr_hand/model/hand_urdf/finger/little_finger.urdf.xacro (robot description, xacro)
@@ -39,6 +39,7 @@
       <limit lower="-0.43633231299858238" upper="0.43633231299858238"
       effort="10" velocity="1.0"/>
+      <dynamics damping="3.5"/>
     </joint>
-    <transmission type="SimpleTransmission" name="lfknuckle_transmission">
+    <transmission type="pr2_mechanism_model/SimpleTransmission" name="lfknuckle_transmission">
       <actuator name="LFJ4" />
       <joint name="LFJ4" />

File: shadow_robot/sr_hand/model/hand_urdf/finger/middle/middle.transmission.xacro (robot description, xacro)
@@ -5,5 +5,5 @@
        xmlns:xacro="http://ros.org/wiki/xacro">
   <xacro:macro name="middle_transmission">
-    <transmission type="SimpleTransmission" name="${link_prefix}middle_transmission">
+    <transmission type="pr2_mechanism_model/SimpleTransmission" name="${link_prefix}middle_transmission">
       <actuator name="${joint_prefix}J2" />
       <joint name="${joint_prefix}J2" />

File: shadow_robot/sr_hand/model/hand_urdf/finger/middle/middle.urdf.xacro (robot description, xacro)
@@ -33,4 +33,5 @@
       <limit lower="0" upper="${M_PI/2}" effort="10"
       velocity="1.0" />
+      <dynamics damping="3.5"/>
     </joint>
     <xacro:middle_transmission />

File: shadow_robot/sr_hand/model/hand_urdf/finger/proximal/proximal.transmission.xacro (robot description, xacro)
@@ -5,5 +5,5 @@
        xmlns:xacro="http://ros.org/wiki/xacro">
   <xacro:macro name="proximal_transmission">
-    <transmission type="SimpleTransmission" name="${link_prefix}proximal_transmission">
+    <transmission type="pr2_mechanism_model/SimpleTransmission" name="${link_prefix}proximal_transmission">
       <actuator name="${joint_prefix}J3" />
       <joint name="${joint_prefix}J3" />

File: shadow_robot/sr_hand/model/hand_urdf/finger/proximal/proximal.urdf.xacro (robot description, xacro)
@@ -33,4 +33,5 @@
       <limit lower="0" upper="${M_PI/2}" effort="10"
       velocity="1.0"/>
+      <dynamics damping="3.5"/>
     </joint>
     <xacro:proximal_transmission />

File: shadow_robot/sr_hand/model/hand_urdf/palm/palm.transmission.xacro (robot description, xacro)
@@ -5,5 +5,5 @@
        xmlns:xacro="http://ros.org/wiki/xacro">
   <xacro:macro name="shadowhand_palm_transmission">
-    <transmission type="SimpleTransmission" name="palm_transmission">
+    <transmission type="pr2_mechanism_model/SimpleTransmission" name="palm_transmission">
       <actuator name="WRJ1" />
       <joint name="WRJ1" />

File: shadow_robot/sr_hand/model/hand_urdf/palm/palm.urdf.xacro (robot description, xacro)
@@ -33,4 +33,5 @@
       <limit lower="-0.78539816339744828" upper="0.6108652381980153"
       effort="10" velocity="1.0"/>
+      <dynamics damping="3.5"/>
     </joint>
     <xacro:shadowhand_palm_transmission />

File: shadow_robot/sr_hand/model/hand_urdf/thumb/thbase.transmission.xacro (robot description, xacro)
@@ -5,5 +5,5 @@
        xmlns:xacro="http://ros.org/wiki/xacro">
   <xacro:macro name="thbase_transmission">
-    <transmission type="SimpleTransmission" name="thbase_transmission">
+    <transmission type="pr2_mechanism_model/SimpleTransmission" name="thbase_transmission">
       <actuator name="THJ5" />
       <joint name="THJ5" />

File: shadow_robot/sr_hand/model/hand_urdf/thumb/thbase.urdf.xacro (robot description, xacro)
@@ -35,4 +35,5 @@
       <limit lower="-1.047" upper="1.047" effort="10"
       velocity="1.0" />
+      <dynamics damping="3.5"/>
     </joint>
     <xacro:thbase_transmission />

File: shadow_robot/sr_hand/model/hand_urdf/thumb/thdistal.transmission.xacro (robot description, xacro)
@@ -5,5 +5,5 @@
        xmlns:xacro="http://ros.org/wiki/xacro">
   <xacro:macro name="thdistal_transmission">
-    <transmission type="SimpleTransmission" name="thdistal_transmission">
+    <transmission type="pr2_mechanism_model/SimpleTransmission" name="thdistal_transmission">
       <actuator name="THJ1" />
       <joint name="THJ1" />

File: shadow_robot/sr_hand/model/hand_urdf/thumb/thdistal.urdf.xacro (robot description, xacro)
@@ -35,4 +35,5 @@
       <limit lower="0" upper="1.571" effort="10"
       velocity="1.0" />
+      <dynamics damping="3.5"/>
     </joint>
     <xacro:thdistal_transmission />

File: shadow_robot/sr_hand/model/hand_urdf/thumb/thhub.transmission.xacro (robot description, xacro)
@@ -5,5 +5,5 @@
        xmlns:xacro="http://ros.org/wiki/xacro">
   <xacro:macro name="thhub_transmission">
-    <transmission type="SimpleTransmission" name="thhub_transmission">
+    <transmission type="pr2_mechanism_model/SimpleTransmission" name="thhub_transmission">
       <actuator name="THJ3" />
       <joint name="THJ3" />

File: shadow_robot/sr_hand/model/hand_urdf/thumb/thhub.urdf.xacro (robot description, xacro)
@@ -35,4 +35,5 @@
       <limit lower="-0.2618" upper="0.2618" effort="10"
       velocity="1.0" />
+      <dynamics damping="3.5"/>
     </joint>
     <xacro:thhub_transmission />

File: shadow_robot/sr_hand/model/hand_urdf/thumb/thmiddle.transmission.xacro (robot description, xacro)
@@ -5,5 +5,5 @@
        xmlns:xacro="http://ros.org/wiki/xacro">
   <xacro:macro name="thmiddle_transmission">
-    <transmission type="SimpleTransmission" name="thmiddle_transmission">
+    <transmission type="pr2_mechanism_model/SimpleTransmission" name="thmiddle_transmission">
       <actuator name="THJ2" />
       <joint name="THJ2" />
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