Commit message: Proposed new hand meshes in two modes original one are saved full is the optimized version of the meshes envelop is the light version of the meshes without internal details
saved hand_urdf to original
proposed new hand_urdf adapted to new meshes and more cleaner (without many orientation change)

File: shadow_robot/sr_hand/model/hand_urdf/finger/distal/distal.urdf.xacro (robot description, xacro)
@@ -1,9 +1,3 @@
-<robot xmlns:xacro="http://ros.org/wiki/xacro"
-	xmlns:sensor="http://playerstage.sourceforge.net/gazebo/xmlschema/#sensor"
-	xmlns:controller="http://playerstage.sourceforge.net/gazebo/xmlschema/#controller"
-       xmlns:joint="http://playerstage.sourceforge.net/gazebo/xmlschema/#slider"
-       xmlns:interface="http://playerstage.sourceforge.net/gazebo/xmlschema/#interface"
-       xmlns:body="http://playerstage.sourceforge.net/gazebo/xmlschema/#body"
-       xmlns:geom="http://playerstage.sourceforge.net/gazebo/xmlschema/#geom">
+<robot xmlns:xacro="http://ros.org/wiki/xacro">
   <include filename="$(find sr_hand)/model/hand_urdf/finger/distal/distal.transmission.xacro" />
   <xacro:macro name="distal" params="link_prefix joint_prefix parent">
@@ -16,5 +10,5 @@
       </inertial>
       <visual>
-	<origin xyz="0 0 0" rpy="0 -${M_PI/2} 0" />
+	<origin xyz="0 0 0" rpy="0 0 0" />
 	<geometry name="distal_visual">
       <mesh filename="package://sr_hand/model/meshes/F1.mesh" scale="0.001 0.001 0.001" />
@@ -30,15 +24,4 @@
     </link>
     <gazebo reference="${link_prefix}distal">
-      <sensor:contact name="${link_prefix}distal_contact_sensor">
-        <geom>${link_prefix}distal_geom</geom>
-        <updateRate>100.0</updateRate>
-        <controller:gazebo_ros_bumper name="${link_prefix}distal_gazebo_ros_bumper_controller" plugin="libgazebo_ros_bumper.so">
-          <alwaysOn>true</alwaysOn>
-          <updateRate>100.0</updateRate>
-          <frameName>${link_prefix}distal</frameName>
-          <bumperTopicName>${link_prefix}distal_bumper</bumperTopicName>
-          <interface:bumper name="${link_prefix}distal_gazebo_ros_bumper_iface" />
-        </controller:gazebo_ros_bumper>
-      </sensor:contact>
       <material>Gazebo/Grey</material>
     </gazebo>

File: shadow_robot/sr_hand/model/hand_urdf/finger/knuckle/knuckle.urdf.xacro (robot description, xacro)
@@ -1,9 +1,3 @@
-<robot xmlns:xacro="http://ros.org/wiki/xacro"
-        xmlns:sensor="http://playerstage.sourceforge.net/gazebo/xmlschema/#sensor"
-       xmlns:controller="http://playerstage.sourceforge.net/gazebo/xmlschema/#controller"
-       xmlns:joint="http://playerstage.sourceforge.net/gazebo/xmlschema/#slider"
-       xmlns:interface="http://playerstage.sourceforge.net/gazebo/xmlschema/#interface"
-       xmlns:body="http://playerstage.sourceforge.net/gazebo/xmlschema/#body"
-       xmlns:geom="http://playerstage.sourceforge.net/gazebo/xmlschema/#geom">
+<robot xmlns:xacro="http://ros.org/wiki/xacro">
   <include filename="$(find sr_hand)/model/hand_urdf/finger/knuckle/knuckle.transmission.xacro" />
   <xacro:macro name="knuckle" params="link_prefix joint_prefix parent *origin">
@@ -17,5 +11,5 @@
       </inertial>
       <visual>
-	<origin xyz="0 0 0.0005" rpy="${M_PI} -${M_PI/2} -${M_PI/2}" />
+	<origin xyz="0 0 0.0005" rpy="0 0 0" />
 	<geometry name="knuckle_visual">
       <mesh filename="package://sr_hand/model/meshes/knuckle.mesh" scale="0.001 0.001 0.001" />
@@ -31,15 +25,4 @@
     </link>
     <gazebo reference="${link_prefix}knuckle">
-      <sensor:contact name="${link_prefix}knuckle_contact_sensor">
-        <geom>${link_prefix}knuckle_geom</geom>
-       <updateRate>100.0</updateRate>
-        <controller:gazebo_ros_bumper name="${link_prefix}knuckle_gazebo_ros_bumper_controller" plugin="libgazebo_ros_bumper.so">
-          <alwaysOn>true</alwaysOn>
-          <updateRate>100.0</updateRate>
-          <frameName>${link_prefix}knuckle</frameName>
-          <bumperTopicName>${link_prefix}knuckle_bumper</bumperTopicName>
-          <interface:bumper name="${link_prefix}knuckle_gazebo_ros_bumper_iface" />
-        </controller:gazebo_ros_bumper>
-      </sensor:contact>
       <material>PR2/Grey2</material>
     </gazebo>

File: shadow_robot/sr_hand/model/hand_urdf/finger/lfmetacarpal/lfmetacarpal.urdf.xacro (robot description, xacro)
@@ -1,14 +1,8 @@
-<robot xmlns:xacro="http://ros.org/wiki/xacro"
-        xmlns:sensor="http://playerstage.sourceforge.net/gazebo/xmlschema/#sensor"
-       xmlns:controller="http://playerstage.sourceforge.net/gazebo/xmlschema/#controller"
-       xmlns:joint="http://playerstage.sourceforge.net/gazebo/xmlschema/#slider"
-       xmlns:interface="http://playerstage.sourceforge.net/gazebo/xmlschema/#interface"
-       xmlns:body="http://playerstage.sourceforge.net/gazebo/xmlschema/#body"
-       xmlns:geom="http://playerstage.sourceforge.net/gazebo/xmlschema/#geom">
+<robot xmlns:xacro="http://ros.org/wiki/xacro">
   <include filename="$(find sr_hand)/model/hand_urdf/finger/lfmetacarpal/lfmetacarpal.transmission.xacro" />
   <xacro:macro name="lfmetacarpal" params="parent">
     <link name="lfmetacarpal">
       <inertial>
-	<origin xyz="0.00568 0 -0.12061" rpy="0 0 0" />
+	<origin xyz="-0.033 0 0.02071" rpy="0 0 0" />
 	<mass value="0.075" />
 	<inertia  ixx="1.0" ixy="0.0"  ixz="0.0"  iyy="0.0"  iyz="0.0"
@@ -16,5 +10,5 @@
       </inertial>
       <visual>
-	<origin xyz="0 0 0" rpy="0 -${M_PI/2} 0" />
+	<origin xyz="0 0 0" rpy="0 0 0" />
 	<geometry name="lfmetacarpal_visual">
 	  <mesh filename="package://sr_hand/model/meshes/lfmetacarpal.mesh" scale="0.001 0.001 0.001" />
@@ -30,15 +24,4 @@
     </link>
     <gazebo reference="lfmetacarpal">
-      <sensor:contact name="lfmetacarpal_contact_sensor">
-        <geom>lfmetacarpal_geom</geom>
-       <updateRate>100.0</updateRate>
-        <controller:gazebo_ros_bumper name="lfmetacarpal_gazebo_ros_bumper_controller" plugin="libgazebo_ros_bumper.so">
-          <alwaysOn>true</alwaysOn>
-          <updateRate>100.0</updateRate>
-          <frameName>lfmetacarpal</frameName>
-          <bumperTopicName>lfmetacarpal_bumper</bumperTopicName>
-          <interface:bumper name="lfmetacarpal_gazebo_ros_bumper_iface" />
-        </controller:gazebo_ros_bumper>
-      </sensor:contact>
       <material>Gazebo/Grey</material>
     </gazebo>
@@ -46,5 +29,5 @@
       <parent link="${parent}"/>
       <child link="lfmetacarpal"/>
-      <origin xyz="-0.01671 0 0.044" rpy="0 0 0" />
+      <origin xyz="-0.033 0 0.02071" rpy="0 0 0" />
       <axis xyz="0.57 0 0.82" />
       <limit lower="0" upper="0.69813170079773179" effort="10"

File: shadow_robot/sr_hand/model/hand_urdf/finger/little_finger.urdf.xacro (robot description, xacro)
@@ -1,9 +1,3 @@
-<robot xmlns:xacro="http://www.ros.org/wiki/xacro"
-        xmlns:sensor="http://playerstage.sourceforge.net/gazebo/xmlschema/#sensor"
-       xmlns:controller="http://playerstage.sourceforge.net/gazebo/xmlschema/#controller"
-       xmlns:joint="http://playerstage.sourceforge.net/gazebo/xmlschema/#slider"
-       xmlns:interface="http://playerstage.sourceforge.net/gazebo/xmlschema/#interface"
-       xmlns:body="http://playerstage.sourceforge.net/gazebo/xmlschema/#body"
-       xmlns:geom="http://playerstage.sourceforge.net/gazebo/xmlschema/#geom">
+<robot xmlns:xacro="http://www.ros.org/wiki/xacro">
   <include filename="$(find sr_hand)/model/hand_urdf/finger/knuckle/knuckle.urdf.xacro" />
   <include filename="$(find sr_hand)/model/hand_urdf/finger/proximal/proximal.urdf.xacro" />
@@ -16,5 +10,5 @@
     <link name="lfknuckle">
       <inertial>
-	<origin xyz="0 0 0.0425" rpy="0 0 0" />
+	<origin xyz="0 0 0.06579" rpy="0 0 0" />
 	<mass value="0.008" />
 	<inertia  ixx="1.0" ixy="0.0"  ixz="0.0"  iyy="0.0"  iyz="0.0"
@@ -22,5 +16,5 @@
       </inertial>
       <visual>
-	<origin xyz="0 0 0.0005" rpy="${M_PI} -${M_PI/2} -${M_PI/2}" />
+	<origin xyz="0 0 0" rpy="0 0 0" />
 	<geometry name="knuckle_visual">
       <mesh filename="package://sr_hand/model/meshes/knuckle.mesh" scale="0.001 0.001 0.001" />
@@ -36,15 +30,4 @@
     </link>
     <gazebo reference="lfknuckle">
-      <sensor:contact name="lfknuckle_contact_sensor">
-        <geom>lfknuckle_geom</geom>
-       <updateRate>100.0</updateRate>
-        <controller:gazebo_ros_bumper name="lfknuckle_gazebo_ros_bumper_controller" plugin="libgazebo_ros_bumper.so">
-          <alwaysOn>true</alwaysOn>
-          <updateRate>100.0</updateRate>
-          <frameName>lfknuckle</frameName>
-          <bumperTopicName>lfknuckle_bumper</bumperTopicName>
-          <interface:bumper name="lfknuckle_gazebo_ros_bumper_iface" />
-        </controller:gazebo_ros_bumper>
-      </sensor:contact>
       <material>PR2/Grey2</material>
     </gazebo>
@@ -52,5 +35,5 @@
       <parent link="lfmetacarpal"/>
       <child link="lfknuckle"/>
-      <origin xyz="-0.01671 0 0.044" rpy="0 0 0" />
+      <origin xyz="0 0 0.06579" rpy="0 0 0" />
       <axis xyz="0 1 0" />
       <limit lower="-0.43633231299858238" upper="0.43633231299858238"

File: shadow_robot/sr_hand/model/hand_urdf/finger/middle/middle.urdf.xacro (robot description, xacro)
@@ -1,9 +1,3 @@
-<robot xmlns:xacro="http://ros.org/wiki/xacro"
-        xmlns:sensor="http://playerstage.sourceforge.net/gazebo/xmlschema/#sensor"
-       xmlns:controller="http://playerstage.sourceforge.net/gazebo/xmlschema/#controller"
-       xmlns:joint="http://playerstage.sourceforge.net/gazebo/xmlschema/#slider"
-       xmlns:interface="http://playerstage.sourceforge.net/gazebo/xmlschema/#interface"
-       xmlns:body="http://playerstage.sourceforge.net/gazebo/xmlschema/#body"
-       xmlns:geom="http://playerstage.sourceforge.net/gazebo/xmlschema/#geom">
+<robot xmlns:xacro="http://ros.org/wiki/xacro">
   <include filename="$(find sr_hand)/model/hand_urdf/finger/middle/middle.transmission.xacro" />
   <xacro:macro name="middle" params="link_prefix joint_prefix parent">
@@ -16,5 +10,5 @@
       </inertial>
       <visual>
-	<origin xyz="0 0 0" rpy="0 -${M_PI/2} 0" />
+	<origin xyz="0 0 0" rpy="0 0 0" />
 	<geometry name="middle_visual">
       <mesh filename="package://sr_hand/model/meshes/F2.mesh" scale="0.001 0.001 0.001" />
@@ -30,15 +24,4 @@
     </link>
     <gazebo reference="${link_prefix}middle">
-      <sensor:contact name="${link_prefix}middle_contact_sensor">
-        <geom>${link_prefix}middle_geom</geom>
-       <updateRate>100.0</updateRate>
-        <controller:gazebo_ros_bumper name="${link_prefix}middle_gazebo_ros_bumper_controller" plugin="libgazebo_ros_bumper.so">
-          <alwaysOn>true</alwaysOn>
-          <updateRate>100.0</updateRate>
-          <frameName>${link_prefix}middle</frameName>
-          <bumperTopicName>${link_prefix}middle_bumper</bumperTopicName>
-          <interface:bumper name="${link_prefix}middle_gazebo_ros_bumper_iface" />
-        </controller:gazebo_ros_bumper>
-      </sensor:contact>
       <material>Gazebo/Grey</material>
     </gazebo>

File: shadow_robot/sr_hand/model/hand_urdf/finger/proximal/proximal.urdf.xacro (robot description, xacro)
@@ -1,9 +1,3 @@
-<robot xmlns:xacro="http://ros.org/wiki/xacro"
-        xmlns:sensor="http://playerstage.sourceforge.net/gazebo/xmlschema/#sensor"
-       xmlns:controller="http://playerstage.sourceforge.net/gazebo/xmlschema/#controller"
-       xmlns:joint="http://playerstage.sourceforge.net/gazebo/xmlschema/#slider"
-       xmlns:interface="http://playerstage.sourceforge.net/gazebo/xmlschema/#interface"
-       xmlns:body="http://playerstage.sourceforge.net/gazebo/xmlschema/#body"
-       xmlns:geom="http://playerstage.sourceforge.net/gazebo/xmlschema/#geom">
+<robot xmlns:xacro="http://ros.org/wiki/xacro">
   <include filename="$(find sr_hand)/model/hand_urdf/finger/proximal/proximal.transmission.xacro" />
   <xacro:macro name="proximal" params="link_prefix joint_prefix parent">
@@ -16,5 +10,5 @@
       </inertial>
       <visual>
-	<origin xyz="0 0 0" rpy="0 -${M_PI/2} ${M_PI/2}" />
+	<origin xyz="0 0 0" rpy="0 0 0" />
 	<geometry name="proximal_visual">
       <mesh filename="package://sr_hand/model/meshes/F3.mesh" scale="0.001 0.001 0.001" />
@@ -30,15 +24,4 @@
     </link>
     <gazebo reference="${link_prefix}proximal">
-      <sensor:contact name="${link_prefix}proximal_contact_sensor">
-        <geom>${link_prefix}proximal_geom</geom>
-       <updateRate>100.0</updateRate>
-        <controller:gazebo_ros_bumper name="${link_prefix}proximal_gazebo_ros_bumper_controller" plugin="libgazebo_ros_bumper.so">
-          <alwaysOn>true</alwaysOn>
-          <updateRate>100.0</updateRate>
-          <frameName>${link_prefix}proximal</frameName>
-          <bumperTopicName>${link_prefix}proximal_bumper</bumperTopicName>
-          <interface:bumper name="${link_prefix}proximal_gazebo_ros_bumper_iface" />
-        </controller:gazebo_ros_bumper>
-      </sensor:contact>
       <material>Gazebo/Grey</material>
     </gazebo>

File: shadow_robot/sr_hand/model/hand_urdf/forearm/forearm_motor.urdf.xacro (robot description, xacro)
@@ -9,7 +9,7 @@
       </inertial>
       <visual>
-	<origin xyz="0 0 0" rpy="0 0 -${M_PI/2}" />
+	<origin xyz="0 0 0" rpy="0 0 0" />
 	<geometry name="shadow_forearm_geom">
-	  <mesh filename="package://sr_hand/model/meshes/forearm.mesh" />
+	  <mesh filename="package://sr_hand/model/meshes/forearm.mesh" scale="0.001 0.001 0.001"/>
 	</geometry>
 	<material name="Grey" />

File: shadow_robot/sr_hand/model/hand_urdf/palm/palm.urdf.xacro (robot description, xacro)
@@ -1,9 +1,3 @@
-<robot xmlns:xacro="http://ros.org/wiki/xacro"
-        xmlns:sensor="http://playerstage.sourceforge.net/gazebo/xmlschema/#sensor"
-       xmlns:controller="http://playerstage.sourceforge.net/gazebo/xmlschema/#controller"
-       xmlns:joint="http://playerstage.sourceforge.net/gazebo/xmlschema/#slider"
-       xmlns:interface="http://playerstage.sourceforge.net/gazebo/xmlschema/#interface"
-       xmlns:body="http://playerstage.sourceforge.net/gazebo/xmlschema/#body"
-       xmlns:geom="http://playerstage.sourceforge.net/gazebo/xmlschema/#geom">
+<robot xmlns:xacro="http://ros.org/wiki/xacro">
   <include filename="$(find sr_hand)/model/hand_urdf/palm/palm.transmission.xacro" />
   <xacro:macro name="palm" params="parent">
@@ -16,5 +10,5 @@
       </inertial>
       <visual>
-	<origin xyz="0 0 0" rpy="0 -${M_PI/2} 0" />
+	<origin xyz="0 0 0" rpy="0 0 0" />
 	<geometry name="palm_visual">
 	  <mesh filename="package://sr_hand/model/meshes/palm.mesh" scale="0.001 0.001 0.001" />
@@ -30,15 +24,4 @@
     </link>
     <gazebo reference="palm">
-      <sensor:contact name="palm_contact_sensor">
-       <geom>palm_geom</geom>
-       <updateRate>100.0</updateRate>
-       <controller:gazebo_ros_bumper name="palm_gazebo_ros_bumper_controller" plugin="libgazebo_ros_bumper.so">
-          <alwaysOn>true</alwaysOn>
-          <updateRate>100.0</updateRate>
-          <frameName>palm</frameName>
-          <bumperTopicName>palm_bumper</bumperTopicName>
-          <interface:bumper name="palm_gazebo_ros_bumper_iface" />
-       </controller:gazebo_ros_bumper>
-      </sensor:contact>
       <material>Gazebo/Grey</material>
     </gazebo>

File: shadow_robot/sr_hand/model/hand_urdf/thumb/thbase.urdf.xacro (robot description, xacro)
@@ -1,9 +1,3 @@
-<robot xmlns:xacro="http://ros.org/wiki/xacro"
-        xmlns:sensor="http://playerstage.sourceforge.net/gazebo/xmlschema/#sensor"
-       xmlns:controller="http://playerstage.sourceforge.net/gazebo/xmlschema/#controller"
-       xmlns:joint="http://playerstage.sourceforge.net/gazebo/xmlschema/#slider"
-       xmlns:interface="http://playerstage.sourceforge.net/gazebo/xmlschema/#interface"
-       xmlns:body="http://playerstage.sourceforge.net/gazebo/xmlschema/#body"
-       xmlns:geom="http://playerstage.sourceforge.net/gazebo/xmlschema/#geom">
+<robot xmlns:xacro="http://ros.org/wiki/xacro">
   <include filename="$(find sr_hand)/model/hand_urdf/thumb/thbase.transmission.xacro" />
   <xacro:macro name="thbase" params="parent">
@@ -11,5 +5,5 @@
       <inertial>
 	<mass value="0.010" />
-	<origin xyz="0.034 0.0085 0.02924" rpy="0 0 0"/>
+	<origin xyz="0.034 0.0085 0.029" rpy="0 0 0"/>
 	<inertia  ixx="1.0" ixy="0.0"  ixz="0.0"  iyy="0.0"  iyz="0.0"
 	izz="0.0" />
@@ -32,15 +26,4 @@
     </link>
     <gazebo reference="thbase">
-      <sensor:contact name="thbase_contact_sensor">
-        <geom>thbase_geom</geom>
-       <updateRate>100.0</updateRate>
-        <controller:gazebo_ros_bumper name="thbase_gazebo_ros_bumper_controller" plugin="libgazebo_ros_bumper.so">
-          <alwaysOn>true</alwaysOn>
-          <updateRate>100.0</updateRate>
-          <frameName>thbase</frameName>
-          <bumperTopicName>thbase_bumper</bumperTopicName>
-          <interface:bumper name="thbase_gazebo_ros_bumper_iface" />
-        </controller:gazebo_ros_bumper>
-      </sensor:contact>
       <material>Gazebo/Grey</material>
     </gazebo>
@@ -48,5 +31,5 @@
       <parent link="${parent}"/>
       <child link="thbase"/>
-      <origin xyz="0.034 -0.0085 0.02924" rpy="0 ${M_PI/4} 0" />
+      <origin xyz="0.034 -0.0085 0.029" rpy="0 ${M_PI/4} 0" />
       <axis xyz="0 0 -1" />
       <limit lower="-1.047" upper="1.047" effort="10"

File: shadow_robot/sr_hand/model/hand_urdf/thumb/thdistal.urdf.xacro (robot description, xacro)
@@ -1,9 +1,3 @@
-<robot xmlns:xacro="http://ros.org/wiki/xacro"
-        xmlns:sensor="http://playerstage.sourceforge.net/gazebo/xmlschema/#sensor"
-       xmlns:controller="http://playerstage.sourceforge.net/gazebo/xmlschema/#controller"
-       xmlns:joint="http://playerstage.sourceforge.net/gazebo/xmlschema/#slider"
-       xmlns:interface="http://playerstage.sourceforge.net/gazebo/xmlschema/#interface"
-       xmlns:body="http://playerstage.sourceforge.net/gazebo/xmlschema/#body"
-       xmlns:geom="http://playerstage.sourceforge.net/gazebo/xmlschema/#geom">
+<robot xmlns:xacro="http://ros.org/wiki/xacro">
   <include filename="$(find sr_hand)/model/hand_urdf/thumb/thdistal.transmission.xacro" />
   <xacro:macro name="thdistal" params="parent">
@@ -16,5 +10,5 @@
       </inertial>
       <visual>
-	<origin xyz="0 0 0" rpy="${M_PI} -${M_PI/2} ${M_PI}" />
+	<origin xyz="0 0 0" rpy="0 0 0" />
 	<geometry name="thdistal_visual">
 	<mesh filename="package://sr_hand/model/meshes/TH1_z.mesh" scale="0.001 0.001 0.001" />
@@ -32,17 +26,5 @@
     </link>
     <gazebo reference="thdistal">
-      <sensor:contact name="thdistal_contact_sensor">
-        <geom>thdistal_geom</geom>
-       <updateRate>100.0</updateRate>
-        <controller:gazebo_ros_bumper name="thdistal_gazebo_ros_bumper_controller" plugin="libgazebo_ros_bumper.so">
-          <alwaysOn>true</alwaysOn>
-          <updateRate>100.0</updateRate>
-          <frameName>thdistal</frameName>
-          <bumperTopicName>thdistal_bumper</bumperTopicName>
-          <interface:bumper name="thdistal_gazebo_ros_bumper_iface" />
-        </controller:gazebo_ros_bumper>
-      </sensor:contact>
       <material>Gazebo/Grey</material>
-  	  <selfCollide>false</selfCollide>
     </gazebo>
     <joint name="THJ1" type="revolute">

File: shadow_robot/sr_hand/model/hand_urdf/thumb/thhub.urdf.xacro (robot description, xacro)
@@ -1,9 +1,3 @@
-<robot xmlns:xacro="http://ros.org/wiki/xacro"
-        xmlns:sensor="http://playerstage.sourceforge.net/gazebo/xmlschema/#sensor"
-       xmlns:controller="http://playerstage.sourceforge.net/gazebo/xmlschema/#controller"
-       xmlns:joint="http://playerstage.sourceforge.net/gazebo/xmlschema/#slider"
-       xmlns:interface="http://playerstage.sourceforge.net/gazebo/xmlschema/#interface"
-       xmlns:body="http://playerstage.sourceforge.net/gazebo/xmlschema/#body"
-       xmlns:geom="http://playerstage.sourceforge.net/gazebo/xmlschema/#geom">
+<robot xmlns:xacro="http://ros.org/wiki/xacro">
   <include filename="$(find sr_hand)/model/hand_urdf/thumb/thhub.transmission.xacro" />
   <xacro:macro name="thhub" params="parent">
@@ -32,15 +26,4 @@
     </link>
     <gazebo reference="thhub">
-      <sensor:contact name="thhub_contact_sensor">
-        <geom>thhub_geom</geom>
-       <updateRate>100.0</updateRate>
-        <controller:gazebo_ros_bumper name="thhub_gazebo_ros_bumper_controller" plugin="libgazebo_ros_bumper.so">
-          <alwaysOn>true</alwaysOn>
-          <updateRate>100.0</updateRate>
-          <frameName>thhub</frameName>
-          <bumperTopicName>thhub_bumper</bumperTopicName>
-          <interface:bumper name="thhub_gazebo_ros_bumper_iface" />
-        </controller:gazebo_ros_bumper>
-      </sensor:contact>
       <material>Gazebo/Grey</material>
     </gazebo>

File: shadow_robot/sr_hand/model/hand_urdf/thumb/thmiddle.urdf.xacro (robot description, xacro)
@@ -1,9 +1,3 @@
-<robot xmlns:xacro="http://ros.org/wiki/xacro"
-        xmlns:sensor="http://playerstage.sourceforge.net/gazebo/xmlschema/#sensor"
-       xmlns:controller="http://playerstage.sourceforge.net/gazebo/xmlschema/#controller"
-       xmlns:joint="http://playerstage.sourceforge.net/gazebo/xmlschema/#slider"
-       xmlns:interface="http://playerstage.sourceforge.net/gazebo/xmlschema/#interface"
-       xmlns:body="http://playerstage.sourceforge.net/gazebo/xmlschema/#body"
-       xmlns:geom="http://playerstage.sourceforge.net/gazebo/xmlschema/#geom">
+<robot xmlns:xacro="http://ros.org/wiki/xacro">
   <include filename="$(find sr_hand)/model/hand_urdf/thumb/thmiddle.transmission.xacro" />
   <xacro:macro name="thmiddle" params="parent">
@@ -16,5 +10,5 @@
       </inertial>
       <visual>
-	<origin xyz="0 0 0" rpy="0 -${M_PI/2} 0" />
+	<origin xyz="0 0 0" rpy="0 0 0" />
 	<geometry name="thmiddle_visual">
 	<mesh filename="package://sr_hand/model/meshes/TH2_z.mesh" scale="0.001 0.001 0.001" />
@@ -32,15 +26,4 @@
     </link>
     <gazebo reference="thmiddle">
-      <sensor:contact name="thmiddle_contact_sensor">
-        <geom>thmiddle_geom</geom>
-       <updateRate>100.0</updateRate>
-        <controller:gazebo_ros_bumper name="thmiddle_gazebo_ros_bumper_controller" plugin="libgazebo_ros_bumper.so">
-          <alwaysOn>true</alwaysOn>
-          <updateRate>100.0</updateRate>
-          <frameName>thmiddle</frameName>
-          <bumperTopicName>thmiddle_bumper</bumperTopicName>
-          <interface:bumper name="thmiddle_gazebo_ros_bumper_iface" />
-        </controller:gazebo_ros_bumper>
-      </sensor:contact>
       <material>Gazebo/Grey</material>
     </gazebo>
