Commit message: Proposed new hand meshes in two modes original one are saved full is the optimized version of the meshes envelop is the light version of the meshes without internal details
saved hand_urdf to original
proposed new hand_urdf adapted to new meshes and more cleaner (without many orientation change)

File: shadow_robot/sr_hand/model/hand_urdf/thumb/thproximal.urdf.xacro (robot description, xacro)
@@ -1,9 +1,3 @@
-<robot xmlns:xacro="http://ros.org/wiki/xacro"
-        xmlns:sensor="http://playerstage.sourceforge.net/gazebo/xmlschema/#sensor"
-       xmlns:controller="http://playerstage.sourceforge.net/gazebo/xmlschema/#controller"
-       xmlns:joint="http://playerstage.sourceforge.net/gazebo/xmlschema/#slider"
-       xmlns:interface="http://playerstage.sourceforge.net/gazebo/xmlschema/#interface"
-       xmlns:body="http://playerstage.sourceforge.net/gazebo/xmlschema/#body"
-       xmlns:geom="http://playerstage.sourceforge.net/gazebo/xmlschema/#geom">
+<robot xmlns:xacro="http://ros.org/wiki/xacro">
   <include filename="$(find sr_hand)/model/hand_urdf/thumb/thproximal.transmission.xacro" />
   <xacro:macro name="thproximal" params="parent">
@@ -18,5 +12,5 @@
 	<origin xyz="0 0 0" rpy="0 0 0" />
 	<geometry name="thproximal_visual">
-      <mesh filename="package://sr_hand/model/meshes/TH3_z.mesh" scale="0.01 0.01 0.01" />
+      <mesh filename="package://sr_hand/model/meshes/TH3_z.mesh" scale="0.001 0.001 0.001" />
       </geometry>
       <material name="shadow_thproximal_material">
@@ -32,15 +26,4 @@
     </link>
     <gazebo reference="thproximal">
-      <sensor:contact name="thproximal_contact_sensor">
-        <geom>thproximal_geom</geom>
-       <updateRate>100.0</updateRate>
-        <controller:gazebo_ros_bumper name="thproximal_gazebo_ros_bumper_controller" plugin="libgazebo_ros_bumper.so">
-          <alwaysOn>true</alwaysOn>
-          <updateRate>100.0</updateRate>
-          <frameName>thproximal</frameName>
-          <bumperTopicName>thproximal_bumper</bumperTopicName>
-          <interface:bumper name="thproximal_gazebo_ros_bumper_iface" />
-        </controller:gazebo_ros_bumper>
-      </sensor:contact>
       <material>Gazebo/Grey</material>
     </gazebo>

File: shadow_robot/sr_hand/model/hand_urdf/wrist/wrist.urdf.xacro (robot description, xacro)
@@ -11,5 +11,5 @@
       </inertial>
       <visual>
-	<origin xyz="0 0 0" rpy="${M_PI/2} 0 0" />
+	<origin xyz="0 0 0" rpy="0 0 0" />
 	<geometry name="wrist_visual">
 	  <mesh filename="package://sr_hand/model/meshes/wrist.mesh" scale="0.001 0.001 0.001" />

File: shadow_robot/sr_hand/model/robots/shadowhand_motor.urdf (robot description, URDF)
Before this commit: robot shadowhand_motor, 25 links, 24 joints
Links:
- link forearm_motor: geometry collision cylinder length=0.180 radius=0.06; visual mesh filename=package://sr_hand/model/meshes/forearm.mesh scale=0.001 0.001 0.001
- link thproximal: geometry collision box size=0.005 0.005 0.02; visual mesh filename=package://sr_hand/model/meshes/TH3_z.mesh scale=0.001 0.001 0.001
Joints:
- joint LFJ4: origin xyz=-0.01671 0 0.044 rpy=0 0 0 -> xyz=0 0 0.06579 rpy=0 0 0
- joint LFJ5: origin xyz=-0.01671 0 0.044 rpy=0 0 0 -> xyz=-0.033 0 0.02071 rpy=0 0 0
- joint THJ5: origin xyz=0.034 -0.0085 0.02924 rpy=0 0.785398163397 0 -> xyz=0.034 -0.0085 0.029 rpy=0 0.785398163397 0
