Commit message: fixes the bug for the J4s. (LFJ4 and RFJ4 don't move in the same direction as FFJ4 and MFJ4)

File: shadow_robot/sr_hand/model/hand_urdf/finger/classic_finger.urdf.xacro (robot description, xacro)
@@ -4,7 +4,8 @@
   <include filename="$(find sr_hand)/model/hand_urdf/finger/middle/middle.urdf.xacro" />
   <include filename="$(find sr_hand)/model/hand_urdf/finger/distal/distal.urdf.xacro" />
-  <xacro:macro name="finger" params="link_prefix joint_prefix parent *origin">
+  <xacro:macro name="finger" params="link_prefix joint_prefix parent *origin *axis">
     <xacro:knuckle link_prefix="${link_prefix}" joint_prefix="${joint_prefix}" parent="${parent}" >
       <insert_block name="origin" />
+      <insert_block name="axis"/>
     </xacro:knuckle>
     <xacro:proximal link_prefix="${link_prefix}" joint_prefix="${joint_prefix}" parent="${link_prefix}knuckle" >

File: shadow_robot/sr_hand/model/hand_urdf/finger/knuckle/knuckle.urdf.xacro (robot description, xacro)
@@ -32,5 +32,5 @@
       <!--<origin xyz="0.033 0 0.095" rpy="0 0 0" />-->
       <insert_block name="origin" />
-      <axis xyz="0 -1 0" />
+      <insert_block name="axis"/>
       <limit lower="-0.43633231299858238" upper="0.43633231299858238"
       effort="10" velocity="1.0"/>

File: shadow_robot/sr_hand/model/hand_urdf/finger/little_finger.urdf.xacro (robot description, xacro)
@@ -36,5 +36,5 @@
       <child link="lfknuckle"/>
       <origin xyz="-0.01671 0 0.044" rpy="0 0 0" />
-      <axis xyz="0 -1 0" />
+      <axis xyz="0 1 0" />
       <limit lower="-0.43633231299858238" upper="0.43633231299858238"
       effort="10" velocity="1.0"/>

File: shadow_robot/sr_hand/model/hand_urdf/full_hand_motor.urdf.xacro (robot description, xacro)
@@ -19,10 +19,13 @@
     <xacro:finger link_prefix="ff" joint_prefix="FF" parent="palm">
       <origin xyz="0.033 0 0.095" rpy="0 0 0" />
+      <axis xyz="0 -1 0" />
     </xacro:finger>
     <xacro:finger link_prefix="mf" joint_prefix="MF" parent="palm">
       <origin xyz="0.011 0 0.099" rpy="0 0 0" />
+      <axis xyz="0 -1 0" />
     </xacro:finger>
     <xacro:finger link_prefix="rf" joint_prefix="RF" parent="palm">
       <origin xyz="-0.011 0 0.095" rpy="0 0 0" />
+      <axis xyz="0 1 0" />
     </xacro:finger>
     <xacro:little_finger link_prefix="lf" joint_prefix="LF" parent="palm">

File: shadow_robot/sr_hand/model/hand_urdf/full_hand_muscle.urdf.xacro (robot description, xacro)
@@ -19,10 +19,13 @@
     <xacro:finger link_prefix="ff" joint_prefix="FF" parent="palm">
       <origin xyz="0.033 0 0.095" rpy="0 0 0" />
+      <axis xyz="0 -1 0" />
     </xacro:finger>
     <xacro:finger link_prefix="mf" joint_prefix="MF" parent="palm">
       <origin xyz="0.011 0 0.099" rpy="0 0 0" />
+      <axis xyz="0 -1 0" />
     </xacro:finger>
     <xacro:finger link_prefix="rf" joint_prefix="RF" parent="palm">
       <origin xyz="-0.011 0 0.095" rpy="0 0 0" />
+      <axis xyz="0 1 0" />
     </xacro:finger>
     <xacro:little_finger link_prefix="lf" joint_prefix="LF" parent="palm">

File: shadow_robot/sr_hand/model/robots/arm_and_hand_muscle.urdf (robot description, URDF)
Before this commit: robot arm_and_hand, 31 links, 30 joints
Joints:
- joint LFJ4: axis 0 -1 0 -> 0 1 0
- joint RFJ4: axis 0 -1 0 -> 0 1 0

File: shadow_robot/sr_hand/model/robots/shadowhand_muscle.urdf (robot description, URDF)
Before this commit: robot shadowhand_muscle, 25 links, 24 joints
Joints:
- joint LFJ4: axis 0 -1 0 -> 0 1 0
- joint RFJ4: axis 0 -1 0 -> 0 1 0
