Commit message: Corrected elements of arm_urdf to have correct positive joint orientation Corresponding meshes orientations still need to be fixed

File: shadow_robot/sr_hand/model/arm_urdf/hand_support/shadowarm_handsupport_motor.urdf.xacro (robot description, xacro)
@@ -30,5 +30,5 @@
       <child link="shadowarm_handsupport_motor"/>
       <origin xyz="0.131 0 -0.08" rpy="0 0 0" />
-      <axis xyz="1 0 0" />
+      <axis xyz="-1 0 0" />
       <limit lower="-${M_PI/2}" upper="${M_PI/2}"
       effort="10" velocity="1.0"/>

File: shadow_robot/sr_hand/model/arm_urdf/trunk/shadowarm_trunk.urdf.xacro (robot description, xacro)
@@ -30,6 +30,6 @@
       <child link="shadowarm_trunk"/>
       <origin xyz="0 0 0.01" rpy="0 0 0" />
-      <axis xyz="0 0 1" />
-      <limit lower="-${M_PI/2}" upper="${M_PI/4}"
+      <axis xyz="0 0 -1" />
+      <limit lower="-${M_PI/4}" upper="${M_PI/2}"
       effort="10" velocity="1.0"/>
       <dynamics damping="200.5"/>

File: shadow_robot/sr_hand/model/arm_urdf/upper_arm/shadowarm_upperarm.urdf.xacro (robot description, xacro)
@@ -9,5 +9,5 @@
       </inertial>
       <visual>
-	<origin xyz="0 0.067 0" rpy="-${M_PI/2} 0 -${M_PI/2}" />
+	<origin xyz="0 0.067 0" rpy="-${M_PI/2} -${M_PI/2} -${M_PI/2}" />
 	<geometry name="shadowarm_upperarm_visual">
 	  <mesh filename="package://sr_hand/model/meshes/arm/upper_arm.mesh" scale="0.001 0.001 0.001" />
@@ -30,5 +30,5 @@
       <child link="shadowarm_upperarm"/>
       <origin xyz="0 -0.134 0.5405" rpy="0 0 0" />
-      <axis xyz="0 1 0" />
+      <axis xyz="0 -1 0" />
       <limit lower="0" upper="${M_PI/2}" effort="10" velocity="1.0"/>
       <dynamics damping="50.5"/>

File: shadow_robot/sr_hand/model/robots/arm_and_hand_motor.urdf (robot description, URDF)
Before this commit: robot arm_and_hand, 31 links, 30 joints
Links:
- link forearm_motor: geometry collision cylinder length=0.180 radius=0.06; visual mesh filename=package://sr_hand/model/meshes/forearm.mesh scale=0.001 0.001 0.001
- link thproximal: geometry collision box size=0.005 0.005 0.02; visual mesh filename=package://sr_hand/model/meshes/TH3_z.mesh scale=0.001 0.001 0.001
Joints:
- joint LFJ4: origin xyz=-0.01671 0 0.044 rpy=0 0 0 -> xyz=0 0 0.06579 rpy=0 0 0
- joint LFJ5: origin xyz=-0.01671 0 0.044 rpy=0 0 0 -> xyz=-0.033 0 0.02071 rpy=0 0 0
- joint THJ5: origin xyz=0.034 -0.0085 0.02924 rpy=0 0.785398163397 0 -> xyz=0.034 -0.0085 0.029 rpy=0 0.785398163397 0
- joint forearm_rotation: axis 1 0 0 -> -1 0 0
- joint shoulder_rotation: axis 0 1 0 -> 0 -1 0
- joint trunk_rotation: axis 0 0 1 -> 0 0 -1; limit lower=-1.57079632679 upper=0.785398163397 effort=10 velocity=1.0 -> lower=-0.785398163397 upper=1.57079632679 effort=10 velocity=1.0

File: shadow_robot/sr_hand/model/robots/sr_arm_motor.urdf (robot description, URDF)
Before this commit: robot sr_arm_motor, 6 links, 5 joints
Joints:
- joint forearm_rotation: axis 1 0 0 -> -1 0 0
- joint shoulder_rotation: axis 0 1 0 -> 0 -1 0
- joint trunk_rotation: axis 0 0 1 -> 0 0 -1; limit lower=-1.57079632679 upper=0.785398163397 effort=10 velocity=1.0 -> lower=-0.785398163397 upper=1.57079632679 effort=10 velocity=1.0

Commit message: Finished correction of arm_urdf's to match existing hardware Changed arm to hand transform in sr_arm_motor.launch

File: shadow_robot/sr_hand/model/arm_urdf/hand_support/shadowarm_handsupport_motor.urdf.xacro (robot description, xacro)
@@ -9,5 +9,5 @@
       </inertial>
       <visual>
-	<origin xyz="-0.04 0 0" rpy="0 0 -${M_PI/2}"/>
+	<origin xyz="0 0 -0.04" rpy="${M_PI/2} 0 0"/>
 	<geometry name="shadowarm_handsupport_visual">
 	  <mesh filename="package://sr_hand/model/meshes/arm/elbow_rotate_motor.mesh" scale="0.001 0.001 0.001" />
@@ -16,5 +16,5 @@
       </visual>
       <collision>
-	<origin xyz="0 0 0" rpy="0 ${M_PI/2} 0"/>
+	<origin xyz="0 0 0" rpy="0 0 0"/>
 	<geometry name="shadowarm_handsupport_collision">
 	  <cylinder radius="0.06" length="0.001"/>
@@ -29,6 +29,6 @@
       <parent link="${parent}"/>
       <child link="shadowarm_handsupport_motor"/>
-      <origin xyz="0.131 0 -0.08" rpy="0 0 0" />
-      <axis xyz="-1 0 0" />
+      <origin xyz="0.08 0 0.131" rpy="0 0 0" />
+      <axis xyz="0 0 -1" />
       <limit lower="-${M_PI/2}" upper="${M_PI/2}"
       effort="10" velocity="1.0"/>

File: shadow_robot/sr_hand/model/arm_urdf/lower_arm/shadowarm_lowerarm.urdf.xacro (robot description, xacro)
@@ -4,10 +4,10 @@
     <link name="shadowarm_lowerarm">
 	<inertial>
-	  <origin xyz="0.0655 0 -0.08" rpy="0 0 0" />
+	  <origin xyz="0.08 0 0.0655" rpy="0 0 0" />
 	  <mass value="1.7" />
 	  <inertia  ixx="1.0" ixy="0.0"  ixz="0.0"  iyy="0.0"  iyz="0.0"  izz="0.0" />
 	</inertial>
 	<visual>
-	  <origin xyz="0.036 0 -0.03" rpy="${M_PI} 0.5 0"/>
+	  <origin xyz="0.03 0 0.036" rpy="${M_PI} ${0.5-M_PI/2} 0"/>
 	  <geometry name="shadowarm_lowerarm_visual">
 	    <mesh filename="package://sr_hand/model/meshes/arm/elbow_flex.mesh" scale="0.001 0.001 0.001" />
@@ -16,5 +16,5 @@
 	</visual>
 	<collision>
-	  <origin xyz="0.0655 0 -0.08" rpy="0 ${M_PI/2} 0"/>
+	  <origin xyz="0.08 0 0.0655" rpy="0 0 0"/>
 	  <geometry name="shadowarm_lowerarm_collision">
 	    <box size="0.03 0.03 0.131"/>
@@ -29,5 +29,5 @@
       <parent link="${parent}"/>
       <child link="shadowarm_lowerarm"/>
-      <origin xyz="0.369 0 0" rpy="0 0 0" />
+      <origin xyz="0 0 0.369" rpy="0 0 0" />
       <axis xyz="0 -1 0" />
       <limit lower="0" upper="2.09439510239"

File: shadow_robot/sr_hand/model/arm_urdf/upper_arm/shadowarm_upperarm.urdf.xacro (robot description, xacro)
@@ -4,10 +4,10 @@
     <link name="shadowarm_upperarm">
       <inertial>
-	<origin xyz="0.1845 -0.067 0" rpy="0 0 0" />
+	<origin xyz="0 -0.067 -0.1845" rpy="0 0 0" />
 	<mass value="2" />
 	<inertia  ixx="1.0" ixy="0.0"  ixz="0.0"  iyy="0.0"  iyz="0.0"  izz="0.0" />
       </inertial>
       <visual>
-	<origin xyz="0 0.067 0" rpy="-${M_PI/2} -${M_PI/2} -${M_PI/2}" />
+	<origin xyz="0 0.067 0" rpy="0 0 -${M_PI/2}" />
 	<geometry name="shadowarm_upperarm_visual">
 	  <mesh filename="package://sr_hand/model/meshes/arm/upper_arm.mesh" scale="0.001 0.001 0.001" />
@@ -16,5 +16,5 @@
       </visual>
       <collision>
-	<origin xyz="0.1845 0 0" rpy="0 ${M_PI/2} 0"/>
+	<origin xyz="0 0 0.1845" rpy="0 -${M_PI} 0"/>
 	<geometry name="shadowarm_upperarm_collision">
 	  <box size="0.03 0.03 0.369"/>
@@ -29,5 +29,5 @@
       <parent link="${parent}"/>
       <child link="shadowarm_upperarm"/>
-      <origin xyz="0 -0.134 0.5405" rpy="0 0 0" />
+      <origin xyz="0 -0.134 0.5405" rpy="0 -${M_PI} 0" />
       <axis xyz="0 -1 0" />
       <limit lower="0" upper="${M_PI/2}" effort="10" velocity="1.0"/>

File: shadow_robot/sr_hand/model/robots/sr_arm_motor.urdf (robot description, URDF)
Before this commit: robot sr_arm_motor, 6 links, 5 joints
Joints:
- joint elbow_abduction: origin xyz=0.369 0 0 rpy=0 0 0 -> xyz=0 0 0.369 rpy=0 0 0
- joint forearm_rotation: axis -1 0 0 -> 0 0 -1; origin xyz=0.131 0 -0.08 rpy=0 0 0 -> xyz=0.08 0 0.131 rpy=0 0 0
- joint shoulder_rotation: origin xyz=0 -0.134 0.5405 rpy=0 0 0 -> xyz=0 -0.134 0.5405 rpy=0 -3.14159265359 0
