Commit message: arm controller better tuned + fixed small things in models.

File: shadow_robot/sr_hand/model/arm_urdf/hand_support/shadowarm_handsupport_motor.transmission.xacro (robot description, xacro)
@@ -5,5 +5,5 @@
        xmlns:xacro="http://ros.org/wiki/xacro">
   <xacro:macro name="shadowarm_handsupport_motor_transmission">
-    <transmission type="SimpleTransmission" name="forearm_rotation_transmission">
+    <transmission type="pr2_mechanism_model/SimpleTransmission" name="forearm_rotation_transmission">
       <actuator name="forearm_rotation" />
       <joint name="forearm_rotation" />

File: shadow_robot/sr_hand/model/arm_urdf/hand_support/shadowarm_handsupport_motor.urdf.xacro (robot description, xacro)
@@ -33,5 +33,5 @@
       <limit lower="-${M_PI/2}" upper="${M_PI/2}"
       effort="10" velocity="1.0"/>
-      <dynamics damping="1"/>
+      <dynamics damping="3.5"/>
     </joint>
     <xacro:shadowarm_handsupport_motor_transmission />

File: shadow_robot/sr_hand/model/arm_urdf/hand_support/shadowarm_handsupport_muscle.transmission.xacro (robot description, xacro)
@@ -5,5 +5,5 @@
        xmlns:xacro="http://ros.org/wiki/xacro">
   <xacro:macro name="shadowarm_handsupport_muscle_transmission">
-    <transmission type="SimpleTransmission" name="forearm_rotation_transmission">
+    <transmission type="pr2_mechanism_model/SimpleTransmission" name="forearm_rotation_transmission">
       <actuator name="forearm_rotation" />
       <joint name="forearm_rotation" />

File: shadow_robot/sr_hand/model/arm_urdf/hand_support/shadowarm_handsupport_muscle.urdf.xacro (robot description, xacro)
@@ -33,5 +33,5 @@
       <limit lower="-${M_PI/2}" upper="${M_PI/2}"
       effort="10" velocity="1.0"/>
-      <dynamics damping="1"/>
+      <dynamics damping="3.5"/>
     </joint>
     <xacro:shadowarm_handsupport_muscle_transmission />

File: shadow_robot/sr_hand/model/arm_urdf/lower_arm/shadowarm_lowerarm.transmission.xacro (robot description, xacro)
@@ -5,5 +5,5 @@
        xmlns:xacro="http://ros.org/wiki/xacro">
   <xacro:macro name="shadowarm_lowerarm_transmission">
-    <transmission type="SimpleTransmission" name="elbow_abduction_transmission">
+    <transmission type="pr2_mechanism_model/SimpleTransmission" name="elbow_abduction_transmission">
       <actuator name="elbow_abduction" />
       <joint name="elbow_abduction" />

File: shadow_robot/sr_hand/model/arm_urdf/lower_arm/shadowarm_lowerarm.urdf.xacro (robot description, xacro)
@@ -33,5 +33,5 @@
       <limit lower="0" upper="2.09439510239"
       effort="10" velocity="1.0"/>
-      <dynamics damping="1"/>
+      <dynamics damping="3.5"/>
     </joint>
     <xacro:shadowarm_lowerarm_transmission />

File: shadow_robot/sr_hand/model/arm_urdf/trunk/shadowarm_trunk.transmission.xacro (robot description, xacro)
@@ -5,5 +5,5 @@
        xmlns:xacro="http://ros.org/wiki/xacro">
   <xacro:macro name="shadowarm_trunk_transmission">
-    <transmission type="SimpleTransmission" name="trunk_rotation_transmission">
+    <transmission type="pr2_mechanism_model/SimpleTransmission" name="trunk_rotation_transmission">
       <actuator name="trunk_rotation" />
       <joint name="trunk_rotation" />

File: shadow_robot/sr_hand/model/arm_urdf/trunk/shadowarm_trunk.urdf.xacro (robot description, xacro)
@@ -33,5 +33,5 @@
       <limit lower="-${M_PI/2}" upper="${M_PI/4}"
       effort="10" velocity="1.0"/>
-      <dynamics damping="1"/>
+      <dynamics damping="3.5"/>
     </joint>
     <xacro:shadowarm_trunk_transmission />

File: shadow_robot/sr_hand/model/arm_urdf/upper_arm/shadowarm_upperarm.transmission.xacro (robot description, xacro)
@@ -5,5 +5,5 @@
        xmlns:xacro="http://ros.org/wiki/xacro">
   <xacro:macro name="shadowarm_upperarm_transmission">
-    <transmission type="SimpleTransmission" name="shoulder_rotation_transmission">
+    <transmission type="pr2_mechanism_model/SimpleTransmission" name="shoulder_rotation_transmission">
       <actuator name="shoulder_rotation" />
       <joint name="shoulder_rotation" />

File: shadow_robot/sr_hand/model/arm_urdf/upper_arm/shadowarm_upperarm.urdf.xacro (robot description, xacro)
@@ -32,5 +32,5 @@
       <axis xyz="0 1 0" />
       <limit lower="0" upper="${M_PI/2}" effort="10" velocity="1.0"/>
-      <dynamics damping="1"/>
+      <dynamics damping="3.5"/>
     </joint>
     <xacro:shadowarm_upperarm_transmission />

Commit message: Changed arm_joint names in for virtual_arm to match platform joint names : trunk_rotation => ShoulderJRotate shoulder_rotation => ShoulderJSwing elbow_abduction => ElbowJSwing forearm_rotation => ElbowJRotate
Kept old names for transmissions, actuator and so on
Regenerated each of the urdfs to use new names

File: shadow_robot/sr_hand/model/arm_urdf/hand_support/shadowarm_handsupport_motor.transmission.xacro (robot description, xacro)
@@ -7,5 +7,5 @@
     <transmission type="pr2_mechanism_model/SimpleTransmission" name="forearm_rotation_transmission">
       <actuator name="forearm_rotation" />
-      <joint name="forearm_rotation" />
+      <joint name="ElbowJRotate" />
       <mechanicalReduction>1</mechanicalReduction>
       <motorTorqueConstant>1</motorTorqueConstant>

File: shadow_robot/sr_hand/model/arm_urdf/hand_support/shadowarm_handsupport_motor.urdf.xacro (robot description, xacro)
@@ -26,5 +26,5 @@
       <selfCollide>true</selfCollide>
     </gazebo>
-    <joint name="forearm_rotation" type="revolute">
+    <joint name="ElbowJRotate" type="revolute">
       <parent link="${parent}"/>
       <child link="shadowarm_handsupport_motor"/>

File: shadow_robot/sr_hand/model/arm_urdf/hand_support/shadowarm_handsupport_muscle.transmission.xacro (robot description, xacro)
@@ -7,5 +7,5 @@
     <transmission type="pr2_mechanism_model/SimpleTransmission" name="forearm_rotation_transmission">
       <actuator name="forearm_rotation" />
-      <joint name="forearm_rotation" />
+      <joint name="ElbowJRotate" />
       <mechanicalReduction>1</mechanicalReduction>
       <motorTorqueConstant>1</motorTorqueConstant>

File: shadow_robot/sr_hand/model/arm_urdf/hand_support/shadowarm_handsupport_muscle.urdf.xacro (robot description, xacro)
@@ -26,5 +26,5 @@
       <selfCollide>true</selfCollide>
     </gazebo>
-    <joint name="forearm_rotation" type="revolute">
+    <joint name="ElbowJRotate" type="revolute">
       <parent link="${parent}"/>
       <child link="shadowarm_handsupport_muscle"/>

File: shadow_robot/sr_hand/model/arm_urdf/lower_arm/shadowarm_lowerarm.transmission.xacro (robot description, xacro)
@@ -7,5 +7,5 @@
     <transmission type="pr2_mechanism_model/SimpleTransmission" name="elbow_abduction_transmission">
       <actuator name="elbow_abduction" />
-      <joint name="elbow_abduction" />
+      <joint name="ElbowJSwing" />
       <mechanicalReduction>1</mechanicalReduction>
       <motorTorqueConstant>1</motorTorqueConstant>

File: shadow_robot/sr_hand/model/arm_urdf/lower_arm/shadowarm_lowerarm.urdf.xacro (robot description, xacro)
@@ -26,5 +26,5 @@
 	<selfCollide>true</selfCollide>
     </gazebo>
-    <joint name="elbow_abduction" type="revolute">
+    <joint name="ElbowJSwing" type="revolute">
       <parent link="${parent}"/>
       <child link="shadowarm_lowerarm"/>

File: shadow_robot/sr_hand/model/arm_urdf/trunk/shadowarm_trunk.transmission.xacro (robot description, xacro)
@@ -7,5 +7,5 @@
     <transmission type="pr2_mechanism_model/SimpleTransmission" name="trunk_rotation_transmission">
       <actuator name="trunk_rotation" />
-      <joint name="trunk_rotation" />
+      <joint name="ShadowJRotate" />
       <mechanicalReduction>1</mechanicalReduction>
       <motorTorqueConstant>1</motorTorqueConstant>

File: shadow_robot/sr_hand/model/arm_urdf/trunk/shadowarm_trunk.urdf.xacro (robot description, xacro)
@@ -26,5 +26,5 @@
 	<selfCollide>true</selfCollide>
       </gazebo>
-    <joint name="trunk_rotation" type="revolute">
+    <joint name="ShoulderJRotate" type="revolute">
       <parent link="${parent}"/>
       <child link="shadowarm_trunk"/>

File: shadow_robot/sr_hand/model/arm_urdf/upper_arm/shadowarm_upperarm.transmission.xacro (robot description, xacro)
@@ -7,5 +7,5 @@
     <transmission type="pr2_mechanism_model/SimpleTransmission" name="shoulder_rotation_transmission">
       <actuator name="shoulder_rotation" />
-      <joint name="shoulder_rotation" />
+      <joint name="ShoulderJSwing" />
       <mechanicalReduction>1</mechanicalReduction>
       <motorTorqueConstant>1</motorTorqueConstant>

File: shadow_robot/sr_hand/model/arm_urdf/upper_arm/shadowarm_upperarm.urdf.xacro (robot description, xacro)
@@ -26,5 +26,5 @@
       <selfCollide>true</selfCollide>
     </gazebo>
-    <joint name="shoulder_rotation" type="revolute">
+    <joint name="ShoulderJSwing" type="revolute">
       <parent link="${parent}"/>
       <child link="shadowarm_upperarm"/>

File: shadow_robot/sr_hand/model/robots/arm_and_hand_motor.urdf (robot description, URDF)
Before this commit: robot arm_and_hand, 31 links, 30 joints
Joints:
- removed joint elbow_abduction
- removed joint forearm_rotation
- removed joint shoulder_rotation
- removed joint trunk_rotation
- added joint ElbowJRotate: type revolute, parent shadowarm_lowerarm, child shadowarm_handsupport_motor, origin xyz=0.08 0 0.131 rpy=0 0 0, axis 0 0 -1, limit lower=-1.57079632679 upper=1.57079632679 effort=10 velocity=1.0
- added joint ElbowJSwing: type revolute, parent shadowarm_upperarm, child shadowarm_lowerarm, origin xyz=0 0 0.369 rpy=0 0 0, axis 0 -1 0, limit lower=0 upper=2.09439510239 effort=10 velocity=1.0
- added joint ShoulderJRotate: type revolute, parent shadowarm_base, child shadowarm_trunk, origin xyz=0 0 0.01 rpy=0 0 0, axis 0 0 -1, limit lower=-0.785398163397 upper=1.57079632679 effort=10 velocity=1.0
- added joint ShoulderJSwing: type revolute, parent shadowarm_trunk, child shadowarm_upperarm, origin xyz=0 -0.134 0.5405 rpy=0 -3.14159265359 0, axis 0 -1 0, limit lower=0 upper=1.57079632679 effort=10 velocity=1.0

File: shadow_robot/sr_hand/model/robots/arm_and_hand_muscle.urdf (robot description, URDF)
Before this commit: robot arm_and_hand, 31 links, 30 joints
Links:
- link thproximal: geometry collision box size=0.005 0.005 0.02; visual mesh filename=package://sr_hand/model/meshes/TH3_z.mesh scale=0.001 0.001 0.001
Joints:
- removed joint elbow_abduction
- removed joint forearm_rotation
- removed joint shoulder_rotation
- removed joint trunk_rotation
- added joint ElbowJRotate: type revolute, parent shadowarm_lowerarm, child shadowarm_handsupport_muscle, origin xyz=0.131 0 -0.08 rpy=0 0 0, axis 1 0 0, limit lower=-1.57079632679 upper=1.57079632679 effort=10 velocity=1.0
- added joint ElbowJSwing: type revolute, parent shadowarm_upperarm, child shadowarm_lowerarm, origin xyz=0 0 0.369 rpy=0 0 0, axis 0 -1 0, limit lower=0 upper=2.09439510239 effort=10 velocity=1.0
- added joint ShoulderJRotate: type revolute, parent shadowarm_base, child shadowarm_trunk, origin xyz=0 0 0.01 rpy=0 0 0, axis 0 0 -1, limit lower=-0.785398163397 upper=1.57079632679 effort=10 velocity=1.0
- added joint ShoulderJSwing: type revolute, parent shadowarm_trunk, child shadowarm_upperarm, origin xyz=0 -0.134 0.5405 rpy=0 -3.14159265359 0, axis 0 -1 0, limit lower=0 upper=1.57079632679 effort=10 velocity=1.0
- joint LFJ4: origin xyz=-0.01671 0 0.044 rpy=0 0 0 -> xyz=0 0 0.06579 rpy=0 0 0
- joint LFJ5: origin xyz=-0.01671 0 0.044 rpy=0 0 0 -> xyz=-0.033 0 0.02071 rpy=0 0 0
- joint THJ5: origin xyz=0.034 -0.0085 0.02924 rpy=0 0.785398163397 0 -> xyz=0.034 -0.0085 0.029 rpy=0 0.785398163397 0

File: shadow_robot/sr_hand/model/robots/shadowhand_muscle.urdf (robot description, URDF)
Before this commit: robot shadowhand_muscle, 25 links, 24 joints
Links:
- link thproximal: geometry collision box size=0.005 0.005 0.02; visual mesh filename=package://sr_hand/model/meshes/TH3_z.mesh scale=0.001 0.001 0.001
Joints:
- joint LFJ4: origin xyz=-0.01671 0 0.044 rpy=0 0 0 -> xyz=0 0 0.06579 rpy=0 0 0
- joint LFJ5: origin xyz=-0.01671 0 0.044 rpy=0 0 0 -> xyz=-0.033 0 0.02071 rpy=0 0 0
- joint THJ5: origin xyz=0.034 -0.0085 0.02924 rpy=0 0.785398163397 0 -> xyz=0.034 -0.0085 0.029 rpy=0 0.785398163397 0

File: shadow_robot/sr_hand/model/robots/sr_arm_motor.urdf (robot description, URDF)
Before this commit: robot sr_arm_motor, 6 links, 5 joints
Joints:
- removed joint elbow_abduction
- removed joint forearm_rotation
- removed joint shoulder_rotation
- removed joint trunk_rotation
- added joint ElbowJRotate: type revolute, parent shadowarm_lowerarm, child shadowarm_handsupport_motor, origin xyz=0.08 0 0.131 rpy=0 0 0, axis 0 0 -1, limit lower=-1.57079632679 upper=1.57079632679 effort=10 velocity=1.0
- added joint ElbowJSwing: type revolute, parent shadowarm_upperarm, child shadowarm_lowerarm, origin xyz=0 0 0.369 rpy=0 0 0, axis 0 -1 0, limit lower=0 upper=2.09439510239 effort=10 velocity=1.0
- added joint ShoulderJRotate: type revolute, parent shadowarm_base, child shadowarm_trunk, origin xyz=0 0 0.01 rpy=0 0 0, axis 0 0 -1, limit lower=-0.785398163397 upper=1.57079632679 effort=10 velocity=1.0
- added joint ShoulderJSwing: type revolute, parent shadowarm_trunk, child shadowarm_upperarm, origin xyz=0 -0.134 0.5405 rpy=0 -3.14159265359 0, axis 0 -1 0, limit lower=0 upper=1.57079632679 effort=10 velocity=1.0

File: shadow_robot/sr_hand/model/robots/sr_arm_muscle.urdf (robot description, URDF)
Before this commit: robot sr_arm_muscle, 6 links, 5 joints
Joints:
- removed joint elbow_abduction
- removed joint forearm_rotation
- removed joint shoulder_rotation
- removed joint trunk_rotation
- added joint ElbowJRotate: type revolute, parent shadowarm_lowerarm, child shadowarm_handsupport_muscle, origin xyz=0.131 0 -0.08 rpy=0 0 0, axis 1 0 0, limit lower=-1.57079632679 upper=1.57079632679 effort=10 velocity=1.0
- added joint ElbowJSwing: type revolute, parent shadowarm_upperarm, child shadowarm_lowerarm, origin xyz=0 0 0.369 rpy=0 0 0, axis 0 -1 0, limit lower=0 upper=2.09439510239 effort=10 velocity=1.0
- added joint ShoulderJRotate: type revolute, parent shadowarm_base, child shadowarm_trunk, origin xyz=0 0 0.01 rpy=0 0 0, axis 0 0 -1, limit lower=-0.785398163397 upper=1.57079632679 effort=10 velocity=1.0
- added joint ShoulderJSwing: type revolute, parent shadowarm_trunk, child shadowarm_upperarm, origin xyz=0 -0.134 0.5405 rpy=0 -3.14159265359 0, axis 0 -1 0, limit lower=0 upper=1.57079632679 effort=10 velocity=1.0

File: shadow_robot/sr_hand/model/sr_arm_motor.urdf (robot description, URDF)
Before this commit: robot sr_arm_motor, 5 links, 4 joints
Links:
- added link world
Joints:
- removed joint elbow_abduction
- removed joint forearm_rotation
- removed joint shoulder_rotation
- removed joint trunk_rotation
- added joint ElbowJRotate: type revolute, parent shadowarm_lowerarm, child shadowarm_handsupport_motor, origin xyz=0.08 0 0.131 rpy=0 0 0, axis 0 0 -1, limit lower=-1.57079632679 upper=1.57079632679 effort=10 velocity=1.0
- added joint ElbowJSwing: type revolute, parent shadowarm_upperarm, child shadowarm_lowerarm, origin xyz=0 0 0.369 rpy=0 0 0, axis 0 -1 0, limit lower=0 upper=2.09439510239 effort=10 velocity=1.0
- added joint ShoulderJRotate: type revolute, parent shadowarm_base, child shadowarm_trunk, origin xyz=0 0 0.01 rpy=0 0 0, axis 0 0 -1, limit lower=-0.785398163397 upper=1.57079632679 effort=10 velocity=1.0
- added joint ShoulderJSwing: type revolute, parent shadowarm_trunk, child shadowarm_upperarm, origin xyz=0 -0.134 0.5405 rpy=0 -3.14159265359 0, axis 0 -1 0, limit lower=0 upper=1.57079632679 effort=10 velocity=1.0
- added joint base_fix: type fixed, parent world, child shadowarm_base, origin xyz=0 0 0 rpy=0 0 0
