Commit message: muscle hand position corrected.

File: shadow_robot/sr_hand/model/arm_urdf/hand_support/shadowarm_handsupport_muscle.urdf.xacro (robot description, xacro)
@@ -4,10 +4,10 @@
     <link name="shadowarm_handsupport_muscle">
       <inertial>
-	<origin xyz="0 0 0" rpy="0 ${M_PI/2} 0" />
+	<origin xyz="0 0 0" rpy="0 0 0" />
 	<mass value="0.75" />
 	<inertia  ixx="1.0" ixy="0.0"  ixz="0.0"  iyy="0.0"  iyz="0.0"  izz="0.0" />
       </inertial>
       <visual>
-	<origin xyz="-0.04 0 0" rpy="0 0 -${M_PI/2}"/>
+	<origin xyz="0 0 -0.04" rpy="${M_PI/2} 0 0"/>
 	<geometry name="shadowarm_handsupport_visual">
 	  <mesh filename="package://sr_hand/model/meshes/arm/elbow_rotate_muscle.mesh" scale="0.001 0.001 0.001" />
@@ -16,5 +16,5 @@
       </visual>
       <collision>
-	<origin xyz="0 0 0" rpy="0 ${M_PI/2} 0"/>
+	<origin xyz="0 0 0" rpy="0 0 0"/>
 	<geometry name="shadowarm_handsupport_collision">
 	  <cylinder radius="0.06" length="0.001"/>
@@ -29,5 +29,5 @@
       <parent link="${parent}"/>
       <child link="shadowarm_handsupport_muscle"/>
-      <origin xyz="0.131 0 -0.08" rpy="0 0 0" />
+      <origin xyz="0.08 0 0.131" rpy="0 0 0" />
       <axis xyz="1 0 0" />
       <limit lower="-${M_PI/2}" upper="${M_PI/2}"

File: shadow_robot/sr_hand/model/robots/arm_and_hand_muscle.urdf (robot description, URDF)
Before this commit: robot arm_and_hand, 31 links, 30 joints
Joints:
- joint ElbowJRotate: origin xyz=0.131 0 -0.08 rpy=0 0 0 -> xyz=0.08 0 0.131 rpy=0 0 0

File: shadow_robot/sr_hand/model/robots/sr_arm_muscle.urdf (robot description, URDF)
Before this commit: robot sr_arm_muscle, 6 links, 5 joints
Joints:
- joint ElbowJRotate: origin xyz=0.131 0 -0.08 rpy=0 0 0 -> xyz=0.08 0 0.131 rpy=0 0 0

Commit message: Solved some orientation issues in the model.

File: shadow_robot/sr_hand/model/arm_urdf/hand_support/shadowarm_handsupport_muscle.urdf.xacro (robot description, xacro)
@@ -30,5 +30,5 @@
       <child link="shadowarm_handsupport_muscle"/>
       <origin xyz="0.08 0 0.131" rpy="0 0 0" />
-      <axis xyz="1 0 0" />
+      <axis xyz="0 0 -1" />
       <limit lower="-${M_PI/2}" upper="${M_PI/2}"
       effort="10" velocity="1.0"/>

File: shadow_robot/sr_hand/model/arm_urdf/trunk/shadowarm_trunk.urdf.xacro (robot description, xacro)
@@ -30,5 +30,5 @@
       <child link="shadowarm_trunk"/>
       <origin xyz="0 0 0.01" rpy="0 0 0" />
-      <axis xyz="0 0 -1" />
+      <axis xyz="0 0 1" />
       <limit lower="-${M_PI/4}" upper="${M_PI/2}"
       effort="10" velocity="1.0"/>

File: shadow_robot/sr_hand/model/robots/arm_and_hand_motor.urdf (robot description, URDF)
Before this commit: robot arm_and_hand, 31 links, 30 joints
Joints:
- joint ShoulderJRotate: axis 0 0 -1 -> 0 0 1

File: shadow_robot/sr_hand/model/robots/arm_and_hand_muscle.urdf (robot description, URDF)
Before this commit: robot arm_and_hand, 31 links, 30 joints
Joints:
- joint ElbowJRotate: axis 1 0 0 -> 0 0 -1
- joint ShoulderJRotate: axis 0 0 -1 -> 0 0 1

File: shadow_robot/sr_hand/model/robots/sr_arm_motor.urdf (robot description, URDF)
Before this commit: robot sr_arm_motor, 6 links, 5 joints
Joints:
- joint ShoulderJRotate: axis 0 0 -1 -> 0 0 1

File: shadow_robot/sr_hand/model/robots/sr_arm_muscle.urdf (robot description, URDF)
Before this commit: robot sr_arm_muscle, 6 links, 5 joints
Joints:
- joint ElbowJRotate: axis 1 0 0 -> 0 0 -1
- joint ShoulderJRotate: axis 0 0 -1 -> 0 0 1

Commit message: Corrected thdistal frame to be the same orientation as other distal phalanxes Modified thdistal mesh (TH1_z.mesh) to be aligned as other distal phalanxes Added RViz tactile markers (in sr_tactile_sensors) (only tested with virtual sensors) Renamed mesh storage place (provided meshes are all envelop versions in standard or light (30% decimated) mode). Full meshes but still optimized versions available soon

File: shadow_robot/sr_hand/model/arm_urdf/hand_support/shadowarm_handsupport_muscle.urdf.xacro (robot description, xacro)
@@ -4,10 +4,10 @@
     <link name="shadowarm_handsupport_muscle">
       <inertial>
-	<origin xyz="0 0 0" rpy="0 ${M_PI/2} 0" />
+	<origin xyz="0 0 0" rpy="0 0 0" />
 	<mass value="0.75" />
 	<inertia  ixx="1.0" ixy="0.0"  ixz="0.0"  iyy="0.0"  iyz="0.0"  izz="0.0" />
       </inertial>
       <visual>
-	<origin xyz="-0.04 0 0" rpy="0 0 -${M_PI/2}"/>
+	<origin xyz="0 0 -0.04" rpy="${M_PI/2} 0 0"/>
 	<geometry name="shadowarm_handsupport_visual">
 	  <mesh filename="package://sr_hand/model/meshes/arm/elbow_rotate_muscle.mesh" scale="0.001 0.001 0.001" />
@@ -29,6 +29,6 @@
       <parent link="${parent}"/>
       <child link="shadowarm_handsupport_muscle"/>
-      <origin xyz="0.131 0 -0.08" rpy="0 0 0" />
-      <axis xyz="1 0 0" />
+      <origin xyz="0.08 0 0.131" rpy="0 0 0" />
+      <axis xyz="0 0 -1" />
       <limit lower="-${M_PI/2}" upper="${M_PI/2}"
       effort="10" velocity="1.0"/>

File: shadow_robot/sr_hand/model/hand_urdf/thumb/thdistal.urdf.xacro (robot description, xacro)
@@ -31,6 +31,6 @@
       <parent link="${parent}"/>
       <child link="thdistal"/>
-      <origin xyz="0 0 0.032" rpy="0 0 0" />
-      <axis xyz="0 -1 0" />
+      <origin xyz="0 0 0.032" rpy="0 0 -1.570796327" />
+      <axis xyz="1 0 0" />
       <limit lower="0" upper="1.571" effort="10"
       velocity="1.0" />

File: shadow_robot/sr_hand/model/robots/arm_and_hand_motor.urdf (robot description, URDF)
Before this commit: robot arm_and_hand, 31 links, 30 joints
Joints:
- joint THJ1: axis 0 -1 0 -> 1 0 0; origin xyz=0 0 0.032 rpy=0 0 0 -> xyz=0 0 0.032 rpy=0 0 -1.570796327

File: shadow_robot/sr_hand/model/robots/arm_and_hand_muscle.urdf (robot description, URDF)
Before this commit: robot arm_and_hand, 31 links, 30 joints
Joints:
- joint ElbowJRotate: axis 1 0 0 -> 0 0 -1; origin xyz=0.131 0 -0.08 rpy=0 0 0 -> xyz=0.08 0 0.131 rpy=0 0 0
- joint THJ1: axis 0 -1 0 -> 1 0 0; origin xyz=0 0 0.032 rpy=0 0 0 -> xyz=0 0 0.032 rpy=0 0 -1.570796327

File: shadow_robot/sr_hand/model/robots/shadowhand_motor.urdf (robot description, URDF)
Before this commit: robot shadowhand_motor, 25 links, 24 joints
Joints:
- joint THJ1: axis 0 -1 0 -> 1 0 0; origin xyz=0 0 0.032 rpy=0 0 0 -> xyz=0 0 0.032 rpy=0 0 -1.570796327

File: shadow_robot/sr_hand/model/robots/shadowhand_muscle.urdf (robot description, URDF)
Before this commit: robot shadowhand_muscle, 25 links, 24 joints
Joints:
- joint THJ1: axis 0 -1 0 -> 1 0 0; origin xyz=0 0 0.032 rpy=0 0 0 -> xyz=0 0 0.032 rpy=0 0 -1.570796327

File: shadow_robot/sr_hand/model/robots/sr_arm_muscle.urdf (robot description, URDF)
Before this commit: robot sr_arm_muscle, 6 links, 5 joints
Joints:
- joint ElbowJRotate: axis 1 0 0 -> 0 0 -1; origin xyz=0.131 0 -0.08 rpy=0 0 0 -> xyz=0.08 0 0.131 rpy=0 0 0
