Commit message: solves weird hand orientation in Gazebo

File: shadow_robot/sr_hand/model/robots/xacro/arm_and_hand_motor.urdf.xacro (robot description, xacro)
@@ -9,5 +9,5 @@
     <parent link="shadowarm_handsupport_motor"/>
     <child link="forearm_motor"/>
-    <origin xyz="0 0 0" rpy="${M_PI/2} 0 ${M_PI/2}" />
+    <origin xyz="0 0 0" rpy="0 0 ${M_PI/2}" />
     <axis xyz="0 -1 0" />
     <limit lower="0" upper="0" effort="10"

File: shadow_robot/sr_hand/model/robots/xacro/arm_and_hand_muscle.urdf.xacro (robot description, xacro)
@@ -9,5 +9,5 @@
     <parent link="shadowarm_handsupport_muscle"/>
     <child link="forearm_muscle"/>
-    <origin xyz="0 0 0" rpy="${M_PI/2} 0 ${M_PI/2}" />
+    <origin xyz="0 0 0" rpy="0 0 ${M_PI/2}" />
     <axis xyz="0 -1 0" />
     <limit lower="0" upper="0" effort="10"
