Commit message: better organization of the models + added the desk to the arm_and_hand_motor.urdf.xacro file

File: shadow_robot/sr_hand/model/desk/desk.urdf.xacro (robot description, xacro)
@@ -1,6 +1,4 @@
 <robot name="desk" xmlns:body="http://playerstage.sourceforge.net/gazebo/xmlschema/#body" xmlns:geom="http://playerstage.sourceforge.net/gazebo/xmlschema/#geom" xmlns:interface="http://playerstage.sourceforge.net/gazebo/xmlschema/#interface" xmlns:joint="http://playerstage.sourceforge.net/gazebo/xmlschema/#slider" xmlns:xacro="http://ros.org/wiki/xacro">
-  <material name="Green">
-    <color rgba="0.0 0.8 0.0 1.0"/>
-  </material>
+  <xacro:macro name="desk">
   <link name="desk_pillar">
     <inertial>
@@ -56,3 +54,4 @@
     <origin rpy="0 0 0" xyz="0 0 0.01"/>
   </joint>
+  </xacro:macro>
 </robot>

File: shadow_robot/sr_hand/model/robots/xacro/arm_and_hand_motor.urdf.xacro (robot description, xacro)
@@ -4,4 +4,11 @@
   <include filename="$(find sr_hand)/model/hand_urdf/full_hand_motor.urdf.xacro" />
   <include filename="$(find sr_hand)/model/gazebo/gazebo.urdf.xacro" />
+  <include filename="$(find sr_hand)/model/desk/desk.urdf.xacro" />
+  <xacro:desk/>
+  <joint name="base_fix" type="fixed">
+    <parent link="desk_pillar"/>
+    <child link="shadowarm_base"/>
+    <origin rpy="0 0 0" xyz="0 0 1.0"/>
+  </joint>
   <xacro:sr_arm_motor>
   </xacro:sr_arm_motor>
