Commit message: gazebo controllers added for the whole hand and arm models. PID need to be set in yaml controller files

File: shadow_robot/sr_hand/model/arm_urdf/base/shadowarm_base.urdf.xacro (robot description, xacro)
@@ -2,4 +2,5 @@
 <property name="M_PI" value="3.1415926535897931" />
 <xacro:macro name="shadowarm_base">
+  <link name="world" />
   <link name="shadowarm_base">
     <inertial>
@@ -26,4 +27,9 @@
     <selfCollide>true</selfCollide>
   </gazebo>
+  <joint name="base_fix" type="fixed">
+    <parent link="world"/>
+    <child link="shadowarm_base"/>
+    <origin rpy="0 0 0" xyz="0 0 0"/>
+  </joint>
 </xacro:macro>
 </robot>

File: shadow_robot/sr_hand/model/arm_urdf/hand_support/shadowarm_handsupport_motor.urdf.xacro (robot description, xacro)
@@ -33,4 +33,5 @@
       <limit lower="-${M_PI/2}" upper="${M_PI/2}"
       effort="10" velocity="1.0"/>
+      <dynamics damping="1"/>
     </joint>
     <xacro:shadowarm_handsupport_motor_transmission />

File: shadow_robot/sr_hand/model/arm_urdf/hand_support/shadowarm_handsupport_muscle.urdf.xacro (robot description, xacro)
@@ -33,4 +33,5 @@
       <limit lower="-${M_PI/2}" upper="${M_PI/2}"
       effort="10" velocity="1.0"/>
+      <dynamics damping="1"/>
     </joint>
     <xacro:shadowarm_handsupport_muscle_transmission />

File: shadow_robot/sr_hand/model/arm_urdf/lower_arm/shadowarm_lowerarm.urdf.xacro (robot description, xacro)
@@ -27,10 +27,11 @@
     </gazebo>
     <joint name="elbow_abduction" type="revolute">
-	<parent link="${parent}"/>
-	<child link="shadowarm_lowerarm"/>
-	<origin xyz="0.369 0 0" rpy="0 0 0" />
-	<axis xyz="0 -1 0" />
-	<limit lower="0" upper="2.09439510239"
-	effort="10" velocity="1.0"/>
+      <parent link="${parent}"/>
+      <child link="shadowarm_lowerarm"/>
+      <origin xyz="0.369 0 0" rpy="0 0 0" />
+      <axis xyz="0 -1 0" />
+      <limit lower="0" upper="2.09439510239"
+      effort="10" velocity="1.0"/>
+      <dynamics damping="1"/>
     </joint>
     <xacro:shadowarm_lowerarm_transmission />

File: shadow_robot/sr_hand/model/arm_urdf/trunk/shadowarm_trunk.urdf.xacro (robot description, xacro)
@@ -33,4 +33,5 @@
       <limit lower="-${M_PI/2}" upper="${M_PI/4}"
       effort="10" velocity="1.0"/>
+      <dynamics damping="1"/>
     </joint>
     <xacro:shadowarm_trunk_transmission />

File: shadow_robot/sr_hand/model/arm_urdf/upper_arm/shadowarm_upperarm.urdf.xacro (robot description, xacro)
@@ -32,4 +32,5 @@
       <axis xyz="0 1 0" />
       <limit lower="0" upper="${M_PI/2}" effort="10" velocity="1.0"/>
+      <dynamics damping="1"/>
     </joint>
     <xacro:shadowarm_upperarm_transmission />

File: shadow_robot/sr_hand/model/hand_urdf/finger/distal/distal.urdf.xacro (robot description, xacro)
@@ -1,3 +1,4 @@
 <robot xmlns:xacro="http://ros.org/wiki/xacro">
+  <include filename="$(find sr_hand)/model/hand_urdf/finger/distal/distal.transmission.xacro" />
   <xacro:macro name="distal" params="link_prefix joint_prefix parent">
     <link name="${link_prefix}distal">
@@ -33,4 +34,5 @@
       velocity="1.0" />
     </joint>
+    <xacro:distal_transmission />
   </xacro:macro>
 </robot>

File: shadow_robot/sr_hand/model/hand_urdf/finger/knuckle/knuckle.urdf.xacro (robot description, xacro)
@@ -1,3 +1,4 @@
 <robot xmlns:xacro="http://ros.org/wiki/xacro">
+  <include filename="$(find sr_hand)/model/hand_urdf/finger/knuckle/knuckle.transmission.xacro" />
   <xacro:macro name="knuckle" params="link_prefix joint_prefix parent *origin">
     <link name="${link_prefix}knuckle">
@@ -35,4 +36,5 @@
       effort="10" velocity="1.0"/>
     </joint>
+    <xacro:knuckle_transmission />
   </xacro:macro>
 </robot>

File: shadow_robot/sr_hand/model/hand_urdf/finger/lfmetacarpal/lfmetacarpal.urdf.xacro (robot description, xacro)
@@ -1,3 +1,4 @@
 <robot xmlns:xacro="http://ros.org/wiki/xacro">
+  <include filename="$(find sr_hand)/model/hand_urdf/finger/lfmetacarpal/lfmetacarpal.transmission.xacro" />
   <xacro:macro name="lfmetacarpal" params="parent">
     <link name="lfmetacarpal">
@@ -33,4 +34,5 @@
       velocity="1.0" />
     </joint>
+    <xacro:lfmetacarpal_transmission />
   </xacro:macro>
 </robot>

File: shadow_robot/sr_hand/model/hand_urdf/finger/little_finger.urdf.xacro (robot description, xacro)
@@ -40,4 +40,11 @@
       effort="10" velocity="1.0"/>
     </joint>
+    <transmission type="SimpleTransmission" name="lfknuckle_transmission">
+      <actuator name="LFJ4" />
+      <joint name="LFJ4" />
+      <mechanicalReduction>1</mechanicalReduction>
+      <motorTorqueConstant>1</motorTorqueConstant>
+      <pulsesPerRevolution>90000</pulsesPerRevolution>
+    </transmission>
     <xacro:proximal link_prefix="${link_prefix}" joint_prefix="${joint_prefix}" parent="${link_prefix}knuckle" >
     </xacro:proximal>

File: shadow_robot/sr_hand/model/hand_urdf/finger/middle/middle.urdf.xacro (robot description, xacro)
@@ -1,3 +1,4 @@
 <robot xmlns:xacro="http://ros.org/wiki/xacro">
+  <include filename="$(find sr_hand)/model/hand_urdf/finger/middle/middle.transmission.xacro" />
   <xacro:macro name="middle" params="link_prefix joint_prefix parent">
     <link name="${link_prefix}middle">
@@ -33,4 +34,5 @@
       velocity="1.0" />
     </joint>
+    <xacro:middle_transmission />
   </xacro:macro>
 </robot>

File: shadow_robot/sr_hand/model/hand_urdf/finger/proximal/proximal.urdf.xacro (robot description, xacro)
@@ -1,3 +1,4 @@
 <robot xmlns:xacro="http://ros.org/wiki/xacro">
+  <include filename="$(find sr_hand)/model/hand_urdf/finger/proximal/proximal.transmission.xacro" />
   <xacro:macro name="proximal" params="link_prefix joint_prefix parent">
     <link name="${link_prefix}proximal">
@@ -33,4 +34,5 @@
       velocity="1.0"/>
     </joint>
+    <xacro:proximal_transmission />
   </xacro:macro>
 </robot>

File: shadow_robot/sr_hand/model/hand_urdf/palm/palm.urdf.xacro (robot description, xacro)
@@ -1,3 +1,4 @@
 <robot xmlns:xacro="http://ros.org/wiki/xacro">
+  <include filename="$(find sr_hand)/model/hand_urdf/palm/palm.transmission.xacro" />
   <xacro:macro name="palm" params="parent">
     <link name="palm" >
@@ -33,4 +34,5 @@
       effort="10" velocity="1.0"/>
     </joint>
+    <xacro:shadowhand_palm_transmission />
   </xacro:macro>
 </robot>

File: shadow_robot/sr_hand/model/hand_urdf/thumb/thbase.urdf.xacro (robot description, xacro)
@@ -1,3 +1,4 @@
 <robot xmlns:xacro="http://ros.org/wiki/xacro">
+  <include filename="$(find sr_hand)/model/hand_urdf/thumb/thbase.transmission.xacro" />
   <xacro:macro name="thbase" params="parent">
     <link name="thbase">
@@ -35,4 +36,5 @@
       velocity="1.0" />
     </joint>
+    <xacro:thbase_transmission />
   </xacro:macro>
 </robot>

File: shadow_robot/sr_hand/model/hand_urdf/thumb/thdistal.urdf.xacro (robot description, xacro)
@@ -1,3 +1,4 @@
 <robot xmlns:xacro="http://ros.org/wiki/xacro">
+  <include filename="$(find sr_hand)/model/hand_urdf/thumb/thdistal.transmission.xacro" />
   <xacro:macro name="thdistal" params="parent">
     <link name="thdistal">
@@ -35,4 +36,5 @@
       velocity="1.0" />
     </joint>
+    <xacro:thdistal_transmission />
   </xacro:macro>
 </robot>

File: shadow_robot/sr_hand/model/hand_urdf/thumb/thhub.urdf.xacro (robot description, xacro)
@@ -1,3 +1,4 @@
 <robot xmlns:xacro="http://ros.org/wiki/xacro">
+  <include filename="$(find sr_hand)/model/hand_urdf/thumb/thhub.transmission.xacro" />
   <xacro:macro name="thhub" params="parent">
     <link name="thhub">
@@ -35,4 +36,5 @@
       velocity="1.0" />
     </joint>
+    <xacro:thhub_transmission />
   </xacro:macro>
 </robot>

File: shadow_robot/sr_hand/model/hand_urdf/thumb/thmiddle.urdf.xacro (robot description, xacro)
@@ -1,3 +1,4 @@
 <robot xmlns:xacro="http://ros.org/wiki/xacro">
+  <include filename="$(find sr_hand)/model/hand_urdf/thumb/thmiddle.transmission.xacro" />
   <xacro:macro name="thmiddle" params="parent">
     <link name="thmiddle">
@@ -35,4 +36,5 @@
       velocity="1.0" />
     </joint>
+    <xacro:thmiddle_transmission />
   </xacro:macro>
 </robot>

File: shadow_robot/sr_hand/model/hand_urdf/thumb/thproximal.urdf.xacro (robot description, xacro)
@@ -1,3 +1,4 @@
 <robot xmlns:xacro="http://ros.org/wiki/xacro">
+  <include filename="$(find sr_hand)/model/hand_urdf/thumb/thproximal.transmission.xacro" />
   <xacro:macro name="thproximal" params="parent">
     <link name="thproximal">
@@ -35,4 +36,5 @@
       velocity="1.0" />
     </joint>
+    <xacro:thproximal_transmission />
   </xacro:macro>
 </robot>

File: shadow_robot/sr_hand/model/hand_urdf/wrist/wrist.urdf.xacro (robot description, xacro)
@@ -1,3 +1,4 @@
 <robot xmlns:xacro="http://ros.org/wiki/xacro">
+  <include filename="$(find sr_hand)/model/hand_urdf/wrist/wrist.transmission.xacro" />
   <xacro:macro name="wrist" params="parent *origin">
     <link name="wrist" >
@@ -36,4 +37,5 @@
       effort="10" velocity="1.0"/>
     </joint>
+    <xacro:shadowhand_wrist_transmission />
   </xacro:macro>
 </robot>

File: shadow_robot/sr_hand/model/robots/arm_and_hand_motor.urdf (robot description, URDF)
Before this commit: robot arm_and_hand, 30 links, 29 joints
Links:
- added link world
Joints:
- added joint base_fix: type fixed, parent world, child shadowarm_base, origin xyz=0 0 0 rpy=0 0 0
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
Commit message: PID very approximately set for the arm, launchers created to launch every hand and / or arm in launch/gazebo

File: shadow_robot/sr_hand/model/arm_urdf/base/shadowarm_base.urdf.xacro (robot description, xacro)
@@ -6,5 +6,5 @@
     <inertial>
       <origin xyz="0 0 0" rpy="0 0 0"/>
-      <mass value="1000" />
+      <mass value="0.4" />
       <inertia  ixx="1.0" ixy="0.0"  ixz="0.0"  iyy="100.0"  iyz="0.0"  izz="1.0" />
     </inertial>

File: shadow_robot/sr_hand/model/arm_urdf/hand_support/shadowarm_handsupport_motor.urdf.xacro (robot description, xacro)
@@ -5,5 +5,5 @@
       <inertial>
 	<origin xyz="0 0 0" rpy="0 0 0" />
-	<mass value="1" />
+	<mass value="0.75" />
 	<inertia  ixx="1.0" ixy="0.0"  ixz="0.0"  iyy="100.0"  iyz="0.0"  izz="1.0" />
       </inertial>

File: shadow_robot/sr_hand/model/arm_urdf/hand_support/shadowarm_handsupport_muscle.urdf.xacro (robot description, xacro)
@@ -5,5 +5,5 @@
       <inertial>
 	<origin xyz="0 0 0" rpy="0 0 0" />
-	<mass value="1" />
+	<mass value="0.75" />
 	<inertia  ixx="1.0" ixy="0.0"  ixz="0.0"  iyy="100.0"  iyz="0.0"  izz="1.0" />
       </inertial>

File: shadow_robot/sr_hand/model/arm_urdf/lower_arm/shadowarm_lowerarm.urdf.xacro (robot description, xacro)
@@ -5,5 +5,5 @@
 	<inertial>
 	  <origin xyz="0.0655 0 -0.08" rpy="0 0 0" />
-	  <mass value="5" />
+	  <mass value="1.7" />
 	  <inertia  ixx="1.0" ixy="0.0"  ixz="0.0"  iyy="100.0"  iyz="0.0"  izz="1.0" />
 	</inertial>

File: shadow_robot/sr_hand/model/arm_urdf/upper_arm/shadowarm_upperarm.urdf.xacro (robot description, xacro)
@@ -5,5 +5,5 @@
       <inertial>
 	<origin xyz="0.1845 -0.067 0" rpy="0 0 0" />
-	<mass value="5" />
+	<mass value="2" />
 	<inertia  ixx="1.0" ixy="0.0"  ixz="0.0"  iyy="100.0"  iyz="0.0"  izz="1.0" />
       </inertial>

File: shadow_robot/sr_hand/model/robots/arm_and_hand_motor.urdf (robot description, URDF)
Before this commit: robot arm_and_hand, 31 links, 30 joints
Links:
- link shadowarm_base: mass 1000 -> 0.4
- link shadowarm_handsupport_motor: mass 1 -> 0.75
- link shadowarm_lowerarm: mass 5 -> 1.7
- link shadowarm_upperarm: mass 5 -> 2

File: shadow_robot/sr_hand/model/robots/arm_and_hand_muscle.urdf (robot description, URDF)
Before this commit: robot arm_and_hand, 31 links, 30 joints
Links:
- link shadowarm_base: mass 1000 -> 0.4
- link shadowarm_handsupport_muscle: mass 1 -> 0.75
- link shadowarm_lowerarm: mass 5 -> 1.7
- link shadowarm_upperarm: mass 5 -> 2
Joints:
- joint arm_link: origin xyz=0 0 0 rpy=0 0 0 -> xyz=0 0 0 rpy=1.57079632679 0 1.57079632679

File: shadow_robot/sr_hand/model/robots/sr_arm_motor.urdf (robot description, URDF)
Before this commit: robot sr_arm_motor, 6 links, 5 joints
Links:
- link shadowarm_base: mass 1000 -> 0.4
- link shadowarm_handsupport_motor: mass 1 -> 0.75
- link shadowarm_lowerarm: mass 5 -> 1.7
- link shadowarm_upperarm: mass 5 -> 2

File: shadow_robot/sr_hand/model/robots/sr_arm_muscle.urdf (robot description, URDF)
Before this commit: robot sr_arm_muscle, 6 links, 5 joints
Links:
- link shadowarm_base: mass 1000 -> 0.4
- link shadowarm_handsupport_muscle: mass 1 -> 0.75
- link shadowarm_lowerarm: mass 5 -> 1.7
- link shadowarm_upperarm: mass 5 -> 2

File: shadow_robot/sr_hand/model/robots/xacro/arm_and_hand_muscle.urdf.xacro (robot description, xacro)
@@ -9,5 +9,5 @@
     <parent link="shadowarm_handsupport_muscle"/>
     <child link="forearm_muscle"/>
-    <origin xyz="0 0 0" rpy="0 0 0" />
+    <origin xyz="0 0 0" rpy="${M_PI/2} 0 ${M_PI/2}" />
     <axis xyz="0 -1 0" />
     <limit lower="0" upper="0" effort="10"
