Commit message: The model is now a lot easier to control. It still needs to be refined.

File: shadow_robot/sr_hand/model/arm_urdf/base/shadowarm_base.urdf.xacro (robot description, xacro)
@@ -7,5 +7,5 @@
       <origin xyz="0 0 0" rpy="0 0 0"/>
       <mass value="0.4" />
-      <inertia  ixx="1.0" ixy="0.0"  ixz="0.0"  iyy="100.0"  iyz="0.0"  izz="1.0" />
+      <inertia  ixx="1.0" ixy="0.0"  ixz="0.0"  iyy="0.0"  iyz="0.0"  izz="0.0" />
     </inertial>
     <visual>

File: shadow_robot/sr_hand/model/arm_urdf/hand_support/shadowarm_handsupport_motor.urdf.xacro (robot description, xacro)
@@ -6,5 +6,5 @@
 	<origin xyz="0 0 0" rpy="0 0 0" />
 	<mass value="0.75" />
-	<inertia  ixx="1.0" ixy="0.0"  ixz="0.0"  iyy="100.0"  iyz="0.0"  izz="1.0" />
+	<inertia  ixx="1.0" ixy="0.0"  ixz="0.0"  iyy="0.0"  iyz="0.0"  izz="0.0" />
       </inertial>
       <visual>
@@ -33,5 +33,5 @@
       <limit lower="-${M_PI/2}" upper="${M_PI/2}"
       effort="10" velocity="1.0"/>
-      <dynamics damping="3.5"/>
+      <dynamics damping="10.5"/>
     </joint>
     <xacro:shadowarm_handsupport_motor_transmission />

File: shadow_robot/sr_hand/model/arm_urdf/hand_support/shadowarm_handsupport_muscle.urdf.xacro (robot description, xacro)
@@ -6,5 +6,5 @@
 	<origin xyz="0 0 0" rpy="0 0 0" />
 	<mass value="0.75" />
-	<inertia  ixx="1.0" ixy="0.0"  ixz="0.0"  iyy="100.0"  iyz="0.0"  izz="1.0" />
+	<inertia  ixx="1.0" ixy="0.0"  ixz="0.0"  iyy="0.0"  iyz="0.0"  izz="0.0" />
       </inertial>
       <visual>
@@ -33,5 +33,5 @@
       <limit lower="-${M_PI/2}" upper="${M_PI/2}"
       effort="10" velocity="1.0"/>
-      <dynamics damping="3.5"/>
+      <dynamics damping="10.5"/>
     </joint>
     <xacro:shadowarm_handsupport_muscle_transmission />

File: shadow_robot/sr_hand/model/arm_urdf/lower_arm/shadowarm_lowerarm.urdf.xacro (robot description, xacro)
@@ -6,5 +6,5 @@
 	  <origin xyz="0.0655 0 -0.08" rpy="0 0 0" />
 	  <mass value="1.7" />
-	  <inertia  ixx="1.0" ixy="0.0"  ixz="0.0"  iyy="100.0"  iyz="0.0"  izz="1.0" />
+	  <inertia  ixx="1.0" ixy="0.0"  ixz="0.0"  iyy="0.0"  iyz="0.0"  izz="0.0" />
 	</inertial>
 	<visual>
@@ -33,5 +33,5 @@
       <limit lower="0" upper="2.09439510239"
       effort="10" velocity="1.0"/>
-      <dynamics damping="3.5"/>
+      <dynamics damping="50.5"/>
     </joint>
     <xacro:shadowarm_lowerarm_transmission />

File: shadow_robot/sr_hand/model/arm_urdf/trunk/shadowarm_trunk.urdf.xacro (robot description, xacro)
@@ -6,5 +6,5 @@
 	  <origin xyz="0 0 0.27025" rpy="0 0 0" />
 	  <mass value="5" />
-	  <inertia  ixx="1.0" ixy="0.0"  ixz="0.0"  iyy="100.0"  iyz="0.0"  izz="1.0" />
+	  <inertia  ixx="1.0" ixy="0.0"  ixz="0.0"  iyy="0.0"  iyz="0.0"  izz="0.0" />
 	</inertial>
 	<visual>
@@ -33,5 +33,5 @@
       <limit lower="-${M_PI/2}" upper="${M_PI/4}"
       effort="10" velocity="1.0"/>
-      <dynamics damping="3.5"/>
+      <dynamics damping="200.5"/>
     </joint>
     <xacro:shadowarm_trunk_transmission />

File: shadow_robot/sr_hand/model/arm_urdf/upper_arm/shadowarm_upperarm.urdf.xacro (robot description, xacro)
@@ -6,5 +6,5 @@
 	<origin xyz="0.1845 -0.067 0" rpy="0 0 0" />
 	<mass value="2" />
-	<inertia  ixx="1.0" ixy="0.0"  ixz="0.0"  iyy="100.0"  iyz="0.0"  izz="1.0" />
+	<inertia  ixx="1.0" ixy="0.0"  ixz="0.0"  iyy="0.0"  iyz="0.0"  izz="0.0" />
       </inertial>
       <visual>
@@ -32,5 +32,5 @@
       <axis xyz="0 1 0" />
       <limit lower="0" upper="${M_PI/2}" effort="10" velocity="1.0"/>
-      <dynamics damping="3.5"/>
+      <dynamics damping="50.5"/>
     </joint>
     <xacro:shadowarm_upperarm_transmission />

File: shadow_robot/sr_hand/model/hand_urdf/finger/distal/distal.urdf.xacro (robot description, xacro)
@@ -6,6 +6,6 @@
 	<mass value="0.010" />
 	<origin xyz="0 0 0.025" />
-	<inertia  ixx="1.0" ixy="0.0"  ixz="0.0"  iyy="100.0"  iyz="0.0"
-	izz="1.0" />
+	<inertia  ixx="1.0" ixy="0.0"  ixz="0.0"  iyy="0.0"  iyz="0.0"
+	izz="0.0" />
       </inertial>
       <visual>
@@ -33,5 +33,5 @@
       <limit lower="0" upper="${M_PI/2}" effort="10"
       velocity="1.0" />
-      <dynamics damping="3.5"/>
+      <dynamics damping="50.5"/>
     </joint>
     <xacro:distal_transmission />

File: shadow_robot/sr_hand/model/hand_urdf/finger/knuckle/knuckle.urdf.xacro (robot description, xacro)
@@ -7,6 +7,6 @@
 	<insert_block name="origin" />
 	<mass value="0.008" />
-	<inertia  ixx="1.0" ixy="0.0"  ixz="0.0"  iyy="100.0"  iyz="0.0"
-	izz="1.0" />
+	<inertia  ixx="1.0" ixy="0.0"  ixz="0.0"  iyy="0.0"  iyz="0.0"
+	izz="0.0" />
       </inertial>
       <visual>
@@ -35,5 +35,5 @@
       <limit lower="-0.43633231299858238" upper="0.43633231299858238"
       effort="10" velocity="1.0"/>
-      <dynamics damping="3.5"/>
+      <dynamics damping="50.5"/>
     </joint>
     <xacro:knuckle_transmission />

File: shadow_robot/sr_hand/model/hand_urdf/finger/lfmetacarpal/lfmetacarpal.urdf.xacro (robot description, xacro)
@@ -6,6 +6,6 @@
 	<origin xyz="0.00568 0 -0.12061" rpy="0 0 0" />
 	<mass value="0.075" />
-	<inertia  ixx="1.0" ixy="0.0"  ixz="0.0"  iyy="100.0"  iyz="0.0"
-	izz="1.0" />
+	<inertia  ixx="1.0" ixy="0.0"  ixz="0.0"  iyy="0.0"  iyz="0.0"
+	izz="0.0" />
       </inertial>
       <visual>
@@ -33,5 +33,5 @@
       <limit lower="0" upper="0.69813170079773179" effort="10"
       velocity="1.0" />
-      <dynamics damping="3.5"/>
+      <dynamics damping="50.5"/>
     </joint>
     <xacro:lfmetacarpal_transmission />

File: shadow_robot/sr_hand/model/hand_urdf/finger/little_finger.urdf.xacro (robot description, xacro)
@@ -12,6 +12,6 @@
 	<origin xyz="0 0 0.0425" rpy="0 0 0" />
 	<mass value="0.008" />
-	<inertia  ixx="1.0" ixy="0.0"  ixz="0.0"  iyy="100.0"  iyz="0.0"
-	izz="1.0" />
+	<inertia  ixx="1.0" ixy="0.0"  ixz="0.0"  iyy="0.0"  iyz="0.0"
+	izz="0.0" />
       </inertial>
       <visual>
@@ -39,5 +39,5 @@
       <limit lower="-0.43633231299858238" upper="0.43633231299858238"
       effort="10" velocity="1.0"/>
-      <dynamics damping="3.5"/>
+      <dynamics damping="50.5"/>
     </joint>
     <transmission type="pr2_mechanism_model/SimpleTransmission" name="lfknuckle_transmission">

File: shadow_robot/sr_hand/model/hand_urdf/finger/middle/middle.urdf.xacro (robot description, xacro)
@@ -6,6 +6,6 @@
 	<origin xyz="0 0 0.045" rpy="0 0 0" />
 	<mass value="0.012" />
-	<inertia  ixx="1.0" ixy="0.0"  ixz="0.0"  iyy="100.0"  iyz="0.0"
-	izz="1.0" />
+	<inertia  ixx="1.0" ixy="0.0"  ixz="0.0"  iyy="0.0"  iyz="0.0"
+	izz="0.0" />
       </inertial>
       <visual>
@@ -33,5 +33,5 @@
       <limit lower="0" upper="${M_PI/2}" effort="10"
       velocity="1.0" />
-      <dynamics damping="3.5"/>
+      <dynamics damping="50.5"/>
     </joint>
     <xacro:middle_transmission />

File: shadow_robot/sr_hand/model/hand_urdf/finger/proximal/proximal.urdf.xacro (robot description, xacro)
@@ -6,6 +6,6 @@
 	<mass value="0.014" />
 	<origin xyz="0 0 0" />
-	<inertia  ixx="1.0" ixy="0.0"  ixz="0.0"  iyy="100.0"  iyz="0.0"
-	izz="1.0" />
+	<inertia  ixx="1.0" ixy="0.0"  ixz="0.0"  iyy="0.0"  iyz="0.0"
+	izz="0.0" />
       </inertial>
       <visual>
@@ -33,5 +33,5 @@
       <limit lower="0" upper="${M_PI/2}" effort="10"
       velocity="1.0"/>
-      <dynamics damping="3.5"/>
+      <dynamics damping="50.5"/>
     </joint>
     <xacro:proximal_transmission />

File: shadow_robot/sr_hand/model/hand_urdf/forearm/forearm_motor.urdf.xacro (robot description, xacro)
@@ -6,5 +6,5 @@
 	<origin xyz="0 0 0" />
 	<mass value="3.0" />
-	<inertia  ixx="1.0" ixy="0.0"  ixz="0.0"  iyy="100.0"  iyz="0.0"  izz="1.0" />
+	<inertia  ixx="1.0" ixy="0.0"  ixz="0.0"  iyy="0.0"  iyz="0.0"  izz="0.0" />
       </inertial>
       <visual>

File: shadow_robot/sr_hand/model/hand_urdf/forearm/forearm_muscle.urdf.xacro (robot description, xacro)
@@ -6,5 +6,5 @@
 	<origin xyz="0 0 0" />
 	<mass value="3.0" />
-	<inertia  ixx="1.0" ixy="0.0"  ixz="0.0"  iyy="100.0"  iyz="0.0"  izz="1.0" />
+	<inertia  ixx="1.0" ixy="0.0"  ixz="0.0"  iyy="0.0"  iyz="0.0"  izz="0.0" />
       </inertial>
       <visual>

File: shadow_robot/sr_hand/model/hand_urdf/palm/palm.urdf.xacro (robot description, xacro)
@@ -6,6 +6,6 @@
 	<origin xyz="0 0.010 0.247" rpy="0 0 0" />
 	<mass value="0.3" />
-	<inertia  ixx="1.0" ixy="0.0"  ixz="0.0"  iyy="100.0"  iyz="0.0"
-	izz="1.0" />
+	<inertia  ixx="1.0" ixy="0.0"  ixz="0.0"  iyy="0.0"  iyz="0.0"
+	izz="0.0" />
       </inertial>
       <visual>
@@ -33,5 +33,5 @@
       <limit lower="-0.78539816339744828" upper="0.6108652381980153"
       effort="10" velocity="1.0"/>
-      <dynamics damping="3.5"/>
+      <dynamics damping="50.5"/>
     </joint>
     <xacro:shadowhand_palm_transmission />

File: shadow_robot/sr_hand/model/hand_urdf/thumb/thbase.urdf.xacro (robot description, xacro)
@@ -6,6 +6,6 @@
 	<mass value="0.010" />
 	<origin xyz="0.034 0.0085 0.02924" rpy="0 0 0"/>
-	<inertia  ixx="1.0" ixy="0.0"  ixz="0.0"  iyy="100.0"  iyz="0.0"
-	izz="1.0" />
+	<inertia  ixx="1.0" ixy="0.0"  ixz="0.0"  iyy="0.0"  iyz="0.0"
+	izz="0.0" />
       </inertial>
       <visual>
@@ -35,5 +35,5 @@
       <limit lower="-1.047" upper="1.047" effort="10"
       velocity="1.0" />
-      <dynamics damping="3.5"/>
+      <dynamics damping="50.5"/>
     </joint>
     <xacro:thbase_transmission />

File: shadow_robot/sr_hand/model/hand_urdf/thumb/thdistal.urdf.xacro (robot description, xacro)
@@ -6,6 +6,6 @@
 	<mass value="0.016" />
 	<origin xyz="-0.02263 0 0.02263" rpy="0 0 0"/>
-	<inertia  ixx="1.0" ixy="0.0"  ixz="0.0"  iyy="100.0"  iyz="0.0"
-	izz="1.0" />
+	<inertia  ixx="1.0" ixy="0.0"  ixz="0.0"  iyy="0.0"  iyz="0.0"
+	izz="0.0" />
       </inertial>
       <visual>
@@ -35,5 +35,5 @@
       <limit lower="0" upper="1.571" effort="10"
       velocity="1.0" />
-      <dynamics damping="3.5"/>
+      <dynamics damping="50.5"/>
     </joint>
     <xacro:thdistal_transmission />

File: shadow_robot/sr_hand/model/hand_urdf/thumb/thhub.urdf.xacro (robot description, xacro)
@@ -6,6 +6,6 @@
 	<mass value="0.002" />
 	<origin xyz="0.02687 0 0.02687" rpy="0 0 0"/>
-	<inertia  ixx="1.0" ixy="0.0"  ixz="0.0"  iyy="100.0"  iyz="0.0"
-	izz="1.0" />
+	<inertia  ixx="1.0" ixy="0.0"  ixz="0.0"  iyy="0.0"  iyz="0.0"
+	izz="0.0" />
       </inertial>
       <visual>
@@ -35,5 +35,5 @@
       <limit lower="-0.2618" upper="0.2618" effort="10"
       velocity="1.0" />
-      <dynamics damping="3.5"/>
+      <dynamics damping="50.5"/>
     </joint>
     <xacro:thhub_transmission />

File: shadow_robot/sr_hand/model/hand_urdf/thumb/thmiddle.urdf.xacro (robot description, xacro)
@@ -6,6 +6,6 @@
 	<mass value="0.016" />
 	<origin xyz="0 0 0" rpy="0 0 0"/>
-	<inertia  ixx="1.0" ixy="0.0"  ixz="0.0"  iyy="100.0"  iyz="0.0"
-	izz="1.0" />
+	<inertia  ixx="1.0" ixy="0.0"  ixz="0.0"  iyy="0.0"  iyz="0.0"
+	izz="0.0" />
       </inertial>
       <visual>
@@ -35,5 +35,5 @@
       <limit lower="-0.5237" upper="0.5237" effort="10"
       velocity="1.0" />
-      <dynamics damping="3.5"/>
+      <dynamics damping="50.5"/>
     </joint>
     <xacro:thmiddle_transmission />

File: shadow_robot/sr_hand/model/hand_urdf/thumb/thproximal.urdf.xacro (robot description, xacro)
@@ -6,6 +6,6 @@
 	<mass value="0.016" />
 	<origin xyz="0 0 0" rpy="0 0 0"/>
-	<inertia  ixx="1.0" ixy="0.0"  ixz="0.0"  iyy="100.0"  iyz="0.0"
-	izz="1.0" />
+	<inertia  ixx="1.0" ixy="0.0"  ixz="0.0"  iyy="0.0"  iyz="0.0"
+	izz="0.0" />
       </inertial>
       <visual>
@@ -35,5 +35,5 @@
       <limit lower="0" upper="1.309" effort="10"
       velocity="1.0" />
-      <dynamics damping="3.5"/>
+      <dynamics damping="50.5"/>
     </joint>
     <xacro:thproximal_transmission />
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
Commit message: Ok, desk is now added cleanly through a xacro frile for the motor and muscle arms.

File: shadow_robot/sr_hand/model/arm_urdf/base/shadowarm_base.urdf.xacro (robot description, xacro)
@@ -2,5 +2,4 @@
 <property name="M_PI" value="3.1415926535897931" />
 <xacro:macro name="shadowarm_base">
-  <link name="world" />
   <link name="shadowarm_base">
     <inertial>
@@ -27,9 +26,4 @@
     <selfCollide>true</selfCollide>
   </gazebo>
-  <joint name="base_fix" type="fixed">
-    <parent link="world"/>
-    <child link="shadowarm_base"/>
-    <origin rpy="0 0 0" xyz="0 0 0"/>
-  </joint>
 </xacro:macro>
 </robot>

File: shadow_robot/sr_hand/model/robots/arm_and_hand_motor.urdf (robot description, URDF)
Before this commit: robot arm_and_hand, 32 links, 31 joints
Joints:
- joint arm_link: origin xyz=0 0 0 rpy=0 0 1.57079632679 -> xyz=0 0 0 rpy=0 0 3.14159265359

File: shadow_robot/sr_hand/model/robots/arm_and_hand_muscle.urdf (robot description, URDF)
Before this commit: robot arm_and_hand, 31 links, 30 joints
Links:
- removed link world
- added link desk_pillar, mass 100.0; collision cylinder length=1.0 radius=0.1; visual cylinder length=1.0 radius=0.1
- added link desk_support, mass 1000.0; collision cylinder length=0.02 radius=1.0; visual cylinder length=0.02 radius=1.0
Joints:
- added joint desk_joint: type fixed, parent desk_support, child desk_pillar, origin xyz=0 0 0.01 rpy=0 0 0
- joint arm_link: origin xyz=0 0 0 rpy=0 0 1.57079632679 -> xyz=0 0 0 rpy=0 0 3.14159265359
- joint base_fix: origin xyz=0 0 0 rpy=0 0 0 -> xyz=0 0 1.0 rpy=0 0 0; parent world -> desk_pillar

File: shadow_robot/sr_hand/model/robots/sr_arm_motor.urdf (robot description, URDF)
Before this commit: robot sr_arm_motor, 6 links, 5 joints
Links:
- removed link world
Joints:
- removed joint base_fix

File: shadow_robot/sr_hand/model/robots/sr_arm_muscle.urdf (robot description, URDF)
Before this commit: robot sr_arm_muscle, 6 links, 5 joints
Links:
- removed link world
Joints:
- removed joint base_fix

File: shadow_robot/sr_hand/model/robots/xacro/arm_and_hand_motor.urdf.xacro (robot description, xacro)
@@ -16,5 +16,5 @@
     <parent link="shadowarm_handsupport_motor"/>
     <child link="forearm_motor"/>
-    <origin xyz="0 0 0" rpy="0 0 ${M_PI/2}" />
+    <origin xyz="0 0 0" rpy="0 0 ${M_PI}" />
     <axis xyz="0 -1 0" />
     <limit lower="0" upper="0" effort="10"

File: shadow_robot/sr_hand/model/robots/xacro/arm_and_hand_muscle.urdf.xacro (robot description, xacro)
@@ -4,4 +4,11 @@
   <include filename="$(find sr_hand)/model/hand_urdf/full_hand_muscle.urdf.xacro" />
   <include filename="$(find sr_hand)/model/gazebo/gazebo.urdf.xacro" />
+  <include filename="$(find sr_hand)/model/desk/desk.urdf.xacro" />
+  <xacro:desk/>
+  <joint name="base_fix" type="fixed">
+    <parent link="desk_pillar"/>
+    <child link="shadowarm_base"/>
+    <origin rpy="0 0 0" xyz="0 0 1.0"/>
+  </joint>
   <xacro:sr_arm_muscle>
   </xacro:sr_arm_muscle>
@@ -9,5 +16,5 @@
     <parent link="shadowarm_handsupport_muscle"/>
     <child link="forearm_muscle"/>
-    <origin xyz="0 0 0" rpy="0 0 ${M_PI/2}" />
+    <origin xyz="0 0 0" rpy="0 0 ${M_PI}" />
     <axis xyz="0 -1 0" />
     <limit lower="0" upper="0" effort="10"
