Commit message: Changed the model to contain only 4 joints wrj1/2 and ffj3/4. Added actuators to the hardware interface. The joint_states are now being published.

File: shadow_robot/sr_hand_palm_edc/sr_edc_defs/robots/sr_edc.urdf.xacro (robot description, xacro)
@@ -1,17 +1,76 @@
 <?xml version="1.0"?>
 <robot name="SRH">
+  <!-- FIXME: all the limits are not valid -->
+  <property name="wrj1_joint_effort_limit"  value="100.0" />
+  <property name="wrj2_joint_effort_limit"  value="100.0" />
+  <property name="wrj1_upper_angle" value="0.611" />
+  <property name="wrj1_lower_angle" value="-0.786" />
+  <property name="wrj2_upper_angle" value="0.175" />
+  <property name="wrj2_lower_angle" value="-0.524" />
+  <macro name="pr2_wrist1_limits" params="reflect">
+    <limit effort="${wrj1_joint_effort_limit}" velocity="0.5"
+           lower="${wrj1_lower_angle}" upper="${wrj1_upper_angle}" />
+  </macro>
+  <macro name="pr2_wrist2_limits" params="reflect">
+    <limit effort="${wrj2_joint_effort_limit}" velocity="0.5"
+           lower="${wrj2_lower_angle}" upper="${wrj2_upper_angle}" />
+  </macro>
+  <!-- FIXME: all the limits are not valid -->
+  <property name="fj3_joint_effort_limit"  value="100.0" />
+  <property name="fj4_joint_effort_limit"  value="100.0" />
+  <property name="fj3_upper_angle" value="1.571" />
+  <property name="fj3_lower_angle" value="0.00" />
+  <property name="fj4_upper_angle" value="0.436" />
+  <property name="fj4_lower_angle" value="-0.436" />
+  <macro name="pr2_ff3_limits" params="reflect">
+    <limit effort="${fj3_joint_effort_limit}" velocity="1.0"
+           lower="${fj3_lower_angle}" upper="${fj3_upper_angle}" />
+  </macro>
+  <macro name="pr2_ff4_limits" params="reflect">
+    <limit effort="${fj4_joint_effort_limit}" velocity="1.0"
+           lower="${fj4_lower_angle}" upper="${fj4_upper_angle}" />
+  </macro>
+  <include filename="$(find sr_edc_defs)/defs/hand/hand_transmission.xacro" />
+  <property name="M_PI" value="3.1415926535897931" />
   <link name="world"/>
-  <include filename="$(find sr_edc_defs)/defs/hand/hand_defs.urdf.xacro" />
-  <pr2_sr_edc_hand name="shadow_hand" side="r" parent="world"
-               screw_reduction="${2.0/1000.0}" gear_ratio="${29.16}"
-               theta0="${2.97571*M_PI/180.0}"
-               phi0="${29.98717*M_PI/180.0}"
-               t0="${-0.19543/1000.0}"
-               L0="${34.70821/1000.0}"
-               h="${5.200/1000.0}"
-               a="${67.56801/1000.0}"
-               b="${48.97193/1000.0}"
-               r="${91.50000/1000.0}" >
-    <origin xyz="0 0 0" rpy="0 0 0" />
-  </pr2_sr_edc_hand>
+    <joint name="srh_wrj2_joint" type="revolute">
+      <parent link="world"/>
+      <child link="sr_wrist_dummy_link" />
+      <origin xyz="0 0 0" rpy="0 0 0" />
+      <axis xyz="0 1 0" />
+      <pr2_wrist2_limits reflect="1" />
+    </joint>
+    <link name="sr_wrist_dummy_link">
+    </link>
+    <joint name="srh_wrj1_joint" type="revolute">
+      <parent link="sr_wrist_dummy_link"/>
+      <child link="sr_hand_palm_link"/>
+      <origin xyz="0 0 0.034" rpy="0 0 0" />
+      <axis xyz="1 0 0" />
+      <pr2_wrist1_limits reflect="1" />
+    </joint>
+    <link name="sr_hand_palm_link">
+    </link>
+    <!-- ........................................ -->
+    <joint name="srh_ffj4_joint" type="revolute">
+      <parent link="sr_hand_palm_link"/>
+      <child link="sr_hand_ff4_link"/>
+      <origin xyz="0.033 0 0.095" rpy="0 0 0" />
+      <axis xyz="0 -1 0" />
+      <pr2_ff4_limits reflect="1" />
+    </joint>
+    <link name="sr_hand_ff4_link">
+    </link>
+    <joint name="srh_ffj3_joint" type="revolute">
+      <parent link="sr_hand_ff4_link"/>
+      <child link="sr_hand_ff3_link"/>
+      <origin xyz="0 0 0" rpy="0 0 0" />
+      <axis xyz="1 0 0" />
+      <pr2_ff3_limits reflect="1" />
+    </joint>
+    <link name="sr_hand_ff3_link">
+    </link>
+    <!-- ........................................ -->
+    <sr_hand_wrist_transmission joint_name="wr" />
+    <sr_hand_finger_transmission joint_name="ff" />
 </robot>
