Commit message: the data are being published to the joint_states topic.

File: shadow_robot/sr_hand_palm_edc/sr_edc_defs/robots/sr_edc.urdf (robot description, URDF)
Before this commit: robot SRH, 5 links, 4 joints
Joints:
- removed joint srh_ffj3_joint
- removed joint srh_ffj4_joint
- removed joint srh_wrj1_joint
- removed joint srh_wrj2_joint
- added joint FFJ3_joint: type revolute, parent sr_hand_ff4_link, child sr_hand_ff3_link, origin xyz=0 0 0 rpy=0 0 0, axis 1 0 0, limit lower=0.0 upper=1.571 effort=100.0 velocity=1.0
- added joint FFJ4_joint: type revolute, parent sr_hand_palm_link, child sr_hand_ff4_link, origin xyz=0.033 0 0.095 rpy=0 0 0, axis 0 -1 0, limit lower=-0.436 upper=0.436 effort=100.0 velocity=1.0
- added joint WRJ1_joint: type revolute, parent sr_wrist_dummy_link, child sr_hand_palm_link, origin xyz=0 0 0.034 rpy=0 0 0, axis 1 0 0, limit lower=-0.786 upper=0.611 effort=100.0 velocity=0.5
- added joint WRJ2_joint: type revolute, parent world, child sr_wrist_dummy_link, origin xyz=0 0 0 rpy=0 0 0, axis 0 1 0, limit lower=-0.524 upper=0.175 effort=100.0 velocity=0.5
