Commit message: lp:798679 adding a special transmission for the joint 0s. I didn't manage to get it to be loaded, for the time beingm, the cpp / hpp files have to be manually copied to pr2_mechanism_model + the CMakeLists.txt and transmissions_plugin.xml file need to be modified in pr2_mechanism_model.

File: shadow_robot/sr_hand/model/hand_urdf/finger/middle/middle.transmission.xacro (robot description, xacro)
@@ -5,7 +5,8 @@
        xmlns:xacro="http://ros.org/wiki/xacro">
   <xacro:macro name="middle_transmission">
-    <transmission type="pr2_mechanism_model/SimpleTransmission" name="${link_prefix}middle_transmission">
+    <transmission type="sr_mechanism_model/J0Transmission" name="${link_prefix}middle_transmission">
       <actuator name="${joint_prefix}J0" />
-      <joint name="${joint_prefix}J2" />
+      <joint1 name="${joint_prefix}J1" />
+      <joint2 name="${joint_prefix}J2" />
       <mechanicalReduction>1</mechanicalReduction>
       <motorTorqueConstant>1</motorTorqueConstant>
