Commit message: temporary fix for J4s

File: shadow_robot/sr_hand/model/robots/arm_and_hand_motor.urdf (robot description, URDF)
Before this commit: robot arm_and_hand, 31 links, 30 joints
Joints:
- joint LFJ4: axis 0 -1 0 -> 0 1 0
- joint RFJ4: axis 0 -1 0 -> 0 1 0

File: shadow_robot/sr_hand/model/robots/shadowhand_motor.urdf (robot description, URDF)
Before this commit: robot shadowhand_motor, 25 links, 24 joints
Joints:
- joint LFJ4: axis 0 -1 0 -> 0 1 0
- joint RFJ4: axis 0 -1 0 -> 0 1 0

Commit message: starting hand + arm. Also beginning to add the SimpleActionServer for the pickup: when the object is double_clicked in the GUI, a pickup_goal is sent to the Pickup Server (which doesn't have the correct parameters yet).

File: shadow_robot/sr_hand/model/robots/arm_and_hand_motor.urdf (robot description, URDF)
Before this commit: robot arm_and_hand, 31 links, 30 joints
Links:
- removed link world
- added link base_link
Joints:
- joint base_fix: parent world -> base_link

File: shadow_robot/sr_hand/model/robots/sr_arm_motor.urdf (robot description, URDF)
Before this commit: robot sr_arm_motor, 6 links, 5 joints
Links:
- removed link world
- added link base_link
Joints:
- joint base_fix: parent world -> base_link

Commit message: publishing the aggregated tf with a new timestamp + removed the double definition of base_link

File: shadow_robot/sr_hand/model/robots/arm_and_hand_motor.urdf (robot description, URDF)
Before this commit: robot arm_and_hand, 31 links, 30 joints
Links:
- removed link base_link
Joints:
- removed joint base_fix

Commit message: minor model fixes

File: shadow_robot/sr_hand/model/robots/arm_and_hand_motor.urdf (robot description, URDF)
Before this commit: robot arm_and_hand, 31 links, 30 joints
Joints:
- joint arm_link: origin xyz=0 0 0 rpy=1.57079632679 0 1.57079632679 -> xyz=0 0 0 rpy=0 0 1.57079632679

File: shadow_robot/sr_hand/model/robots/arm_and_hand_muscle.urdf (robot description, URDF)
Before this commit: robot arm_and_hand, 31 links, 30 joints
Joints:
- joint arm_link: origin xyz=0 0 0 rpy=1.57079632679 0 1.57079632679 -> xyz=0 0 0 rpy=0 0 1.57079632679

Commit message: Trying to solve the gazebo starting position problem: attaching the arm to a desk. Needs cleaning

File: shadow_robot/sr_hand/model/robots/arm_and_hand_motor.urdf (robot description, URDF)
Before this commit: robot arm_and_hand, 31 links, 30 joints
Links:
- removed link world
- added link desk_pillar, mass 100.0; collision cylinder length=1.0 radius=0.1; visual cylinder length=1.0 radius=0.1
- added link desk_support, mass 1000.0; collision cylinder length=0.02 radius=1.0; visual cylinder length=0.02 radius=1.0
Joints:
- added joint desk_joint: type fixed, parent desk_support, child desk_pillar, origin xyz=0 0 0.01 rpy=0 0 0
- joint base_fix: origin xyz=0 0 0 rpy=0 0 0 -> xyz=0 0 1.0 rpy=0 0 0; parent world -> desk_pillar

Commit message: working again: had to modify a bit to adjust to the ROS changes. It's now working for ROS diamonback with only the openni_camera for the kinect as an overlay.

File: shadow_robot/sr_hand/model/robots/arm_and_hand_motor.urdf (robot description, URDF)
Before this commit: robot arm_and_hand, 32 links, 31 joints
Links:
- removed link desk_pillar
- removed link desk_support
Joints:
- removed joint base_fix
- removed joint desk_joint

File: shadow_robot/sr_hand/model/robots/arm_and_hand_muscle.urdf (robot description, URDF)
Before this commit: robot arm_and_hand, 32 links, 31 joints
Links:
- removed link desk_pillar
- removed link desk_support
Joints:
- removed joint base_fix
- removed joint desk_joint

File: shadow_robot/sr_hand/model/robots/xacro/arm_and_hand_muscle.urdf.xacro (robot description, xacro)
@@ -4,11 +4,4 @@
   <include filename="$(find sr_hand)/model/hand_urdf/full_hand_muscle.urdf.xacro" />
   <include filename="$(find sr_hand)/model/gazebo/gazebo.urdf.xacro" />
-  <include filename="$(find sr_hand)/model/desk/desk.urdf.xacro" />
-  <xacro:desk/>
-  <joint name="base_fix" type="fixed">
-    <parent link="desk_pillar"/>
-    <child link="shadowarm_base"/>
-    <origin rpy="0 0 0" xyz="0 0 1.0"/>
-  </joint>
   <xacro:sr_arm_muscle>
   </xacro:sr_arm_muscle>

File: shadow_robot/sr_hand/model/robots/xacro/desk_arm_and_hand_motor.urdf.xacro (robot description, xacro)
@@ -4,4 +4,11 @@
   <include filename="$(find sr_hand)/model/hand_urdf/full_hand_motor.urdf.xacro" />
   <include filename="$(find sr_hand)/model/gazebo/gazebo.urdf.xacro" />
+  <include filename="$(find sr_hand)/model/desk/desk.urdf.xacro" />
+  <xacro:desk/>
+  <joint name="base_fix" type="fixed">
+    <parent link="desk_pillar"/>
+    <child link="shadowarm_base"/>
+    <origin rpy="0 0 0" xyz="0 0 1.0"/>
+  </joint>
   <xacro:sr_arm_motor>
   </xacro:sr_arm_motor>

Commit message: Turned the hand from pi/4 to be able to grasp from top.

File: shadow_robot/sr_hand/model/robots/arm_and_hand_motor.urdf (robot description, URDF)
Before this commit: robot arm_and_hand, 30 links, 29 joints
Joints:
- joint arm_link: origin xyz=0 0 0 rpy=0 0 3.14159265359 -> xyz=0 0 0 rpy=0 0 2.36

File: shadow_robot/sr_hand/model/robots/xacro/arm_and_hand_motor.urdf.xacro (robot description, xacro)
@@ -9,5 +9,5 @@
     <parent link="shadowarm_handsupport_motor"/>
     <child link="forearm_motor"/>
-    <origin xyz="0 0 0" rpy="0 0 ${M_PI}" />
+    <origin xyz="0 0 0" rpy="0 0 ${2.36}" />
     <axis xyz="0 -1 0" />
     <limit lower="0" upper="0" effort="10"

Commit message: attached the arm to the desk. WARNING: may not work with the rest of the manipulation stack

File: shadow_robot/sr_hand/model/robots/arm_and_hand_motor.urdf (robot description, URDF)
Before this commit: robot arm_and_hand, 30 links, 29 joints
Links:
- added link desk_pillar, mass 100.0; collision cylinder length=1.0 radius=0.1; visual cylinder length=1.0 radius=0.1
- added link desk_support, mass 1000.0; collision cylinder length=0.02 radius=1.0; visual cylinder length=0.02 radius=1.0
Joints:
- added joint arm_to_desk_fixed: type fixed, parent desk_pillar, child shadowarm_base, origin xyz=0 0 1.0 rpy=0 0 0
- added joint desk_joint: type fixed, parent desk_support, child desk_pillar, origin xyz=0 0 0.01 rpy=0 0 0

File: shadow_robot/sr_hand/model/robots/xacro/arm_and_hand_motor.urdf.xacro (robot description, xacro)
@@ -4,4 +4,11 @@
   <include filename="$(find sr_hand)/model/hand_urdf/full_hand_motor.urdf.xacro" />
   <include filename="$(find sr_hand)/model/gazebo/gazebo.urdf.xacro" />
+  <include filename="$(find sr_hand)/model/desk/desk.urdf.xacro" />
+  <xacro:desk/>
+  <joint name="arm_to_desk_fixed" type="fixed">
+    <parent link="desk_pillar"/>
+    <child link="shadowarm_base"/>
+    <origin rpy="0 0 0" xyz="0 0 1.0"/>
+  </joint>
   <xacro:sr_arm_motor>
   </xacro:sr_arm_motor>
