Commit message: More concise model (we don't need the Gazebo informations) + updating the header when publishing joint_states. Still need to modify the model to have the correct kinematics.

File: denso_arm/model/denso_arm.urdf.xacro (robot description, xacro)
@@ -4,12 +4,8 @@
        xmlns:xacro="http://www.ros.org/wiki/xacro"
        name="denso_arm">
-  <include filename="$(find sr_hand)/model/materials.urdf.xacro" />
+  <material name="Grey">
+    <color rgba="0.2 0.2 0.2 1.0"/>
+  </material>
   <link name="base">
-    <inertial>
-      <mass value="0.010" />
-      <origin xyz="0 0 0.025" />
-      <inertia  ixx="1.0" ixy="0.0"  ixz="0.0"  iyy="0.0"  iyz="0.0"
-		izz="0.0" />
-    </inertial>
     <visual>
       <origin xyz="0 0 0" rpy="0 0 0" />
@@ -19,18 +15,6 @@
       <material name="Grey" />
     </visual>
-    <collision>
-      <origin xyz="0 0 0.02" rpy="0 0 0" />
-      <geometry name="base_collision_geom">
-	<box size="0.015 0.015 0.020" />
-      </geometry>
-    </collision>
   </link>
   <link name="link_1">
-    <inertial>
-      <mass value="0.010" />
-      <origin xyz="0 0 0.025" />
-      <inertia  ixx="1.0" ixy="0.0"  ixz="0.0"  iyy="0.0"  iyz="0.0"
-		izz="0.0" />
-    </inertial>
     <visual>
       <origin xyz="0 0 0" rpy="0 0 0" />
@@ -40,10 +24,4 @@
       <material name="Grey" />
     </visual>
-    <collision>
-      <origin xyz="0 0 0.02" rpy="0 0 0" />
-      <geometry name="link_1_collision_geom">
-	<box size="0.015 0.015 0.020" />
-      </geometry>
-    </collision>
   </link>
   <joint name="denso_J0" type="revolute">
@@ -54,13 +32,6 @@
     <limit lower="-2.967" upper="2.967" effort="10"
 	   velocity="1.0" />
-    <dynamics damping="50.5"/>
   </joint>
   <link name="link_2">
-    <inertial>
-      <mass value="0.010" />
-      <origin xyz="0 0 0.025" />
-      <inertia  ixx="1.0" ixy="0.0"  ixz="0.0"  iyy="0.0"  iyz="0.0"
-		izz="0.0" />
-    </inertial>
     <visual>
       <origin xyz="0 0 0" rpy="0 0 0" />
@@ -70,10 +41,4 @@
       <material name="Grey" />
     </visual>
-    <collision>
-      <origin xyz="0 0 0.02" rpy="0 0 0" />
-      <geometry name="link_2_collision_geom">
-	<box size="0.015 0.015 0.020" />
-      </geometry>
-    </collision>
   </link>
   <joint name="denso_J1" type="revolute">
@@ -84,13 +49,6 @@
     <limit lower="-1.745" upper="2.356" effort="10"
 	   velocity="1.0" />
-    <dynamics damping="50.5"/>
   </joint>
   <link name="link_3">
-    <inertial>
-      <mass value="0.010" />
-      <origin xyz="0 0 0.025" />
-      <inertia  ixx="1.0" ixy="0.0"  ixz="0.0"  iyy="0.0"  iyz="0.0"
-		izz="0.0" />
-    </inertial>
     <visual>
       <origin xyz="0 0 0" rpy="0 0 0" />
@@ -100,10 +58,4 @@
       <material name="Grey" />
     </visual>
-    <collision>
-      <origin xyz="0 0 0.02" rpy="0 0 0" />
-      <geometry name="link_3_collision_geom">
-	<box size="0.015 0.015 0.020" />
-      </geometry>
-    </collision>
   </link>
   <joint name="denso_J2" type="revolute">
@@ -114,13 +66,6 @@
     <limit lower="-2.094" upper="2.670" effort="10"
 	   velocity="1.0" />
-    <dynamics damping="50.5"/>
   </joint>
   <link name="link_4">
-    <inertial>
-      <mass value="0.010" />
-      <origin xyz="0 0 0.025" />
-      <inertia  ixx="1.0" ixy="0.0"  ixz="0.0"  iyy="0.0"  iyz="0.0"
-		izz="0.0" />
-    </inertial>
     <visual>
       <origin xyz="0 0 0" rpy="0 0 0" />
@@ -130,10 +75,4 @@
       <material name="Grey" />
     </visual>
-    <collision>
-      <origin xyz="0 0 0.02" rpy="0 0 0" />
-      <geometry name="link_4_collision_geom">
-	<box size="0.015 0.015 0.020" />
-      </geometry>
-    </collision>
   </link>
   <joint name="denso_J3" type="revolute">
@@ -144,13 +83,6 @@
     <limit lower="-4.712" upper="4.712" effort="10"
 	   velocity="1.0" />
-    <dynamics damping="50.5"/>
   </joint>
   <link name="link_5">
-    <inertial>
-      <mass value="0.010" />
-      <origin xyz="0 0 0.025" />
-      <inertia  ixx="1.0" ixy="0.0"  ixz="0.0"  iyy="0.0"  iyz="0.0"
-		izz="0.0" />
-    </inertial>
     <visual>
       <origin xyz="0 0 0" rpy="0 0 0" />
@@ -160,10 +92,4 @@
       <material name="Grey" />
     </visual>
-    <collision>
-      <origin xyz="0 0 0.02" rpy="0 0 0" />
-      <geometry name="link_5_collision_geom">
-	<box size="0.015 0.015 0.020" />
-      </geometry>
-    </collision>
   </link>
   <joint name="denso_J4" type="revolute">
@@ -174,13 +100,6 @@
     <limit lower="-2.094" upper="2.094" effort="10"
 	   velocity="1.0" />
-    <dynamics damping="50.5"/>
   </joint>
   <link name="link_6">
-    <inertial>
-      <mass value="0.010" />
-      <origin xyz="0 0 0.025" />
-      <inertia  ixx="1.0" ixy="0.0"  ixz="0.0"  iyy="0.0"  iyz="0.0"
-		izz="0.0" />
-    </inertial>
     <visual>
       <origin xyz="0 0 0" rpy="0 0 0" />
@@ -190,10 +109,4 @@
       <material name="Grey" />
     </visual>
-    <collision>
-      <origin xyz="0 0 0.02" rpy="0 0 0" />
-      <geometry name="link_6_collision_geom">
-	<box size="0.015 0.015 0.020" />
-      </geometry>
-    </collision>
   </link>
   <joint name="denso_J5" type="revolute">
@@ -204,5 +117,4 @@
     <limit lower="-6.283" upper="6.283" effort="10"
 	   velocity="1.0" />
-    <dynamics damping="50.5"/>
   </joint>
 </robot>

Commit message: Model changed to reflect the denso arm (approximative model).

File: denso_arm/model/denso_arm.urdf.xacro (robot description, xacro)
@@ -7,9 +7,12 @@
     <color rgba="0.2 0.2 0.2 1.0"/>
   </material>
+  <material name="LightGrey">
+    <color rgba="0.6 0.6 0.6 1.0"/>
+  </material>
   <link name="base">
     <visual>
-      <origin xyz="0 0 0" rpy="0 0 0" />
+      <origin xyz="0 0 0.0975" rpy="0 0 0" />
       <geometry name="base_visual">
-	<box size="0.015 0.015 0.020" />
+	<box size="0.195 0.195 0.195" />
       </geometry>
       <material name="Grey" />
@@ -18,7 +21,7 @@
   <link name="link_1">
     <visual>
-      <origin xyz="0 0 0" rpy="0 0 0" />
+      <origin xyz="0 0 0.06" rpy="0 0 0" />
       <geometry name="link_1_visual">
-	<box size="0.015 0.015 0.020" />
+	<box size="0.100 0.100 0.120" />
       </geometry>
       <material name="Grey" />
@@ -28,6 +31,6 @@
     <parent link="base"/>
     <child link="link_1"/>
-    <origin xyz="0 0 0.025" rpy="0 0 0" />
-    <axis xyz="1 0 0" />
+    <origin xyz="0 0 0.198" rpy="0 0 0" />
+    <axis xyz="0 0 1" />
     <limit lower="-2.967" upper="2.967" effort="10"
 	   velocity="1.0" />
@@ -35,7 +38,7 @@
   <link name="link_2">
     <visual>
-      <origin xyz="0 0 0" rpy="0 0 0" />
+      <origin xyz="0 0 0.225" rpy="0 0 0" />
       <geometry name="link_2_visual">
-	<box size="0.015 0.015 0.020" />
+	<box size="0.05 0.05 0.400" />
       </geometry>
       <material name="Grey" />
@@ -45,5 +48,5 @@
     <parent link="link_1"/>
     <child link="link_2"/>
-    <origin xyz="0 0 0.025" rpy="0 0 0" />
+    <origin xyz="0 0 0.190" rpy="0 0 0" />
     <axis xyz="1 0 0" />
     <limit lower="-1.745" upper="2.356" effort="10"
@@ -52,7 +55,7 @@
   <link name="link_3">
     <visual>
-      <origin xyz="0 0 0" rpy="0 0 0" />
+      <origin xyz="0 0 0.1425" rpy="0 0 0" />
       <geometry name="link_3_visual">
-	<box size="0.015 0.015 0.020" />
+	<box size="0.05 0.05 0.20" />
       </geometry>
       <material name="Grey" />
@@ -62,5 +65,5 @@
     <parent link="link_2"/>
     <child link="link_3"/>
-    <origin xyz="0 0 0.025" rpy="0 0 0" />
+    <origin xyz="0 0 0.450" rpy="0 0 0" />
     <axis xyz="1 0 0" />
     <limit lower="-2.094" upper="2.670" effort="10"
@@ -69,7 +72,7 @@
   <link name="link_4">
     <visual>
-      <origin xyz="0 0 0" rpy="0 0 0" />
+      <origin xyz="0 0 0.0675" rpy="0 0 0" />
       <geometry name="link_4_visual">
-	<box size="0.015 0.015 0.020" />
+	<box size="0.05 0.05 0.10" />
       </geometry>
       <material name="Grey" />
@@ -79,6 +82,6 @@
     <parent link="link_3"/>
     <child link="link_4"/>
-    <origin xyz="0 0 0.025" rpy="0 0 0" />
-    <axis xyz="1 0 0" />
+    <origin xyz="0 0 0.285" rpy="0 0 0" />
+    <axis xyz="0 0 1" />
     <limit lower="-4.712" upper="4.712" effort="10"
 	   velocity="1.0" />
@@ -86,7 +89,7 @@
   <link name="link_5">
     <visual>
-      <origin xyz="0 0 0" rpy="0 0 0" />
+      <origin xyz="0 0 0.45" rpy="0 0 0" />
       <geometry name="link_5_visual">
-	<box size="0.015 0.015 0.020" />
+	<box size="0.03 0.03 0.80" />
       </geometry>
       <material name="Grey" />
@@ -96,5 +99,5 @@
     <parent link="link_4"/>
     <child link="link_5"/>
-    <origin xyz="0 0 0.025" rpy="0 0 0" />
+    <origin xyz="0 0 0.135" rpy="0 0 0" />
     <axis xyz="1 0 0" />
     <limit lower="-2.094" upper="2.094" effort="10"
@@ -103,9 +106,9 @@
   <link name="link_6">
     <visual>
-      <origin xyz="0 0 0" rpy="0 0 0" />
+      <origin xyz="0 0 0.0005" rpy="0 0 0" />
       <geometry name="link_6_visual">
-	<box size="0.015 0.015 0.020" />
+	<box size="0.04 0.04 0.001" />
       </geometry>
-      <material name="Grey" />
+      <material name="LightGrey" />
     </visual>
   </link>
@@ -113,6 +116,6 @@
     <parent link="link_5"/>
     <child link="link_6"/>
-    <origin xyz="0 0 0.025" rpy="0 0 0" />
-    <axis xyz="1 0 0" />
+    <origin xyz="0 0 0.90" rpy="0 0 0" />
+    <axis xyz="0 0 1" />
     <limit lower="-6.283" upper="6.283" effort="10"
 	   velocity="1.0" />

Commit message: Wrong scale.

File: denso_arm/model/denso_arm.urdf.xacro (robot description, xacro)
@@ -89,5 +89,5 @@
   <link name="link_5">
     <visual>
-      <origin xyz="0 0 0.45" rpy="0 0 0" />
+      <origin xyz="0 0 0.045" rpy="0 0 0" />
       <geometry name="link_5_visual">
 	<box size="0.03 0.03 0.80" />
@@ -116,5 +116,5 @@
     <parent link="link_5"/>
     <child link="link_6"/>
-    <origin xyz="0 0 0.90" rpy="0 0 0" />
+    <origin xyz="0 0 0.090" rpy="0 0 0" />
     <axis xyz="0 0 1" />
     <limit lower="-6.283" upper="6.283" effort="10"

Commit message: Improved denso arm description to be a bit more accurate and changed denso_arm to publish joint angles in radians.

File: denso_arm/model/denso_arm.urdf.xacro (robot description, xacro)
@@ -12,5 +12,5 @@
   <link name="base">
     <visual>
-      <origin xyz="0 0 0.0975" rpy="0 0 0" />
+      <origin xyz="0 0 0.098" rpy="0 0 0" />
       <geometry name="base_visual">
 	<box size="0.195 0.195 0.195" />
@@ -91,5 +91,5 @@
       <origin xyz="0 0 0.045" rpy="0 0 0" />
       <geometry name="link_5_visual">
-	<box size="0.03 0.03 0.80" />
+	<box size="0.03 0.03 0.08" />
       </geometry>
       <material name="Grey" />

Commit message: The hand is correctly attached to the arm.

File: denso_arm/model/denso_arm.urdf.xacro (robot description, xacro)
@@ -31,5 +31,5 @@
     <parent link="base"/>
     <child link="link_1"/>
-    <origin xyz="0 0 0.198" rpy="0 0 0" />
+    <origin xyz="0 0 0.198" rpy="0 0 1.57" />
     <axis xyz="0 0 1" />
     <limit lower="-2.967" upper="2.967" effort="10"
