Commit message: ok fixed the max effort, the arm is now moving in gazebo

File: sr_description/arm/xacro/hand_support/shadowarm_handsupport_motor.urdf.xacro (robot description, xacro)
@@ -32,5 +32,5 @@
       <axis xyz="0 0 -1" />
       <limit lower="-${M_PI/2}" upper="${M_PI/2}"
-      effort="10" velocity="1.0"/>
+      effort="100" velocity="1.0"/>
       <dynamics damping="10.5"/>
     </joint>

File: sr_description/arm/xacro/hand_support/shadowarm_handsupport_muscle.urdf.xacro (robot description, xacro)
@@ -32,5 +32,5 @@
       <axis xyz="0 0 -1" />
       <limit lower="-${M_PI/2}" upper="${M_PI/2}"
-      effort="10" velocity="1.0"/>
+      effort="100" velocity="1.0"/>
       <dynamics damping="10.5"/>
     </joint>

File: sr_description/arm/xacro/upper_arm/shadowarm_upperarm.urdf.xacro (robot description, xacro)
@@ -31,5 +31,5 @@
       <origin xyz="0 -0.134 0.5305" rpy="0 -${M_PI} 0.0" /> <!-- yaw=-0.026 -->
       <axis xyz="0 -1 0" />
-      <limit lower="0" upper="${M_PI/2}" effort="10" velocity="1.0"/>
+      <limit lower="0" upper="${M_PI/2}" effort="150" velocity="1.0"/>
       <dynamics damping="50.5"/>
     </joint>
