Commit message: Rotate the forearm

File: sr_description/hand/xacro/forearm/forearm_lite.urdf.xacro (robot description, xacro)
@@ -3,4 +3,5 @@
   <!-- prefix can be anything but usually is "r_" or  "l_" for right and left hands distinction -->
   <xacro:macro name="forearm" params="muscle prefix">
+      <property name="M_PI" value="3.1415926535897931" />
       <link name="${prefix}forearm">
         <inertial>
@@ -11,16 +12,16 @@
         </inertial>
         <visual>
-        <origin xyz="0 0 0" rpy="0 0 0" />
-        <geometry name="${prefix}forearm_visual">
-          <xacro:if value="${muscle}">
-             <mesh filename="package://sr_description/hand/model/forearm_lite.dae"
-                   scale="0.001 0.001 0.001"/>
-          </xacro:if>
-          <xacro:unless value="${muscle}">
-             <mesh filename="package://sr_description/hand/model/forearm_lite.dae"
-                   scale="1.0 1.0 1.0"/>
-          </xacro:unless>
-        </geometry>
-        <material name="Grey" />
+          <origin xyz="0 0 0" rpy="0 0 ${M_PI/2}" />
+          <geometry name="${prefix}forearm_visual">
+            <xacro:if value="${muscle}">
+               <mesh filename="package://sr_description/hand/model/forearm_lite.dae"
+                     scale="0.001 0.001 0.001"/>
+            </xacro:if>
+            <xacro:unless value="${muscle}">
+               <mesh filename="package://sr_description/hand/model/forearm_lite.dae"
+                     scale="1.0 1.0 1.0"/>
+            </xacro:unless>
+          </geometry>
+          <material name="Grey" />
         </visual>
         <collision>
@@ -54,8 +55,10 @@
         </collision>
       </link>
+      <!--
       <gazebo reference="${prefix}forearm">
         <material>LightGrey</material>
         <selfCollide>false</selfCollide>
       </gazebo>
+      -->
   </xacro:macro>
 </robot>

Commit message: Fix forearm color in gazebo

File: sr_description/hand/xacro/forearm/forearm_lite.urdf.xacro (robot description, xacro)
@@ -55,10 +55,8 @@
         </collision>
       </link>
-      <!--
       <gazebo reference="${prefix}forearm">
-        <material>LightGrey</material>
+        <material>Grey</material>
         <selfCollide>false</selfCollide>
       </gazebo>
-      -->
   </xacro:macro>
 </robot>

Commit message: Fix forearm collision.

File: sr_description/hand/xacro/forearm/forearm_lite.urdf.xacro (robot description, xacro)
@@ -33,7 +33,7 @@
           </xacro:if>
           <xacro:unless value="${muscle}">
-            <origin xyz="0 0 0.092" rpy="0 0 0" />
+            <origin xyz="0 0 0.0775" rpy="0 0 0" />
             <geometry name="${prefix}forearm_collision">
-              <box size="0.140 0.140 0.184" />
+              <box size="0.109 0.120 0.155" />
             </geometry>
           </xacro:unless>

Commit message: Remove wrist mount collider

File: sr_description/hand/xacro/forearm/forearm_lite.urdf.xacro (robot description, xacro)
@@ -39,19 +39,4 @@
           </xacro:unless>
         </collision>
-        <!-- wrist mount -->
-        <collision>
-          <xacro:if value="${muscle}">
-            <origin xyz="0 0 0.395" rpy="0 0 0" />
-            <geometry>
-              <box size="0.03 0.04 0.06"/>
-            </geometry>
-          </xacro:if>
-          <xacro:unless value="${muscle}">
-            <origin xyz="0 -0.01 0.181" rpy="0 0.78 0" />
-            <geometry>
-              <box size="0.07 0.07 0.07"/>
-            </geometry>
-          </xacro:unless>
-        </collision>
       </link>
       <gazebo reference="${prefix}forearm">

Commit message: Clean up.

File: sr_description/hand/xacro/forearm/forearm_lite.urdf.xacro (robot description, xacro)
@@ -40,8 +40,4 @@
         </collision>
       </link>
-      <gazebo reference="${prefix}forearm">
-        <material>Grey</material>
-        <selfCollide>false</selfCollide>
-      </gazebo>
   </xacro:macro>
 </robot>

Commit message: Rough weight guess for forearm

File: sr_description/hand/xacro/forearm/forearm_lite.urdf.xacro (robot description, xacro)
@@ -7,6 +7,6 @@
         <inertial>
           <origin xyz="0 0 0.09" rpy="0 0 0"/>
-          <!-- TODO: What is the mass of the lite forearm? -->
-          <mass value="3.0" />
+          <!-- TODO: This is a rough estimate. Total hand is 2359g -->
+          <mass value="1.8" />
           <inertia  ixx="0.108" ixy="0.0"  ixz="0.0"  iyy="0.108"  iyz="0.0"  izz="0.054" />
         </inertial>

Commit message: fixing hand lite xacro

File: sr_description/hand/xacro/forearm/forearm_lite.urdf.xacro (robot description, xacro)
@@ -3,5 +3,4 @@
   <!-- prefix can be anything but usually is "r_" or  "l_" for right and left hands distinction -->
   <xacro:macro name="forearm" params="muscle prefix">
-    <xacro:property name="M_PI" value="3.1415926535897931" />
     <link name="${prefix}forearm">
       <inertial>

File: sr_description/hand/xacro/hand_lite.urdf.xacro (robot description, xacro)
@@ -8,5 +8,6 @@
   <xacro:include filename="$(find sr_description)/hand/xacro/finger/fingers.urdf.xacro" />
   <xacro:include filename="$(find sr_description)/hand/xacro/thumb/thumb.urdf.xacro" />
-  <!-- muscletrans is true for muscle transmission to be used, false to use motor transmission -->
+  <xacro:property name="M_PI" value="3.1415926535897931" />
+    <!-- muscletrans is true for muscle transmission to be used, false to use motor transmission -->
   <!-- muscle is true for muscle hand or false for motor hand -->
   <!-- bio is true for biotac finger or false for standard finger -->
