Commit message: Fixed missing includes Corrected wrong names in gazebo includes Replaced deprecated include with xacro:include Fixed wrong includes

File: sr_description/hand/xacro/finger/distal/distal.gazebo.xacro (robot description, xacro)
@@ -1,5 +1,5 @@
 <?xml version="1.0"?>
 <robot xmlns:xacro="http://ros.org/wiki/xacro">
-  <xacro:macro name="middle_gazebo" params="prefix">
+  <xacro:macro name="distal_gazebo" params="prefix">
   <!-- prefix can be anything but usually is "r_" or  "l_" for right and left hands distinction -->
   <gazebo reference="${prefix}${link_prefix}distal">

File: sr_description/hand/xacro/finger/distal/distal.urdf.xacro (robot description, xacro)
@@ -6,4 +6,5 @@
        xmlns:body="http://playerstage.sourceforge.net/gazebo/xmlschema/#body"
        xmlns:geom="http://playerstage.sourceforge.net/gazebo/xmlschema/#geom">
+  <xacro:include filename="$(find sr_description)/hand/xacro/finger/distal/distal.gazebo.xacro" />
   <xacro:include filename="$(find sr_description)/hand/xacro/finger/distal/distal.transmission.xacro" />
   <!-- muscle is true for muscle hand or false for motor hand -->

File: sr_description/hand/xacro/finger/lfmetacarpal/lfmetacarpal.gazebo.xacro (robot description, xacro)
@@ -1,5 +1,5 @@
 <?xml version="1.0"?>
 <robot xmlns:xacro="http://ros.org/wiki/xacro">
-  <xacro:macro name="shadowhand_lfmetacarpal_gazebo" params="prefix">
+  <xacro:macro name="lfmetacarpal_gazebo" params="prefix">
   <!-- prefix can be anything but usually is "r_" or  "l_" for right and left hands distinction -->
   <gazebo reference="${prefix}lfmetacarpal">

File: sr_description/hand/xacro/thumb/thbase.gazebo.xacro (robot description, xacro)
@@ -1,17 +1,17 @@
 <?xml version="1.0"?>
 <robot xmlns:xacro="http://ros.org/wiki/xacro">
-  <xacro:macro name="thmiddle_gazebo" params="prefix">
+  <xacro:macro name="thbase_gazebo" params="prefix">
   <!-- prefix can be anything but usually is "r_" or  "l_" for right and left hands distinction -->
-  <gazebo reference="${prefix}thmiddle">
-      <sensor type="contact" name="${prefix}thmiddle_contact_sensor">
+  <gazebo reference="${prefix}thbase">
+      <sensor type="contact" name="${prefix}thbase_contact_sensor">
         <update_rate>100.0</update_rate>
         <contact>
-          <collision>${prefix}thmiddle_collision_geom</collision>
+          <collision>${prefix}thbase_collision_geom</collision>
         </contact>
-        <plugin name="${prefix}thmiddle_gazebo_ros_bumper_controller" filename="libgazebo_ros_bumper.so">
+        <plugin name="${prefix}thbase_gazebo_ros_bumper_controller" filename="libgazebo_ros_bumper.so">
           <alwaysOn>true</alwaysOn>
-          <frameName>${prefix}thmiddle</frameName>
+          <frameName>${prefix}thbase</frameName>
           <updateRate>100.0</updateRate>
-          <bumperTopicName>${prefix}thmiddle_bumper</bumperTopicName>
+          <bumperTopicName>${prefix}thbase_bumper</bumperTopicName>
         </plugin>
       </sensor>

File: sr_description/hand/xacro/thumb/thdistal.urdf.xacro (robot description, xacro)
@@ -6,4 +6,5 @@
        xmlns:body="http://playerstage.sourceforge.net/gazebo/xmlschema/#body"
        xmlns:geom="http://playerstage.sourceforge.net/gazebo/xmlschema/#geom">
+  <xacro:include filename="$(find sr_description)/hand/xacro/thumb/thdistal.gazebo.xacro" />
   <xacro:include filename="$(find sr_description)/hand/xacro/thumb/thdistal.transmission.xacro" />
   <!-- muscle is true for muscle hand or false for motor hand -->
