Commit message: Added new distal visual models for finger and thumb ellipsoid tips, which include the nano17 sensors and cable Corrected the models to be in meter Modified xacro to use the new models

File: sr_description/hand/xacro/finger/distal/distal.urdf.xacro (robot description, xacro)
@@ -34,5 +34,5 @@
             <!-- Ellispoid distal  -->
             <xacro:if value="${eli}">
-               <mesh filename="package://sr_description/hand/model/distal_ellipsoid.dae" scale="0.001 0.001 0.001" />
+							<mesh filename="package://sr_description/hand/model/distal_ellipsoid_visual.dae" scale="0.001 0.001 0.001" />
             </xacro:if>
             <!-- Check for biotac distal -->

File: sr_description/hand/xacro/thumb/thdistal.urdf.xacro (robot description, xacro)
@@ -116,5 +116,5 @@
 						<!-- Ellispoid distal  -->
 						<xacro:if value="${eli}">
-							<mesh filename="package://sr_description/hand/model/distal_ellipsoid.dae" scale="0.001 0.001 0.001" />
+							<mesh filename="package://sr_description/hand/model/thdistal_ellipsoid_visual.dae" scale="0.001 0.001 0.001" />
 						</xacro:if>
 						<!-- Check for uni distal -->
@@ -139,5 +139,5 @@
 					<!-- Ellispoid distal  -->
 						<xacro:if value="${eli}">
-							<mesh filename="package://sr_description/hand/model/distal_ellipsoid.dae" scale="0.001 0.001 0.001" />
+						  <mesh filename="package://sr_description/hand/model/thdistal_ellipsoid.dae" scale="0.001 0.001 0.001" />
 						</xacro:if>
 						<!-- Check for uni distal -->

Commit message: Removed unnecessary left meshes Moved ellipsoid distal meshes to a subfolder

File: sr_description/hand/xacro/finger/distal/distal.urdf.xacro (robot description, xacro)
@@ -34,5 +34,5 @@
             <!-- Ellispoid distal  -->
             <xacro:if value="${eli}">
-							<mesh filename="package://sr_description/hand/model/distal_ellipsoid_visual.dae" scale="0.001 0.001 0.001" />
+							<mesh filename="package://sr_description/hand/model/ellipsoids/distal_ellipsoid_visual.dae" scale="0.001 0.001 0.001" />
             </xacro:if>
             <!-- Check for biotac distal -->
@@ -62,5 +62,5 @@
             <!-- Ellispoid distal  -->
             <xacro:if value="${eli}">
-               <mesh filename="package://sr_description/hand/model/distal_ellipsoid.dae" scale="0.001 0.001 0.001" />
+               <mesh filename="package://sr_description/hand/model/ellipsoids/distal_ellipsoid.dae" scale="0.001 0.001 0.001" />
             </xacro:if>
             <!-- Check for biotac distal -->

File: sr_description/hand/xacro/thumb/thdistal.urdf.xacro (robot description, xacro)
@@ -116,5 +116,5 @@
 						<!-- Ellispoid distal  -->
 						<xacro:if value="${eli}">
-							<mesh filename="package://sr_description/hand/model/thdistal_ellipsoid_visual.dae" scale="0.001 0.001 0.001" />
+							<mesh filename="package://sr_description/hand/model/ellipsoids/thdistal_ellipsoid_visual.dae" scale="0.001 0.001 0.001" />
 						</xacro:if>
 						<!-- Check for uni distal -->
@@ -139,5 +139,5 @@
 					<!-- Ellispoid distal  -->
 						<xacro:if value="${eli}">
-						  <mesh filename="package://sr_description/hand/model/thdistal_ellipsoid.dae" scale="0.001 0.001 0.001" />
+						  <mesh filename="package://sr_description/hand/model/ellipsoids/thdistal_ellipsoid.dae" scale="0.001 0.001 0.001" />
 						</xacro:if>
 						<!-- Check for uni distal -->

Commit message: Tested real inertia in gazebo indigo, retuned controllers in gazebo and adapted dynamics damping to be coherent with realistic inertia

File: sr_description/hand/xacro/finger/distal/distal.urdf.xacro (robot description, xacro)
@@ -21,6 +21,6 @@
         <mass value="0.010" />
         <origin xyz="0 0 0.012" />
-        <inertia  ixx="0.001" ixy="0.0"  ixz="0.0"  iyy="0.001"  iyz="0.0"
-        izz="0.00025" />
+        <inertia  ixx="0.0000031" ixy="0.0"  ixz="0.0"  iyy="0.0000031"  iyz="0.0"
+        izz="0.00000053" />
       </inertial>
       <visual>
@@ -92,5 +92,5 @@
           velocity="1.0" />
       </xacro:unless>
-      <dynamics damping="0.1"/>
+      <dynamics damping="0.001"/>
     </joint>
     <link name="${prefix}${link_prefix}tip">

File: sr_description/hand/xacro/finger/knuckle/knuckle.urdf.xacro (robot description, xacro)
@@ -19,5 +19,5 @@
         <!--<insert_block name="origin" /> -->
         <mass value="0.08" />
-        <inertia  ixx="0.0026" ixy="0.0"  ixz="0.0"  iyy="0.0026"  iyz="0.0"	izz="0.0032" />
+        <inertia  ixx="0.000026" ixy="0.0"  ixz="0.0"  iyy="0.000026"  iyz="0.0"	izz="0.000032" />
       </inertial>
       <visual>
@@ -43,5 +43,5 @@
       <limit lower="${-20/180*M_PI}" upper="${20/180*M_PI}"
       effort="2" velocity="1.0"/>
-      <dynamics damping="0.1"/>
+      <dynamics damping="0.01"/>
     </joint>
     <!-- extensions -->

File: sr_description/hand/xacro/finger/lfmetacarpal/lfmetacarpal.urdf.xacro (robot description, xacro)
@@ -17,5 +17,5 @@
         <origin xyz="0 0 0.04" rpy="0 0 0" />
         <mass value="0.030" />
-	    <inertia  ixx="0.00545" ixy="0.0"  ixz="0.0"  iyy="0.0056352"  iyz="0.0" izz="0.0004272" />
+	    <inertia  ixx="0.0000545" ixy="0.0"  ixz="0.0"  iyy="0.000056352"  iyz="0.0" izz="0.000004272" />
       </inertial>
       <visual>
@@ -41,5 +41,5 @@
         <limit lower="0" upper="${45/180*M_PI}" effort="2"
       velocity="1.0" />
-      <dynamics damping="0.1"/>
+      <dynamics damping="0.001"/>
     </joint>
     <!-- extensions -->

File: sr_description/hand/xacro/finger/middle/middle.urdf.xacro (robot description, xacro)
@@ -18,6 +18,6 @@
         <origin xyz="0 0 0.0125" rpy="0 0 0" />
         <mass value="0.020" />
-        <inertia  ixx="0.002" ixy="0.0"  ixz="0.0"  iyy="0.002"  iyz="0.0"
-        izz="0.0002" />
+        <inertia  ixx="0.0000067" ixy="0.0"  ixz="0.0"  iyy="0.0000067"  iyz="0.0"
+        izz="0.00000006" />
       </inertial>
       <visual>
@@ -54,5 +54,5 @@
       <limit lower="0" upper="${M_PI/2}" effort="2"
       velocity="1.0" />
-      <dynamics damping="0.1"/>
+      <dynamics damping="0.001"/>
     </joint>
     <!-- extensions -->

File: sr_description/hand/xacro/finger/proximal/proximal.urdf.xacro (robot description, xacro)
@@ -18,6 +18,6 @@
         <mass value="0.030" />
         <origin xyz="0 0 0.0225" />
-        <inertia  ixx="0.003" ixy="0.0"  ixz="0.0"  iyy="0.003"  iyz="0.0"
-        izz="0.0003" />
+        <inertia  ixx="0.000037" ixy="0.0"  ixz="0.0"  iyy="0.000037"  iyz="0.0"
+        izz="0.00000018" />
       </inertial>
       <visual>
@@ -42,5 +42,5 @@
       <limit lower="0" upper="${M_PI/2}" effort="2"
       velocity="1.0"/>
-      <dynamics damping="0.1"/>
+      <dynamics damping="0.001"/>
     </joint>
     <!-- extensions -->

File: sr_description/hand/xacro/palm/palm.urdf.xacro (robot description, xacro)
@@ -17,5 +17,5 @@
         <origin xyz="0 0 0.035" rpy="0 0 0" />
         <mass value="0.3" />
-        <inertia  ixx="0.003581" ixy="0.0"  ixz="0.0"  iyy="0.005287"  iyz="0.0"	izz="0.002545" />
+        <inertia  ixx="0.0003581" ixy="0.0"  ixz="0.0"  iyy="0.0005287"  iyz="0.0"	izz="0.0002545" />
       </inertial>
       <visual>
@@ -82,5 +82,5 @@
       <limit lower="${-40/180*M_PI}" upper="${28/180*M_PI}"
       effort="30" velocity="1.0"/>
-      <dynamics damping="0.1"/>
+      <dynamics damping="0.01"/>
     </joint>
     <!-- extensions -->

File: sr_description/hand/xacro/thumb/thhub.urdf.xacro (robot description, xacro)
@@ -53,5 +53,5 @@
         <limit lower="${-12/180*M_PI}" upper="${12/180*M_PI}" effort="10"
         velocity="1.0" />
-        <dynamics damping="0.1"/>
+        <dynamics damping="0.02"/>
       </joint>
     </xacro:unless>

File: sr_description/hand/xacro/wrist/wrist.urdf.xacro (robot description, xacro)
@@ -10,5 +10,5 @@
 		  <origin xyz="0 0 0" rpy="0 0 0" />
 		  <mass value="0.1" />
-		  <inertia  ixx="0.0120" ixy="0.0"  ixz="0.0"  iyy="0.0148"  iyz="0.0" izz="0.00438" />
+		  <inertia  ixx="0.000024" ixy="0.0"  ixz="0.0"  iyy="0.000104"  iyz="0.0" izz="0.0000867" />
       </inertial>
       <visual>
@@ -61,5 +61,5 @@
       <axis xyz="0 ${reflect} 0" />
       <limit lower="${-30/180*M_PI}" upper="${10/180*M_PI}" effort="30" velocity="1.0"/>
-      <dynamics damping="0.1"/>
+      <dynamics damping="0.01"/>
     </joint>
     <!-- extensions -->

Commit message: adding model, load and test for bt sp hand - not working yet

File: sr_description/hand/xacro/finger/distal/distal.urdf.xacro (robot description, xacro)
@@ -84,7 +84,14 @@
               </xacro:if>
               <xacro:unless value="${bio}">
-                <!-- Standard distal  -->
-                <mesh filename="package://sr_description/hand/model/F1.dae"
-                scale="0.001 0.001 0.001" />
+		<xacro:if value="${bt_sp}">
+                  <!-- bt_sp distal  -->
+                  <mesh filename="package://sr_description/hand/model/biotacs/sp.dae"
+			scale="0.001 0.001 0.001" />
+		</xacro:if>
+		<xacro:unless value="${bt_sp}">
+                  <!-- Standard distal  -->
+                  <mesh filename="package://sr_description/hand/model/F1.dae"
+			scale="0.001 0.001 0.001" />
+		</xacro:unless>
               </xacro:unless>
             </xacro:unless>

File: sr_description/hand/xacro/thumb/thdistal.urdf.xacro (robot description, xacro)
@@ -173,7 +173,14 @@
               </xacro:if>
               <xacro:unless value="${ubi}">
-                <!-- Standard distal  -->
-                <mesh filename="package://sr_description/hand/model/TH1_z.dae"
-                scale="0.001 0.001 0.001" />
+		<xacro:if value="${bt_sp}">
+		  <!-- bt sp distal  -->
+		  <mesh filename="package://sr_description/hand/model/biotacs/sp.dae"
+			scale="0.001 0.001 0.001" />
+		</xacro:if>
+		<xacro:unless value="${bt_sp}">
+                  <!-- Standard distal  -->
+                  <mesh filename="package://sr_description/hand/model/TH1_z.dae"
+			scale="0.001 0.001 0.001" />
+		</xacro:unless>
               </xacro:unless>
             </xacro:unless>

Commit message: fixing scale problem

File: sr_description/hand/xacro/finger/distal/distal.urdf.xacro (robot description, xacro)
@@ -49,6 +49,5 @@
 		<xacro:if value="${bt_sp}">
                   <!-- bt_sp distal  -->
-                  <mesh filename="package://sr_description/hand/model/biotacs/sp.dae"
-			scale="0.001 0.001 0.001" />
+                  <mesh filename="package://sr_description/hand/model/biotacs/sp.dae" />
 		</xacro:if>
 		<xacro:unless value="${bt_sp}">
@@ -86,6 +85,5 @@
 		<xacro:if value="${bt_sp}">
                   <!-- bt_sp distal  -->
-                  <mesh filename="package://sr_description/hand/model/biotacs/sp.dae"
-			scale="0.001 0.001 0.001" />
+                  <mesh filename="package://sr_description/hand/model/biotacs/sp.dae" />
 		</xacro:if>
 		<xacro:unless value="${bt_sp}">

File: sr_description/hand/xacro/thumb/thdistal.urdf.xacro (robot description, xacro)
@@ -143,6 +143,5 @@
 		<xacro:if value="${bt_sp}">
 		  <!-- bt sp distal  -->
-		  <mesh filename="package://sr_description/hand/model/biotacs/sp.dae"
-			scale="0.001 0.001 0.001" />
+		  <mesh filename="package://sr_description/hand/model/biotacs/sp.dae" />
 		</xacro:if>
 		<xacro:unless value="${bt_sp}">
@@ -175,6 +174,5 @@
 		<xacro:if value="${bt_sp}">
 		  <!-- bt sp distal  -->
-		  <mesh filename="package://sr_description/hand/model/biotacs/sp.dae"
-			scale="0.001 0.001 0.001" />
+                  <mesh filename="package://sr_description/hand/model/biotacs/sp.dae" />
 		</xacro:if>
 		<xacro:unless value="${bt_sp}">
