Commit message: Fixed bumper sensors (collision name must be link name + _geom) Changed color of some hand material

File: sr_description/arm/xacro/lower_arm/shadowarm_lowerarm.urdf.xacro (robot description, xacro)
@@ -23,5 +23,5 @@
     </link>
     <gazebo reference="shadowarm_lowerarm">
-	<material>Gazebo/Grey</material>
+	<material>LightGrey</material>
 	<selfCollide>false</selfCollide>
     </gazebo>

File: sr_description/arm/xacro/trunk/shadowarm_trunk.urdf.xacro (robot description, xacro)
@@ -23,5 +23,5 @@
       </link>
       <gazebo reference="shadowarm_trunk">
-	<material>Gazebo/Grey</material>
+	<material>LightGrey</material>
 	<selfCollide>false</selfCollide>
       </gazebo>

File: sr_description/arm/xacro/upper_arm/shadowarm_upperarm.urdf.xacro (robot description, xacro)
@@ -23,5 +23,5 @@
     </link>
     <gazebo reference="shadowarm_upperarm">
-      <material>Gazebo/Grey</material>
+      <material>LightGrey</material>
       <selfCollide>false</selfCollide>
     </gazebo>

File: sr_description/hand/xacro/finger/distal/distal.gazebo.xacro (robot description, xacro)
@@ -4,8 +4,9 @@
   <!-- prefix can be anything but usually is "r_" or  "l_" for right and left hands distinction -->
   <gazebo reference="${prefix}${link_prefix}distal">
-      <sensor type="contact" name="${prefix}${link_prefix}distal_contact_sensor">
+      <sensor type="contact" name="${prefix}${link_prefix}distal_contact">
+				<always_on>true</always_on>
         <update_rate>100.0</update_rate>
         <contact>
-          <collision>${prefix}${link_prefix}distal_collision_geom</collision>
+          <collision>${prefix}${link_prefix}distal_geom</collision>
         </contact>
         <plugin name="${prefix}${link_prefix}distal_gazebo_ros_bumper_controller" filename="libgazebo_ros_bumper.so">
@@ -20,5 +21,5 @@
       <kp  value="10000000.0" />
       <kd  value="1.0" />
-      <material>Gazebo/Grey</material>
+      <material>LightGrey</material>
       <selfCollide>true</selfCollide>
     </gazebo>

File: sr_description/hand/xacro/finger/distal/distal.urdf.xacro (robot description, xacro)
@@ -27,22 +27,20 @@
         <origin xyz="0 0 0" rpy="0 0 0" />
         <geometry name="${prefix}${link_prefix}distal_visual">
-          <!-- Ubi distal -->
           <xacro:if value="${ubi}">
+						<!-- Ubi distal -->
             <mesh filename="package://sr_description/hand/model/F1.dae" scale="0.001 0.001 0.001" />
           </xacro:if>
-          <!-- Check for ellispoid distal -->
           <xacro:unless value="${ubi}">
-            <!-- Ellispoid distal  -->
             <xacro:if value="${eli}">
+							<!-- Ellispoid distal  -->
 							<mesh filename="package://sr_description/hand/model/ellipsoids/distal_ellipsoid_visual.dae" scale="0.001 0.001 0.001" />
             </xacro:if>
-            <!-- Check for biotac distal -->
             <xacro:unless value="${eli}">
-              <!-- biotac distal  -->
               <xacro:if value="${bio}">
-                 <mesh filename="package://sr_description/hand/model/F1.dae" scale="0.001 0.001 0.001" />
+								<!-- biotac distal  -->
+                <mesh filename="package://sr_description/hand/model/F1.dae" scale="0.001 0.001 0.001" />
               </xacro:if>
-              <!-- Standard distal  -->
               <xacro:unless value="${bio}">
+								 <!-- Standard distal  -->
                  <mesh filename="package://sr_description/hand/model/F1.dae" scale="0.001 0.001 0.001" />
               </xacro:unless>
@@ -55,23 +53,21 @@
         <origin xyz="0 0 0" rpy="0 0 0" />
         <geometry name="${prefix}${link_prefix}distal_collision_geom">
-            <!-- Ubi distal -->
           <xacro:if value="${ubi}">
+						<!-- Ubi distal -->
             <mesh filename="package://sr_description/hand/model/F1.dae" scale="0.001 0.001 0.001" />
           </xacro:if>
-          <!-- Check for ellispoid distal -->
           <xacro:unless value="${ubi}">
-            <!-- Ellispoid distal  -->
             <xacro:if value="${eli}">
-               <mesh filename="package://sr_description/hand/model/ellipsoids/distal_ellipsoid.dae" scale="0.001 0.001 0.001" />
+							<!-- Ellispoid distal  -->
+              <mesh filename="package://sr_description/hand/model/ellipsoids/distal_ellipsoid.dae" scale="0.001 0.001 0.001" />
             </xacro:if>
-            <!-- Check for biotac distal -->
             <xacro:unless value="${eli}">
-              <!-- biotac distal  -->
               <xacro:if value="${bio}">
-                 <mesh filename="package://sr_description/hand/model/F1.dae" scale="0.001 0.001 0.001" />
+								<!-- biotac distal  -->
+                <mesh filename="package://sr_description/hand/model/F1.dae" scale="0.001 0.001 0.001" />
               </xacro:if>
-              <!-- Standard distal  -->
               <xacro:unless value="${bio}">
-                 <mesh filename="package://sr_description/hand/model/F1.dae" scale="0.001 0.001 0.001" />
+								<!-- Standard distal  -->
+                <mesh filename="package://sr_description/hand/model/F1.dae" scale="0.001 0.001 0.001" />
               </xacro:unless>
             </xacro:unless>
@@ -86,12 +82,12 @@
       <origin xyz="0 0 0.025" rpy="0 0 0" />
       <axis xyz="1 0 0" />
-       <!-- biotac fixed distal joint -->
       <xacro:if value="${bio}">
+				<!-- biotac fixed distal joint -->
         <limit lower="${20/180*M_PI}" upper="${20/180*M_PI}" effort="10"
           velocity="1.0" />
       </xacro:if>
-      <!-- standard distal joint -->
       <xacro:unless value="${bio}">
-          <limit lower="0" upper="${M_PI/2}" effort="10"
+				<!-- standard distal joint -->
+        <limit lower="0" upper="${M_PI/2}" effort="10"
           velocity="1.0" />
       </xacro:unless>

File: sr_description/hand/xacro/finger/lfmetacarpal/lfmetacarpal.gazebo.xacro (robot description, xacro)
@@ -5,7 +5,8 @@
   <gazebo reference="${prefix}lfmetacarpal">
       <sensor type="contact" name="${prefix}lfmetacarpal_contact_sensor">
+        <always_on>true</always_on>
         <update_rate>100.0</update_rate>
         <contact>
-          <collision>${prefix}lfmetacarpal_collision_geom</collision>
+          <collision>${prefix}lfmetacarpal_geom</collision>
         </contact>
         <plugin name="${prefix}lfmetacarpal_gazebo_ros_bumper_controller" filename="libgazebo_ros_bumper.so">
@@ -16,5 +17,5 @@
         </plugin>
       </sensor>
-      <material>Gazebo/Grey</material>
+      <material>LightGrey</material>
     </gazebo>
   </xacro:macro>

File: sr_description/hand/xacro/thumb/thbase.gazebo.xacro (robot description, xacro)
@@ -5,7 +5,8 @@
   <gazebo reference="${prefix}thbase">
       <sensor type="contact" name="${prefix}thbase_contact_sensor">
+        <always_on>true</always_on>
         <update_rate>100.0</update_rate>
         <contact>
-          <collision>${prefix}thbase_collision_geom</collision>
+          <collision>${prefix}thbase_geom</collision>
         </contact>
         <plugin name="${prefix}thbase_gazebo_ros_bumper_controller" filename="libgazebo_ros_bumper.so">
@@ -16,5 +17,5 @@
         </plugin>
       </sensor>
-      <material>Gazebo/Grey</material>
+      <material>LightGrey</material>
     </gazebo>
   </xacro:macro>

File: sr_description/hand/xacro/thumb/thdistal.urdf.xacro (robot description, xacro)
@@ -15,6 +15,6 @@
   <!-- parent is the parent link for the first joint -->
   <xacro:macro name="thdistal" params="muscle bio ubi eli prefix parent">
-		<!--	BIOTAC -->
 		<xacro:if value="${bio}">
+			<!--	BIOTAC -->
 			<link name="${prefix}thbiotac_J1_dummy">
 				<inertial>
@@ -102,5 +102,4 @@
 			</joint>
 		</xacro:if>
-		 <!-- Check for other distal -->
 			<xacro:unless value="${bio}">
 				<!-- common -->
@@ -115,12 +114,11 @@
 					<origin xyz="0 0 0" rpy="0 0 0" />
 					<geometry name="${prefix}thdistal_visual">
-						<!-- Ellispoid distal  -->
 						<xacro:if value="${eli}">
+							<!-- Ellispoid distal  -->
 							<mesh filename="package://sr_description/hand/model/ellipsoids/thdistal_ellipsoid_visual.dae" scale="0.001 0.001 0.001" />
 						</xacro:if>
-						<!-- Check for uni distal -->
 						<xacro:unless value="${eli}">
-							 <!-- Ubi distal -->
 							<xacro:if value="${ubi}">
+								<!-- Ubi distal -->
 								<mesh filename="package://sr_description/hand/model/TH1_z.dae" scale="0.001 0.001 0.001" />
 							</xacro:if>
@@ -138,16 +136,15 @@
 					<origin xyz="0 0 0" rpy="0 0 0 " />
 					<geometry name="${prefix}thmiddle_collision_geom">
-					<!-- Ellispoid distal  -->
 						<xacro:if value="${eli}">
+							<!-- Ellispoid distal  -->
 						  <mesh filename="package://sr_description/hand/model/ellipsoids/thdistal_ellipsoid.dae" scale="0.001 0.001 0.001" />
 						</xacro:if>
-						<!-- Check for uni distal -->
 						<xacro:unless value="${eli}">
-							 <!-- Ubi distal -->
 							<xacro:if value="${ubi}">
+								<!-- Ubi distal -->
 								<mesh filename="package://sr_description/hand/model/TH1_z.dae" scale="0.001 0.001 0.001" />
 							</xacro:if>
-							<!-- Standard distal  -->
 							<xacro:unless value="${ubi}">
+								<!-- Standard distal  -->
 								<mesh filename="package://sr_description/hand/model/TH1_z.dae" scale="0.001 0.001 0.001" />
 							</xacro:unless>
