Commit message: Fixed dae models to use up_axis Y_UP (for OMPL to work) Collision model changed to avoid bad OMPL planning (spaces between links) Collision model now with multiple collision objects (now handled in hydro) such as cylinders and spheres to create capsules Enabled self_collision to not permit crossed fingers in gazebo

File: sr_description/hand/xacro/finger/knuckle/edc_muscle_knuckle.urdf.xacro (robot description, xacro)
@@ -24,7 +24,7 @@
       </visual>
       <collision>
-	<origin xyz="0 0 0" rpy="0 0 0" />
+	<origin xyz="0 0 0" rpy="0 1.5708 0" />
 	<geometry name="${link_prefix}knuckle_collision_geom">
-	  <box size="0.005 0.005 0.005" />
+	  <cylinder radius="0.007" length="0.014" />
 	</geometry>
       </collision>

File: sr_description/hand/xacro/finger/knuckle/knuckle.urdf.xacro (robot description, xacro)
@@ -24,7 +24,7 @@
       </visual>
       <collision>
-	<origin xyz="0 0 0" rpy="0 0 0" />
+	<origin xyz="0 0 0" rpy="0 1.5708 0" />
 	<geometry name="${link_prefix}knuckle_collision_geom">
-	  <box size="0.005 0.005 0.005" />
+	  <cylinder radius="0.007" length="0.014" />
 	</geometry>
       </collision>

File: sr_description/hand/xacro/finger/lfmetacarpal/edc_muscle_lfmetacarpal.urdf.xacro (robot description, xacro)
@@ -32,7 +32,7 @@
       </visual>
       <collision>
-          <origin xyz="0 0 0.04" rpy="0 0 0" />
+        <origin xyz="0 0 0.042" rpy="0 0 0" />
         <geometry name="lfmetacarpal_collision_geom">
-          <box size="0.008 0.008 0.03" />
+          <box size="0.018 0.024 0.048" />
         </geometry>
       </collision>

File: sr_description/hand/xacro/finger/lfmetacarpal/lfmetacarpal.urdf.xacro (robot description, xacro)
@@ -32,7 +32,7 @@
       </visual>
       <collision>
-          <origin xyz="0 0 0.04" rpy="0 0 0" />
+        <origin xyz="0 0 0.042" rpy="0 0 0" />
         <geometry name="lfmetacarpal_collision_geom">
-          <box size="0.008 0.008 0.03" />
+          <box size="0.018 0.024 0.048" />
         </geometry>
       </collision>

File: sr_description/hand/xacro/finger/middle/middle.urdf.xacro (robot description, xacro)
@@ -22,9 +22,21 @@
       <material name="Grey" />
       </visual>
+    <collision>
+        <origin xyz="0 0 0.0125" rpy="0 0 0 " />
+        <geometry name="${link_prefix}middle_collision_geom">
+          <cylinder radius="0.007" length="0.025" />
+        </geometry>
+      </collision>
       <collision>
-	<origin xyz="0 0 0.0125" rpy="0 0 0" />
-	<geometry name="${link_prefix}middle_collision_geom">
-	  <box size="0.008 0.008 0.015" />
-	</geometry>
+        <origin xyz="0 0 0.0" rpy="0 0 0 " />
+        <geometry>
+          <sphere radius="0.007" />
+        </geometry>
+      </collision>
+      <collision>
+        <origin xyz="0 0 0.025" rpy="0 0 0 " />
+        <geometry>
+          <sphere radius="0.007" />
+        </geometry>
       </collision>
     </link>
@@ -43,4 +55,5 @@
         </plugin>
       </sensor>
+       <selfCollide>true</selfCollide>
       <material>LightGrey</material>
     </gazebo>

File: sr_description/hand/xacro/finger/proximal/edc_muscle_proximal.urdf.xacro (robot description, xacro)
@@ -23,8 +23,8 @@
       </visual>
       <collision>
-	<origin xyz="0 0 0.025" rpy="0 0 0 " />
-	<geometry name="proximal_collision_geom">
-	  <box size="0.008 0.008 0.04" />
-	</geometry>
+        <origin xyz="0 0 0.025" rpy="0 0 0 " />
+        <geometry name="${link_prefix}proximal_collision_geom">
+          <cylinder radius="0.007" length="0.040" />
+        </geometry>
       </collision>
     </link>
@@ -43,4 +43,5 @@
         </plugin>
       </sensor>
+      <selfCollide>true</selfCollide>
       <material>LightGrey</material>
     </gazebo>

File: sr_description/hand/xacro/finger/proximal/proximal.urdf.xacro (robot description, xacro)
@@ -10,21 +10,21 @@
     <link name="${link_prefix}proximal">
       <inertial>
-	<mass value="0.014" />
-	<origin xyz="0 0 0.0225" />
-	<inertia  ixx="0.1" ixy="0.0"  ixz="0.0"  iyy="0.1"  iyz="0.0"
-	izz="0.0" />
+        <mass value="0.014" />
+        <origin xyz="0 0 0.0225" />
+        <inertia  ixx="0.1" ixy="0.0"  ixz="0.0"  iyy="0.1"  iyz="0.0"
+        izz="0.0" />
       </inertial>
       <visual>
-	<origin xyz="0 0 0" rpy="0 0 0" />
-	<geometry name="proximal_visual">
-      <mesh filename="package://sr_description/hand/model/F3.dae" scale="0.001 0.001 0.001" />
-      </geometry>
-      <material name="Grey" />
+      <origin xyz="0 0 0" rpy="0 0 0" />
+        <geometry name="${link_prefix}proximal_visual">
+          <mesh filename="package://sr_description/hand/model/F3.dae" scale="0.001 0.001 0.001" />
+        </geometry>
+        <material name="Grey" />
       </visual>
       <collision>
-	<origin xyz="0 0 0.025" rpy="0 0 0 " />
-	<geometry name="proximal_collision_geom">
-	  <box size="0.008 0.008 0.04" />
-	</geometry>
+        <origin xyz="0 0 0.025" rpy="0 0 0 " />
+        <geometry name="${link_prefix}proximal_collision_geom">
+          <cylinder radius="0.007" length="0.040" />
+        </geometry>
       </collision>
     </link>
@@ -43,4 +43,5 @@
         </plugin>
       </sensor>
+       <selfCollide>true</selfCollide>
       <material>LightGrey</material>
     </gazebo>

File: sr_description/hand/xacro/palm/edc_muscle_palm.urdf.xacro (robot description, xacro)
@@ -31,10 +31,22 @@
 	<material name="Grey"/>
       </visual>
-      <collision>
-	<origin xyz="0.005 0 0.035" rpy="0 0 0" />
+        <collision>
+	<origin xyz="0.011 0 0.038" rpy="0 0 0" />
 	<geometry name="palm_collision_geom">
-	  <box size="0.05 0.02 0.07" />
+	  <box size="0.062 0.024 0.098" />
 	</geometry>
-      </collision>
+    </collision>
+    <collision>
+      <origin xyz="0.011 0 0.089" rpy="0 0 0" />
+	    <geometry>
+        <box size="0.018 0.024 0.004" />
+      </geometry>
+    </collision>
+    <collision>
+      <origin xyz="-0.030 0 0.009" rpy="0 0 0" />
+	    <geometry>
+        <box size="0.020 0.024 0.040" />
+      </geometry>
+    </collision>
     </link>
     <gazebo reference="palm">

File: sr_description/hand/xacro/palm/palm.urdf.xacro (robot description, xacro)
@@ -32,9 +32,21 @@
       </visual>
       <collision>
-	<origin xyz="0.005 0 0.035" rpy="0 0 0" />
+	<origin xyz="0.011 0 0.038" rpy="0 0 0" />
 	<geometry name="palm_collision_geom">
-	  <box size="0.05 0.02 0.07" />
+	  <box size="0.062 0.024 0.098" />
 	</geometry>
-      </collision>
+    </collision>
+    <collision>
+      <origin xyz="0.011 0 0.089" rpy="0 0 0" />
+	    <geometry>
+        <box size="0.018 0.024 0.004" />
+      </geometry>
+    </collision>
+    <collision>
+      <origin xyz="-0.030 0 0.009" rpy="0 0 0" />
+	    <geometry>
+        <box size="0.020 0.024 0.040" />
+      </geometry>
+    </collision>
     </link>
     <gazebo reference="palm">

File: sr_description/hand/xacro/thumb/thbase.urdf.xacro (robot description, xacro)
@@ -34,9 +34,9 @@
 	</material>
       </visual>
-      <collision>
-	<origin xyz="0 0 0" rpy="0 0 0 " />
+       <collision>
+        <origin xyz="0 0 0.0" rpy="0 0 0 " />
 	<geometry name="thbase_collision_geom">
-	  <box size="0.001 0.001 0.001" />
-	</geometry>
+          <sphere radius="0.011" />
+        </geometry>
       </collision>
     </link>
@@ -55,4 +55,5 @@
         </plugin>
       </sensor>
+       <selfCollide>false</selfCollide>
       <material>LightGrey</material>
     </gazebo>

File: sr_description/hand/xacro/thumb/thhub.urdf.xacro (robot description, xacro)
@@ -24,9 +24,9 @@
 	</material>
       </visual>
-      <collision>
-	<origin xyz="0 0 0" rpy="0 0 0 " />
-	<geometry name="thhub_collision_geom">
-	  <box size="0.001 0.001 0.001" />
-	</geometry>
+            <collision>
+        <origin xyz="0 0 0.0" rpy="0 0 0 " />
+       <geometry name="thhub_collision_geom">
+          <sphere radius="0.010" />
+        </geometry>
       </collision>
     </link>
@@ -45,4 +45,5 @@
         </plugin>
       </sensor>
+       <selfCollide>true</selfCollide>
       <material>LightGrey</material>
     </gazebo>

File: sr_description/hand/xacro/thumb/thmiddle.urdf.xacro (robot description, xacro)
@@ -25,8 +25,14 @@
       </visual>
       <collision>
-	<origin xyz="0 0 0.016" rpy="0 0 0 " />
-	<geometry name="thmiddle_collision_geom">
-	  <box size="0.008 0.008 0.015" />
-	</geometry>
+        <origin xyz="0 0 0.016" rpy="0 0 0 " />
+        <geometry name="thmiddle_collision_geom">
+          <cylinder radius="0.011" length="0.031" />
+        </geometry>
+      </collision>
+      <collision>
+        <origin xyz="0 0 0.032" rpy="0 0 0 " />
+        <geometry>
+          <sphere radius="0.010" />
+        </geometry>
       </collision>
     </link>
@@ -45,4 +51,5 @@
         </plugin>
       </sensor>
+      <selfCollide>true</selfCollide>
       <material>LightGrey</material>
     </gazebo>

File: sr_description/hand/xacro/thumb/thproximal.urdf.xacro (robot description, xacro)
@@ -33,9 +33,9 @@
 	</material>
       </visual>
-      <collision>
-	<origin xyz="0 0 0.019" rpy="0 0 0" />
-	<geometry name="thproximal_collision_geom">
-	  <box size="0.008 0.008 0.020" />
-	</geometry>
+       <collision>
+        <origin xyz="0 0 0.020" rpy="0 0 0 " />
+        <geometry name="thproximal_collision_geom">
+          <cylinder radius="0.012" length="0.018" />
+        </geometry>
       </collision>
     </link>
@@ -54,4 +54,5 @@
         </plugin>
       </sensor>
+       <selfCollide>false</selfCollide>
       <material>LightGrey</material>
     </gazebo>

File: sr_description/hand/xacro/wrist/wrist.urdf.xacro (robot description, xacro)
@@ -31,7 +31,31 @@
       </visual>
       <collision>
-	<origin xyz="0 0 0" rpy="0 0 0" />
+	<origin xyz="0 0 0" rpy="1.5708 1.5708 0 " />
 	<geometry name="wrist_collision_geom">
-	  <box size="0.02 0.02 0.02" />
+	  <cylinder radius="0.0135" length="0.030" />
+	</geometry>
+      </collision>
+      <collision>
+	<origin xyz="-0.026 0 0.034" rpy="0 1.5708 0" />
+	<geometry>
+	 <cylinder radius="0.011" length="0.010" />
+	</geometry>
+      </collision>
+      <collision>
+	<origin xyz="0.031 0 0.034" rpy="0 1.5708 0" />
+	<geometry>
+	 <cylinder radius="0.011" length="0.010" />
+	</geometry>
+      </collision>
+       <collision>
+	<origin xyz="-0.021 0 0.011" rpy="0 0.7854 0" />
+	<geometry>
+	  <box size="0.027 0.018 0.010" />
+	</geometry>
+      </collision>
+      <collision>
+	<origin xyz="0.026 0 0.010" rpy="0 -0.7854 0" />
+	<geometry>
+	  <box size="0.027 0.018 0.010" />
 	</geometry>
       </collision>
