Commit message: Fixed dae models to use up_axis Y_UP (for OMPL to work) Collision model changed to avoid bad OMPL planning (spaces between links) Collision model now with multiple collision objects (now handled in hydro) such as cylinders and spheres to create capsules Enabled self_collision to not permit crossed fingers in gazebo Additional non-adjacent self-collision fix for metacarpal and proximal

File: sr_description/hand/xacro/finger/knuckle/knuckle.urdf.xacro (robot description, xacro)
@@ -29,7 +29,7 @@
       </visual>
       <collision>
-        <origin xyz="0 0 0" rpy="0 0 0" />
+        <origin xyz="0 0 0" rpy="0 1.5708 0" />
         <geometry name="${prefix}${link_prefix}knuckle_collision_geom">
-          <box size="0.005 0.005 0.005" />
+          <cylinder radius="0.007" length="0.014" />
         </geometry>
       </collision>

File: sr_description/hand/xacro/finger/lfmetacarpal/lfmetacarpal.gazebo.xacro (robot description, xacro)
@@ -18,4 +18,5 @@
         </plugin>
       </sensor>
+      <selfCollide>true</selfCollide>
       <material>LightGrey</material>
     </gazebo>

File: sr_description/hand/xacro/finger/lfmetacarpal/lfmetacarpal.urdf.xacro (robot description, xacro)
@@ -28,7 +28,7 @@
       </visual>
       <collision>
-        <origin xyz="0 0 0.04" rpy="0 0 0" />
+        <origin xyz="0 0 0.038" rpy="0 0 0" />
         <geometry name="${prefix}lfmetacarpal_collision_geom">
-          <box size="0.008 0.008 0.03" />
+          <box size="0.018 0.024 0.040" />
         </geometry>
       </collision>

File: sr_description/hand/xacro/finger/middle/middle.urdf.xacro (robot description, xacro)
@@ -28,8 +28,20 @@
         <material name="Grey" />
       </visual>
+    <collision>
+      <origin xyz="0 0 0.0125" rpy="0 0 0 " />
+        <geometry name="${prefix}${link_prefix}middle_collision_geom">
+          <cylinder radius="0.007" length="0.025" />
+        </geometry>
+      </collision>
       <collision>
-        <origin xyz="0 0 0.0125" rpy="0 0 0" />
-        <geometry name="${prefix}${link_prefix}middle_collision_geom">
-          <box size="0.008 0.008 0.015" />
+        <origin xyz="0 0 0.0" rpy="0 0 0 " />
+        <geometry>
+          <sphere radius="0.007" />
+        </geometry>
+      </collision>
+      <collision>
+        <origin xyz="0 0 0.025" rpy="0 0 0 " />
+        <geometry>
+          <sphere radius="0.007" />
         </geometry>
       </collision>

File: sr_description/hand/xacro/finger/proximal/proximal.urdf.xacro (robot description, xacro)
@@ -22,5 +22,5 @@
       </inertial>
       <visual>
-        <origin xyz="0 0 0" rpy="0 0 0" />
+      <origin xyz="0 0 0" rpy="0 0 0" />
         <geometry name="${prefix}${link_prefix}proximal_visual">
           <mesh filename="package://sr_description/hand/model/F3.dae" scale="0.001 0.001 0.001" />
@@ -31,5 +31,5 @@
         <origin xyz="0 0 0.025" rpy="0 0 0 " />
         <geometry name="${prefix}${link_prefix}proximal_collision_geom">
-          <box size="0.008 0.008 0.04" />
+          <cylinder radius="0.007" length="0.040" />
         </geometry>
       </collision>

File: sr_description/hand/xacro/palm/palm.urdf.xacro (robot description, xacro)
@@ -28,8 +28,20 @@
       </visual>
       <collision>
-        <origin xyz="${reflect*0.005} 0 0.035" rpy="0 0 0" />
+        <origin xyz="${reflect*0.011} 0 0.038" rpy="0 0 0" />
         <geometry name="${prefix}palm_collision_geom">
-          <box size="0.05 0.02 0.07" />
+          <box size="0.062 0.024 0.098" />
         </geometry>
+      </collision>
+      <collision>
+        <origin xyz="${reflect*0.011} 0 0.089" rpy="0 0 0" />
+        <geometry>
+          <box size="0.018 0.024 0.004" />
+        </geometry>
+      </collision>
+      <collision>
+        <origin xyz="${reflect*-0.030} 0 0.009" rpy="0 0 0" />
+	      <geometry>
+            <box size="0.020 0.024 0.040" />
+          </geometry>
       </collision>
     </link>

File: sr_description/hand/xacro/thumb/thbase.gazebo.xacro (robot description, xacro)
@@ -18,4 +18,5 @@
         </plugin>
       </sensor>
+      <selfCollide>false</selfCollide>
       <material>LightGrey</material>
     </gazebo>

File: sr_description/hand/xacro/thumb/thbase.urdf.xacro (robot description, xacro)
@@ -20,18 +20,18 @@
 			</inertial>
       <visual>
-				<origin xyz="0 0 0" rpy="0 0 0" />
-				<geometry name="${prefix}thbase_visual">
-					<box size="0.001 0.001 0.001" />
-				</geometry>
-				<material name="shadow_thbase_material">
-					<color rgba="0.5 0.5 0.5 1.0"/>
-				</material>
+        <origin xyz="0 0 0" rpy="0 0 0" />
+        <geometry name="${prefix}thbase_visual">
+          <box size="0.001 0.001 0.001" />
+        </geometry>
+        <material name="shadow_thbase_material">
+          <color rgba="0.5 0.5 0.5 1.0"/>
+        </material>
       </visual>
       <collision>
-				<origin xyz="0 0 0" rpy="0 0 0 " />
-				<geometry name="${prefix}thbase_collision_geom">
-					<box size="0.001 0.001 0.001" />
-				</geometry>
-			</collision>
+        <origin xyz="0 0 0" rpy="0 0 0 " />
+        <geometry name="${prefix}thbase_collision_geom">
+          <sphere radius="0.011" />
+        </geometry>
+      </collision>
     </link>
     <joint name="${prefix}THJ5" type="revolute">

File: sr_description/hand/xacro/thumb/thhub.gazebo.xacro (robot description, xacro)
@@ -18,4 +18,5 @@
         </plugin>
       </sensor>
+      <selfCollide>true</selfCollide>
       <material>LightGrey</material>
     </gazebo>

File: sr_description/hand/xacro/thumb/thhub.urdf.xacro (robot description, xacro)
@@ -30,8 +30,8 @@
       </visual>
       <collision>
-				<origin xyz="0 0 0" rpy="0 0 0 " />
-				<geometry name="${prefix}thhub_collision_geom">
-					<box size="0.001 0.001 0.001" />
-				</geometry>
+        <origin xyz="0 0 0" rpy="0 0 0 " />
+        <geometry name="${prefix}thhub_collision_geom">
+          <sphere radius="0.010" />
+        </geometry>
       </collision>
     </link>

File: sr_description/hand/xacro/thumb/thmiddle.gazebo.xacro (robot description, xacro)
@@ -18,4 +18,5 @@
         </plugin>
       </sensor>
+      <selfCollide>true</selfCollide>
       <material>LightGrey</material>
     </gazebo>

File: sr_description/hand/xacro/thumb/thmiddle.urdf.xacro (robot description, xacro)
@@ -15,37 +15,44 @@
     <link name="${prefix}thmiddle">
       <inertial>
-				<mass value="0.027" />
-				<origin xyz="0 0 0.016" rpy="0 0 0"/>
-				<inertia  ixx="0.0026" ixy="0.0"  ixz="0.0"  iyy="0.0026"  iyz="0.0"
-				izz="0.000169" />
+        <mass value="0.027" />
+        <origin xyz="0 0 0.016" rpy="0 0 0"/>
+          <inertia  ixx="0.0026" ixy="0.0"  ixz="0.0"  iyy="0.0026"  iyz="0.0" izz="0.000169" />
       </inertial>
       <visual>
-				<origin xyz="0 0 0" rpy="0 0 0" />
-					<xacro:if value="${bio}">
-						<geometry name="${prefix}thmiddle_visual">
-						  <mesh filename="package://sr_description/hand/model/biotacs/biotac_thumb_adapter.dae" scale="0.001 0.001 0.001" />
-						</geometry>
-						 <material name="BiotacGreen" />
-					</xacro:if>
-					<xacro:unless value="${bio}">
-						<geometry name="${prefix}thmiddle_visual">
-							<mesh filename="package://sr_description/hand/model/TH2_z.dae" scale="0.001 0.001 0.001" />
-						</geometry>
-						<material name="shadow_thmiddle_material">
-							<color rgba="0.2 0.2 0.2 1.0"/>
-						</material>
-					</xacro:unless>
+        <origin xyz="0 0 0" rpy="0 0 0" />
+        <xacro:if value="${bio}">
+        <geometry name="${prefix}thmiddle_visual">
+          <mesh filename="package://sr_description/hand/model/biotacs/biotac_thumb_adapter.dae" scale="0.001 0.001 0.001" />
+        </geometry>
+        <material name="BiotacGreen" />
+        </xacro:if>
+        <xacro:unless value="${bio}">
+        <geometry name="${prefix}thmiddle_visual">
+          <mesh filename="package://sr_description/hand/model/TH2_z.dae" scale="0.001 0.001 0.001" />
+        </geometry>
+        <material name="shadow_thmiddle_material">
+          <color rgba="0.2 0.2 0.2 1.0"/>
+        </material>
+        </xacro:unless>
       </visual>
       <collision>
-				<origin xyz="0 0 0.016" rpy="0 0 0 " />
-				<geometry name="${prefix}thmiddle_collision_geom">
-					 <xacro:if value="${bio}">
-						  <box size="0.008 0.008 0.01" />
-					</xacro:if>
-					<xacro:unless value="${bio}">
-							<box size="0.008 0.008 0.015" />
-					</xacro:unless>
-				</geometry>
+        <origin xyz="0 0 0.016" rpy="0 0 0 " />
+        <geometry name="${prefix}thmiddle_collision_geom">
+          <xacro:if value="${bio}">
+            <box size="0.008 0.008 0.01" />
+          </xacro:if>
+          <xacro:unless value="${bio}">
+            <cylinder radius="0.011" length="0.031" />
+          </xacro:unless>
+        </geometry>
       </collision>
+      <xacro:unless value="${bio}">
+      <collision>
+        <origin xyz="0 0 0.032" rpy="0 0 0 " />
+        <geometry>
+          <sphere radius="0.010" />
+        </geometry>
+      </collision>
+      </xacro:unless>
     </link>
     <joint name="${prefix}THJ2" type="revolute">

File: sr_description/hand/xacro/thumb/thproximal.gazebo.xacro (robot description, xacro)
@@ -18,4 +18,5 @@
         </plugin>
       </sensor>
+      <selfCollide>false</selfCollide>
       <material>LightGrey</material>
     </gazebo>

File: sr_description/hand/xacro/thumb/thproximal.urdf.xacro (robot description, xacro)
@@ -21,17 +21,17 @@
 			</inertial>
       <visual>
-				<origin xyz="0 0 0" rpy="0 0 0" />
-				<geometry name="${prefix}thproximal_visual">
-					<mesh filename="package://sr_description/hand/model/TH3_z.dae" scale="0.001 0.001 0.001" />
-				</geometry>
-				<material name="shadow_thproximal_material">
-					<color rgba="0.2 0.2 0.2 1.0"/>
-				</material>
+        <origin xyz="0 0 0" rpy="0 0 0" />
+        <geometry name="${prefix}thproximal_visual">
+          <mesh filename="package://sr_description/hand/model/TH3_z.dae" scale="0.001 0.001 0.001" />
+        </geometry>
+        <material name="shadow_thproximal_material">
+          <color rgba="0.2 0.2 0.2 1.0"/>
+        </material>
       </visual>
       <collision>
-				<origin xyz="0 0 0.019" rpy="0 0 0" />
-				<geometry name="${prefix}thproximal_collision_geom">
-					<box size="0.008 0.008 0.020" />
-				</geometry>
+        <origin xyz="0 0 0.020" rpy="0 0 0" />
+        <geometry name="${prefix}thproximal_collision_geom">
+          <cylinder radius="0.012" length="0.018" />
+        </geometry>
       </collision>
     </link>

File: sr_description/hand/xacro/wrist/wrist.urdf.xacro (robot description, xacro)
@@ -21,8 +21,32 @@
       </visual>
       <collision>
-		  <origin xyz="0 0 0" rpy="0 0 0" />
-		  <geometry name="${prefix}wrist_collision_geom">
-			 <box size="0.02 0.02 0.02" />
-		  </geometry>
+        <origin xyz="0 0 0" rpy="1.5708 1.5708 0 " />
+        <geometry name="${prefix}wrist_collision_geom">
+          <cylinder radius="0.0135" length="0.030" />
+        </geometry>
+      </collision>
+      <collision>
+        <origin xyz="${reflect*-0.026} 0 0.034" rpy="0 1.5708 0" />
+        <geometry>
+          <cylinder radius="0.011" length="0.010" />
+        </geometry>
+      </collision>
+      <collision>
+        <origin xyz="${reflect*0.031} 0 0.034" rpy="0 1.5708 0" />
+        <geometry>
+          <cylinder radius="0.011" length="0.010" />
+        </geometry>
+      </collision>
+      <collision>
+        <origin xyz="${reflect*-0.021} 0 0.011" rpy="0 ${reflect*0.7854} 0" />
+        <geometry>
+          <box size="0.027 0.018 0.010" />
+        </geometry>
+      </collision>
+      <collision>
+        <origin xyz="${reflect*0.026} 0 0.010" rpy="0 ${reflect*-0.7854} 0" />
+        <geometry>
+          <box size="0.027 0.018 0.010" />
+        </geometry>
       </collision>
     </link>

Commit message: Fix inertia, limits, and dynamic damping on the URDFs for the motor hand.

File: sr_description/hand/xacro/finger/knuckle/knuckle.urdf.xacro (robot description, xacro)
@@ -12,7 +12,6 @@
 	<origin xyz="0 0 0" rpy="0 0 0" />
 	<!--<insert_block name="origin" /> -->
-	<mass value="0.008" />
-	<inertia  ixx="0.0" ixy="0.0"  ixz="0.0"  iyy="0.1"  iyz="0.0"
-	izz="0.0" />
+	<mass value="0.08" />
+	<inertia ixx="0.0026" ixy="0.0" ixz="0.0" iyy="0.0026" iyz="0.0" izz="0.0032" />
       </inertial>
       <visual>
@@ -53,6 +52,6 @@
       <insert_block name="axis"/>
       <limit lower="-0.3491" upper="0.3491"
-      effort="1000.0" velocity="10.0"/>
-      <dynamics damping="10.0"/>
+      effort="2" velocity="1.0"/>
+      <dynamics damping="0.1"/>
     </joint>
     <xacro:knuckle_transmission />

File: sr_description/hand/xacro/finger/lfmetacarpal/lfmetacarpal.urdf.xacro (robot description, xacro)
@@ -21,6 +21,6 @@
       <inertial>
         <origin xyz="0 0 0.04" rpy="0 0 0" />
-	    <mass value="0.075" />
-	    <inertia  ixx="0.1" ixy="0.0"  ixz="0.0"  iyy="0.1"  iyz="0.0" izz="0.1" />
+	    <mass value="0.030" />
+	    <inertia ixx="0.00545" ixy="0.0" ixz="0.0" iyy="0.0056352" iyz="0.0" izz="0.0004272" />
       </inertial>
       <visual>
@@ -60,7 +60,7 @@
       <origin xyz="${reflect*-0.033} 0 0.02071" rpy="0 0 0" />
       <axis xyz="0.573576436 0 ${reflect*0.819152044}" />
-      <limit lower="0" upper="0.785398163" effort="1000.0"
-      velocity="10.0" />
-      <dynamics damping="10.0"/>
+      <limit lower="0" upper="${45/180*M_PI}" effort="2"
+      velocity="1.0" />
+      <dynamics damping="0.1"/>
     </joint>
     <xacro:lfmetacarpal_transmission />

File: sr_description/hand/xacro/finger/middle/middle.urdf.xacro (robot description, xacro)
@@ -11,7 +11,6 @@
       <inertial>
 	<origin xyz="0 0 0.0125" rpy="0 0 0" />
-	<mass value="0.012" />
-	<inertia  ixx="0.1" ixy="0.0"  ixz="0.0"  iyy="0.1"  iyz="0.0"
-	izz="0.0" />
+	<mass value="0.020" />
+	<inertia ixx="0.002" ixy="0.0" ixz="0.0" iyy="0.002" iyz="0.0" izz="0.0002" />
       </inertial>
       <visual>
@@ -63,7 +62,7 @@
       <origin xyz="0 0 0.045" rpy="0 0 0" />
       <axis xyz="1 0 0" />
-      <limit lower="0" upper="${M_PI/2}" effort="1000.0"
-      velocity="10.0" />
-      <dynamics damping="10.0"/>
+      <limit lower="0" upper="${M_PI/2}" effort="2"
+      velocity="1.0" />
+      <dynamics damping="0.1"/>
     </joint>
     <xacro:middle_transmission />

File: sr_description/hand/xacro/finger/proximal/proximal.urdf.xacro (robot description, xacro)
@@ -10,8 +10,7 @@
     <link name="${link_prefix}proximal">
       <inertial>
-        <mass value="0.014" />
+        <mass value="0.030" />
         <origin xyz="0 0 0.0225" />
-        <inertia  ixx="0.1" ixy="0.0"  ixz="0.0"  iyy="0.1"  iyz="0.0"
-        izz="0.0" />
+        <inertia ixx="0.003" ixy="0.0" ixz="0.0" iyy="0.003" iyz="0.0" izz="0.0003" />
       </inertial>
       <visual>
@@ -51,7 +50,7 @@
       <origin xyz="0 0 0" rpy="0 0 0" />
       <axis xyz="1 0 0" />
-      <limit lower="0" upper="${M_PI/2}" effort="1000.0"
-      velocity="10.0"/>
-      <dynamics damping="10.0"/>
+      <limit lower="0" upper="${M_PI/2}" effort="2"
+      velocity="1.0"/>
+      <dynamics damping="0.1"/>
     </joint>
     <xacro:proximal_transmission />

File: sr_description/hand/xacro/palm/palm.urdf.xacro (robot description, xacro)
@@ -22,5 +22,5 @@
 	<origin xyz="0 0 0.035" rpy="0 0 0" />
 	<mass value="0.3" />
-	<inertia  ixx="0.5" ixy="0.0"  ixz="0.0"  iyy="0.5"  iyz="0.0"	izz="0.3" />
+	<inertia ixx="0.003581" ixy="0.0" ixz="0.0" iyy="0.005287" iyz="0.0" izz="0.002545" />
       </inertial>
       <visual>
@@ -71,7 +71,7 @@
       <origin xyz="0 0 0.034" rpy="0 0 0" />
       <axis xyz="1 0 0" />
-      <limit lower="-0.7854" upper="0.5236"
-      effort="1000.0" velocity="10.0"/>
-      <dynamics damping="30.0"/>
+      <limit lower="${-40/180*M_PI}" upper="${28/180*M_PI}"
+      effort="30" velocity="1.0"/>
+      <dynamics damping="0.1"/>
     </joint>
     <xacro:shadowhand_palm_transmission />

File: sr_description/hand/xacro/thumb/thbase.urdf.xacro (robot description, xacro)
@@ -22,6 +22,5 @@
 	<mass value="0.010" />
 	  <origin xyz="0 0 0" rpy="0 0 0"/>
-	<inertia  ixx="0.0" ixy="0.0"  ixz="0.0"  iyy="0.0"  iyz="0.0"
-	izz="0.1" />
+	<inertia ixx="0.0003" ixy="0.0" ixz="0.0" iyy="0.0003" iyz="0.0" izz="0.0003" />
       </inertial>
       <visual>
@@ -63,7 +62,7 @@
       <origin xyz="${reflect*0.034} -0.0085 0.029" rpy="0 ${M_PI/4} ${joint_yaw}" />
       <axis xyz="0 0 ${reflect*-1}" />
-      <limit lower="-1.047" upper="1.047" effort="1000.0"
-      velocity="10.0" />
-      <dynamics damping="10.0"/>
+      <limit lower="${-60/180*M_PI}" upper="${60/180*M_PI}" effort="10"
+      velocity="1.0" />
+      <dynamics damping="0.1"/>
     </joint>
     <xacro:thbase_transmission />

File: sr_description/hand/xacro/thumb/thhub.urdf.xacro (robot description, xacro)
@@ -10,8 +10,7 @@
     <link name="thhub">
       <inertial>
-	<mass value="0.002" />
+	<mass value="0.01" />
 	<origin xyz="0 0 0" rpy="0 0 0"/>
-	<inertia  ixx="0.1" ixy="0.0"  ixz="0.0"  iyy="0.1"  iyz="0.0"
-	izz="0.1" />
+	<inertia ixx="0.0003" ixy="0.0" ixz="0.0" iyy="0.0003" iyz="0.0" izz="0.0003" />
       </inertial>
       <visual>
@@ -53,7 +52,6 @@
       <origin xyz="0 0 0.038" rpy="0 0 0" />
       <axis xyz="1 0 0" />
-      <limit lower="-0.2618" upper="0.2618" effort="1000.0"
-      velocity="10.0" />
-      <dynamics damping="10.0"/>
+      <limit lower="${-12/180*M_PI}" upper="${12/180*M_PI}" effort="10" velocity="1.0" />
+      <dynamics damping="0.1"/>
     </joint>
     <xacro:thhub_transmission />

File: sr_description/hand/xacro/thumb/thmiddle.urdf.xacro (robot description, xacro)
@@ -10,8 +10,7 @@
     <link name="thmiddle">
       <inertial>
-	<mass value="0.016" />
+	<mass value="0.027" />
 	<origin xyz="0 0 0.016" rpy="0 0 0"/>
-	<inertia  ixx="0.1" ixy="0.0"  ixz="0.0"  iyy="0.1"  iyz="0.0"
-	izz="0.1" />
+	<inertia ixx="0.0026" ixy="0.0" ixz="0.0" iyy="0.0026" iyz="0.0" izz="0.000169" />
       </inertial>
       <visual>
@@ -59,7 +58,6 @@
       <origin xyz="0 0 0" rpy="0 0 0" />
       <axis xyz="0 -1 0" />
-      <limit lower="-0.6981" upper="0.6981" effort="1000.0"
-      velocity="10.0" />
-      <dynamics damping="10.0"/>
+      <limit lower="${-40/180*M_PI}" upper="${40/180*M_PI}" effort="10" velocity="1.0" />
+      <dynamics damping="0.1"/>
     </joint>
     <xacro:thmiddle_transmission />

File: sr_description/hand/xacro/thumb/thproximal.urdf.xacro (robot description, xacro)
@@ -20,7 +20,7 @@
     <link name="thproximal">
       <inertial>
-	<mass value="0.016" />
+	<mass value="0.040" />
 	<origin xyz="0 0 0.019" rpy="0 0 0"/>
-	<inertia  ixx="0.1" ixy="0.0"  ixz="0.0"  iyy="0.1"  iyz="0.0"	izz="0.1" />
+	<inertia ixx="0.00496" ixy="0.0" ixz="0.0" iyy="0.00496" iyz="0.0" izz="0.000312" />
       </inertial>
       <visual>
@@ -62,7 +62,6 @@
       <origin xyz="0 0 0" rpy="0 0 0" />
       <axis xyz="${reflect*1} 0 0" />
-      <limit lower="0" upper="1.309" effort="1000.0"
-      velocity="10.0" />
-      <dynamics damping="10.0"/>
+      <limit lower="0" upper="${70/180*M_PI}" effort="10" velocity="1.0" />
+      <dynamics damping="0.1"/>
     </joint>
     <xacro:thproximal_transmission />

File: sr_description/hand/xacro/wrist/wrist.urdf.xacro (robot description, xacro)
@@ -21,5 +21,5 @@
 	<!--<insert_block name="origin" />-->
 	<mass value="0.1" />
-	<inertia  ixx="0.120" ixy="0.0"  ixz="0.0"  iyy="0.148"  iyz="0.0" izz="0.0438" />
+	<inertia ixx="0.0120" ixy="0.0" ixz="0.0" iyy="0.0148" iyz="0.0" izz="0.00438" />
       </inertial>
       <visual>
@@ -71,6 +71,6 @@
       <insert_block name="origin" />
       <axis xyz="0 1 0" />
-      <limit lower="-0.52359877559829882" upper="0.17453292519943295" effort="1000.0" velocity="10.0"/>
-      <dynamics damping="30.0"/>
+      <limit lower="${-30/180*M_PI}" upper="${10/180*M_PI}" effort="30" velocity="1.0"/>
+      <dynamics damping="0.1"/>
     </joint>
     <xacro:shadowhand_wrist_transmission />
