Commit message: Working J0 using RQT plugin and Gazebo

File: sr_description/hand/xacro/finger/knuckle/knuckle.transmission.xacro (robot description, xacro)
@@ -19,8 +19,12 @@
     <!-- motor hand -->
     <xacro:unless value="${muscletrans}">
-      <transmission type="sr_mechanism_model/SimpleTransmission" name="${prefix}${link_prefix}knuckle_transmission">
-      <actuator name="${prefix}${joint_prefix}J4" />
-      <joint name="${prefix}${joint_prefix}J4" />
-      <mechanicalReduction>1</mechanicalReduction>
+      <transmission name="${prefix}${link_prefix}knuckle_transmission">
+        <type>sr_mechanism_model/SimpleTransmission</type>
+      <actuator name="${prefix}${joint_prefix}J4">
+        <mechanicalReduction>1</mechanicalReduction>
+      </actuator>
+      <joint name="${prefix}${joint_prefix}J4">
+        <hardwareInterface>EffortJointInterface</hardwareInterface>
+      </joint>
       </transmission>
     </xacro:unless>

File: sr_description/hand/xacro/finger/lfmetacarpal/lfmetacarpal.transmission.xacro (robot description, xacro)
@@ -17,8 +17,12 @@
     <!-- motor hand -->
     <xacro:unless value="${muscletrans}">
-      <transmission type="sr_mechanism_model/SimpleTransmission" name="${prefix}lfmetacarpal_transmission">
-      <actuator name="${prefix}LFJ5" />
-      <joint name="${prefix}LFJ5" />
-      <mechanicalReduction>1</mechanicalReduction>
+      <transmission name="${prefix}lfmetacarpal_transmission">
+        <type>sr_mechanism_model/SimpleTransmission</type>
+      <actuator name="${prefix}LFJ5">
+        <mechanicalReduction>1</mechanicalReduction>
+      </actuator>
+      <joint name="${prefix}LFJ5">
+        <hardwareInterface>EffortJointInterface</hardwareInterface>
+      </joint>
       </transmission>
     </xacro:unless>

File: sr_description/hand/xacro/finger/middle/middle.transmission.xacro (robot description, xacro)
@@ -20,9 +20,12 @@
     <!-- motor hand -->
     <xacro:unless value="${muscletrans}">
-      <transmission type="sr_mechanism_model/J0Transmission" name="${prefix}${link_prefix}middle_transmission">
-      <actuator name="${prefix}${joint_prefix}J0" />
-      <joint name="${prefix}${joint_prefix}J1" />
-      <joint name="${prefix}${joint_prefix}J2" />
-      <mechanicalReduction>1</mechanicalReduction>
+      <transmission name="${prefix}${link_prefix}middle_transmission">
+        <type>sr_mechanism_model/J0Transmission</type>
+        <actuator name="${prefix}${joint_prefix}J0">
+          <mechanicalReduction>1</mechanicalReduction>
+        </actuator>
+        <joint name="${prefix}${joint_prefix}J1">
+          <hardwareInterface>EffortJointInterface</hardwareInterface>
+        </joint>
       </transmission>
     </xacro:unless>

File: sr_description/hand/xacro/finger/proximal/proximal.transmission.xacro (robot description, xacro)
@@ -19,8 +19,12 @@
     <!-- motor hand -->
     <xacro:unless value="${muscletrans}">
-      <transmission type="sr_mechanism_model/SimpleTransmission" name="${prefix}${link_prefix}proximal_transmission">
-      <actuator name="${prefix}${joint_prefix}J3" />
-      <joint name="${prefix}${joint_prefix}J3" />
-      <mechanicalReduction>1</mechanicalReduction>
+      <transmission name="${prefix}${link_prefix}proximal_transmission">
+        <type>sr_mechanism_model/SimpleTransmission</type>
+      <actuator name="${prefix}${joint_prefix}J3">
+        <mechanicalReduction>1</mechanicalReduction>
+      </actuator>
+      <joint name="${prefix}${joint_prefix}J3">
+        <hardwareInterface>EffortJointInterface</hardwareInterface>
+      </joint>
       </transmission>
     </xacro:unless>

File: sr_description/hand/xacro/palm/palm.transmission.xacro (robot description, xacro)
@@ -17,8 +17,12 @@
     <!-- motor hand -->
     <xacro:unless value="${muscletrans}">
-      <transmission type="sr_mechanism_model/SimpleTransmission" name="${prefix}palm_transmission">
-      <actuator name="${prefix}WRJ1" />
-      <joint name="${prefix}WRJ1" />
-      <mechanicalReduction>1</mechanicalReduction>
+      <transmission name="${prefix}palm_transmission">
+        <type>sr_mechanism_model/SimpleTransmission</type>
+      <actuator name="${prefix}WRJ1">
+        <mechanicalReduction>1</mechanicalReduction>
+      </actuator>
+      <joint name="${prefix}WRJ1">
+        <hardwareInterface>EffortJointInterface</hardwareInterface>
+      </joint>
       </transmission>
     </xacro:unless>

File: sr_description/hand/xacro/thumb/thbase.transmission.xacro (robot description, xacro)
@@ -17,8 +17,12 @@
     <!-- motor hand -->
     <xacro:unless value="${muscletrans}">
-      <transmission type="sr_mechanism_model/SimpleTransmission" name="${prefix}thbase_transmission">
-      <actuator name="${prefix}THJ5" />
-      <joint name="${prefix}THJ5" />
-      <mechanicalReduction>1</mechanicalReduction>
+      <transmission name="${prefix}thbase_transmission">
+        <type>sr_mechanism_model/SimpleTransmission</type>
+        <actuator name="${prefix}THJ5">
+          <mechanicalReduction>1</mechanicalReduction>
+        </actuator>
+        <joint name="${prefix}THJ5">
+          <hardwareInterface>EffortJointInterface</hardwareInterface>
+        </joint>
       </transmission>
     </xacro:unless>

File: sr_description/hand/xacro/thumb/thdistal.transmission.xacro (robot description, xacro)
@@ -17,8 +17,12 @@
     <!-- motor hand -->
     <xacro:unless value="${muscletrans}">
-      <transmission type="sr_mechanism_model/SimpleTransmission" name="${prefix}thdistal_transmission">
-      <actuator name="${prefix}THJ1" />
-      <joint name="${prefix}THJ1" />
-      <mechanicalReduction>1</mechanicalReduction>
+      <transmission name="${prefix}thdistal_transmission">
+        <type>sr_mechanism_model/SimpleTransmission</type>
+        <actuator name="${prefix}THJ1">
+          <mechanicalReduction>1</mechanicalReduction>
+        </actuator>
+        <joint name="${prefix}THJ1">
+          <hardwareInterface>EffortJointInterface</hardwareInterface>
+        </joint>
       </transmission>
     </xacro:unless>

File: sr_description/hand/xacro/thumb/thhub.transmission.xacro (robot description, xacro)
@@ -17,8 +17,12 @@
     <!-- motor hand -->
     <xacro:unless value="${muscletrans}">
-      <transmission type="sr_mechanism_model/SimpleTransmission" name="${prefix}thhub_transmission">
-      <actuator name="${prefix}THJ3" />
-      <joint name="${prefix}THJ3" />
-      <mechanicalReduction>1</mechanicalReduction>
+      <transmission name="${prefix}thhub_transmission">
+        <type>sr_mechanism_model/SimpleTransmission</type>
+        <actuator name="${prefix}THJ3">
+          <mechanicalReduction>1</mechanicalReduction>
+        </actuator>
+        <joint name="${prefix}THJ3">
+          <hardwareInterface>EffortJointInterface</hardwareInterface>
+        </joint>
       </transmission>
     </xacro:unless>

File: sr_description/hand/xacro/thumb/thmiddle.transmission.xacro (robot description, xacro)
@@ -17,8 +17,12 @@
     <!-- motor hand -->
     <xacro:unless value="${muscletrans}">
-      <transmission type="sr_mechanism_model/SimpleTransmission" name="${prefix}thmiddle_transmission">
-      <actuator name="${prefix}THJ2" />
-      <joint name="${prefix}THJ2" />
-      <mechanicalReduction>1</mechanicalReduction>
+      <transmission name="${prefix}thmiddle_transmission">
+        <type>sr_mechanism_model/SimpleTransmission</type>
+        <actuator name="${prefix}THJ2">
+          <mechanicalReduction>1</mechanicalReduction>
+        </actuator>
+        <joint name="${prefix}THJ2">
+          <hardwareInterface>EffortJointInterface</hardwareInterface>
+        </joint>
       </transmission>
     </xacro:unless>

File: sr_description/hand/xacro/thumb/thproximal.transmission.xacro (robot description, xacro)
@@ -17,8 +17,12 @@
     <!-- motor hand -->
     <xacro:unless value="${muscletrans}">
-      <transmission type="sr_mechanism_model/SimpleTransmission" name="${prefix}thproximal_transmission">
-      <actuator name="${prefix}THJ4" />
-      <joint name="${prefix}THJ4" />
-      <mechanicalReduction>1</mechanicalReduction>
+      <transmission name="${prefix}thproximal_transmission">
+        <type>sr_mechanism_model/SimpleTransmission</type>
+        <actuator name="${prefix}THJ4">
+          <mechanicalReduction>1</mechanicalReduction>
+        </actuator>
+        <joint name="${prefix}THJ4">
+          <hardwareInterface>EffortJointInterface</hardwareInterface>
+        </joint>
       </transmission>
     </xacro:unless>

File: sr_description/hand/xacro/wrist/wrist.transmission.xacro (robot description, xacro)
@@ -17,8 +17,12 @@
     <!-- motor hand -->
     <xacro:unless value="${muscletrans}">
-      <transmission type="sr_mechanism_model/SimpleTransmission" name="${prefix}wrist_transmission">
-        <actuator name="${prefix}WRJ2" />
-        <joint name="${prefix}WRJ2" />
-        <mechanicalReduction>1</mechanicalReduction>
+      <transmission name="${prefix}wrist_transmission">
+        <type>sr_mechanism_model/SimpleTransmission</type>
+        <actuator name="${prefix}WRJ2">
+          <mechanicalReduction>1</mechanicalReduction>
+        </actuator>
+        <joint name="${prefix}WRJ2">
+          <hardwareInterface>EffortJointInterface</hardwareInterface>
+        </joint>
       </transmission>
     </xacro:unless>

File: sr_description/other/xacro/gazebo/gazebo.urdf.xacro (robot description, xacro)
@@ -4,9 +4,6 @@
 xmlns:interface="http://playerstage.sourceforge.net/gazebo/xmlschema/#interface">
   <gazebo>
-    <plugin name="sr_gazebo_ros_controller_manager"
-    filename="libsr_gazebo_ros_controller_manager.so">
-      <alwaysOn>true</alwaysOn>
-      <updateRate>1400.0</updateRate>
-      <!-- <robotParam>sh_description</robotParam> -->
+    <plugin name="gazebo_ros_control" filename="libgazebo_ros_control.so">
+      <robotSimType>sr_gazebo_sim/SrGazeboHWSim</robotSimType>
     </plugin>
   </gazebo>
