Commit message: Additional non-adjacent self-collision fix for metacarpal and proximal

File: sr_description/hand/xacro/finger/lfmetacarpal/edc_muscle_lfmetacarpal.urdf.xacro (robot description, xacro)
@@ -32,5 +32,5 @@
       </visual>
       <collision>
-        <origin xyz="0 0 0.042" rpy="0 0 0" />
+        <origin xyz="0 0 0.038" rpy="0 0 0" />
         <geometry name="lfmetacarpal_collision_geom">
           <box size="0.018 0.024 0.048" />
@@ -52,4 +52,5 @@
         </plugin>
       </sensor>
+      <selfCollide>true</selfCollide>
       <material>LightGrey</material>
     </gazebo>

File: sr_description/hand/xacro/finger/lfmetacarpal/lfmetacarpal.urdf.xacro (robot description, xacro)
@@ -32,7 +32,7 @@
       </visual>
       <collision>
-        <origin xyz="0 0 0.042" rpy="0 0 0" />
+        <origin xyz="0 0 0.038" rpy="0 0 0" />
         <geometry name="lfmetacarpal_collision_geom">
-          <box size="0.018 0.024 0.048" />
+          <box size="0.018 0.024 0.040" />
         </geometry>
       </collision>
@@ -52,4 +52,5 @@
         </plugin>
       </sensor>
+      <selfCollide>true</selfCollide>
       <material>LightGrey</material>
     </gazebo>
