Commit message: Add missing joint in edc muscle hand thumb biotac.

File: sr_description/hand/xacro/thumb/edc_muscle_thbiotac.urdf.xacro (robot description, xacro)
@@ -128,4 +128,9 @@
       <material>BiotacGreen</material>
     </gazebo>
+    <joint name="th_biotac_joint" type="fixed">
+      <parent link="thmiddle"/>
+      <child link="thbiotac"/>
+      <origin xyz="0 0.0 0.01" rpy="0 0 -1.571" />
+    </joint>
     <!-- extra link to imaginary sphere in fingertip for FK/IK calculations -->
     <!-- remove visual and collision once the correct position is found -->
