Commit message: Fixed arm inertia and collision model Retuned the arm controller in gazebo

File: sr_description/arm/xacro/base/shadowarm_base.urdf.xacro (robot description, xacro)
@@ -6,5 +6,5 @@
       <origin xyz="0 0 0" rpy="0 0 0"/>
       <mass value="0.4" />
-      <inertia  ixx="1.0" ixy="0.0"  ixz="0.0"  iyy="0.0"  iyz="0.0"  izz="0.0" />
+      <inertia  ixx="0.1" ixy="0.0"  ixz="0.0"  iyy="0.1"  iyz="0.0"  izz="0.1" />
     </inertial>
     <visual>
@@ -18,5 +18,5 @@
       <origin xyz="0 0 0.005" rpy="0 0 0" />
       <geometry name="shadowarm_base_collision">
-        <box size="0.03 0.03 0.01"/>
+        <box size="0.145 0.145 0.012"/>
       </geometry>
     </collision>

File: sr_description/arm/xacro/hand_support/shadowarm_handsupport_motor.urdf.xacro (robot description, xacro)
@@ -6,5 +6,5 @@
 	<origin xyz="0 0 0" rpy="0 0 0" />
 	<mass value="0.75" />
-	<inertia  ixx="1.0" ixy="0.0"  ixz="0.0"  iyy="0.0"  iyz="0.0"  izz="0.0" />
+	<inertia  ixx="0.01" ixy="0.0"  ixz="0.0"  iyy="0.01"  iyz="0.0"  izz="0.016" />
       </inertial>
       <visual>
@@ -18,5 +18,5 @@
 	<origin xyz="0 0 -0.005" rpy="0 0 0"/>
 	<geometry name="shadowarm_handsupport_collision">
-	  <cylinder radius="0.06" length="0.001"/>
+	  <cylinder radius="0.0675" length="0.006"/>
 	</geometry>
       </collision>
@@ -32,6 +32,6 @@
       <axis xyz="0 0 -1" />
       <limit lower="-${M_PI/2}" upper="${M_PI/2}"
-      effort="10" velocity="1.0"/>
-      <dynamics damping="10.5"/>
+      effort="30" velocity="1.0"/>
+      <dynamics damping="5.5"/>
     </joint>
     <xacro:shadowarm_handsupport_motor_transmission />

File: sr_description/arm/xacro/hand_support/shadowarm_handsupport_muscle.urdf.xacro (robot description, xacro)
@@ -6,5 +6,5 @@
 	<origin xyz="0 0 0" rpy="0 0 0" />
 	<mass value="0.75" />
-	<inertia  ixx="1.0" ixy="0.0"  ixz="0.0"  iyy="0.0"  iyz="0.0"  izz="0.0" />
+	<inertia  ixx="0.01" ixy="0.0"  ixz="0.0"  iyy="0.01"  iyz="0.0"  izz="0.016" />
       </inertial>
       <visual>
@@ -18,5 +18,5 @@
 	<origin xyz="0 0 0" rpy="0 0 0"/>
 	<geometry name="shadowarm_handsupport_collision">
-	  <cylinder radius="0.06" length="0.001"/>
+	  <cylinder radius="0.07" length="0.006"/>
 	</geometry>
       </collision>
@@ -32,6 +32,6 @@
       <axis xyz="0 0 -1" />
       <limit lower="-${M_PI/2}" upper="${M_PI/2}"
-      effort="10" velocity="1.0"/>
-      <dynamics damping="10.5"/>
+      effort="30" velocity="1.0"/>
+      <dynamics damping="5.5"/>
     </joint>
     <xacro:shadowarm_handsupport_muscle_transmission />

File: sr_description/arm/xacro/lower_arm/shadowarm_lowerarm.urdf.xacro (robot description, xacro)
@@ -6,5 +6,5 @@
 	  <origin xyz="0.08 0 0.0625" rpy="0 0 0" />
 	  <mass value="1.7" />
-	  <inertia  ixx="1.0" ixy="0.0"  ixz="0.0"  iyy="0.0"  iyz="0.0"  izz="0.0" />
+	  <inertia  ixx="0.01" ixy="0.0"  ixz="0.0"  iyy="0.01"  iyz="0.0"  izz="0.01" />
 	</inertial>
 	<visual>
@@ -18,11 +18,11 @@
 	  <origin xyz="0.08 0 0.0625" rpy="0 0 0"/>
 	  <geometry name="shadowarm_lowerarm_collision">
-	    <box size="0.03 0.03 0.10"/>
+	    <box size="0.06 0.08 0.1"/>
 	  </geometry>
 	</collision>
     </link>
     <gazebo reference="shadowarm_lowerarm">
-	<material>LightGrey</material>
-	<selfCollide>false</selfCollide>
+      <material>LightGrey</material>
+      <selfCollide>false</selfCollide>
     </gazebo>
     <joint name="ElbowJSwing" type="revolute">
@@ -32,6 +32,6 @@
       <axis xyz="0 -1 0" />
       <limit lower="0.52" upper="2.09439510239"
-      effort="100" velocity="1.0"/>
-      <dynamics damping="50.5"/>
+      effort="50" velocity="1.0"/>
+      <dynamics damping="5.5"/>
     </joint>
     <xacro:shadowarm_lowerarm_transmission />

File: sr_description/arm/xacro/trunk/shadowarm_trunk.urdf.xacro (robot description, xacro)
@@ -6,5 +6,5 @@
 	  <origin xyz="0 0 0.26525" rpy="0 0 0" />
 	  <mass value="10" />
-	  <inertia  ixx="1.47" ixy="0.0"  ixz="0.0"  iyy="1.47"  iyz="0.0"  izz="2.4" />
+	  <inertia  ixx="0.15" ixy="0.0"  ixz="0.0"  iyy="0.15"  iyz="0.0"  izz="0.02" />
 	</inertial>
 	<visual>
@@ -16,7 +16,7 @@
 	</visual>
 	<collision>
-	  <origin xyz="0 0 0.26525" rpy="0 0 0"/>
+	  <origin xyz="0 0.02 0.30" rpy="0 0 0"/>
 	  <geometry name="shadowarm_trunk_collision">
-	    <box size="0.03 0.03 0.52"/>
+	    <box size="0.170 0.170 0.580"/>
 	  </geometry>
 	</collision>
@@ -32,6 +32,6 @@
       <axis xyz="0 0 1" />
       <limit lower="-${M_PI/4}" upper="${M_PI/2}"
-      effort="100" velocity="1.0"/>
-      <dynamics damping="200.5"/>
+      effort="70" velocity="1.0"/>
+      <dynamics damping="5.5"/>
     </joint>
     <xacro:shadowarm_trunk_transmission />

File: sr_description/arm/xacro/upper_arm/shadowarm_upperarm.urdf.xacro (robot description, xacro)
@@ -6,5 +6,5 @@
 	<origin xyz="0 0 0.1845" rpy="0 0 0" />
 	<mass value="2" />
-	<inertia  ixx="0.5" ixy="0.0"  ixz="0.0"  iyy="0.5"  iyz="0.0"  izz="0.1" />
+	<inertia  ixx="0.4" ixy="0.0"  ixz="0.0"  iyy="0.4"  iyz="0.0"  izz="0.05" />
       </inertial>
       <visual>
@@ -16,7 +16,7 @@
       </visual>
       <collision>
-	<origin xyz="0 0 0.1845" rpy="0 -${M_PI} 0"/>
+	<origin xyz="0 0 0.16" rpy="0 -${M_PI} 0"/>
 	<geometry name="shadowarm_upperarm_collision">
-	  <box size="0.03 0.03 0.369"/>
+	  <box size="0.170 0.133 0.470"/>
 	</geometry>
       </collision>
@@ -32,5 +32,5 @@
       <axis xyz="0 -1 0" />
       <limit lower="0" upper="${M_PI/2}" effort="100" velocity="1.0"/>
-      <dynamics damping="50.5"/>
+      <dynamics damping="5.3"/>
     </joint>
     <xacro:shadowarm_upperarm_transmission />

Commit message: Removed inexistant and unuseful material

File: sr_description/arm/xacro/base/shadowarm_base.urdf.xacro (robot description, xacro)
@@ -23,5 +23,4 @@
   </link>
   <gazebo reference="shadowarm_base">
-    <material>LightGrey</material>
     <selfCollide>false</selfCollide>
   </gazebo>

File: sr_description/arm/xacro/lower_arm/shadowarm_lowerarm.urdf.xacro (robot description, xacro)
@@ -23,5 +23,4 @@
     </link>
     <gazebo reference="shadowarm_lowerarm">
-      <material>LightGrey</material>
       <selfCollide>false</selfCollide>
     </gazebo>

File: sr_description/arm/xacro/trunk/shadowarm_trunk.urdf.xacro (robot description, xacro)
@@ -23,5 +23,4 @@
       </link>
       <gazebo reference="shadowarm_trunk">
-	<material>LightGrey</material>
 	<selfCollide>false</selfCollide>
       </gazebo>

File: sr_description/arm/xacro/upper_arm/shadowarm_upperarm.urdf.xacro (robot description, xacro)
@@ -23,5 +23,4 @@
     </link>
     <gazebo reference="shadowarm_upperarm">
-      <material>LightGrey</material>
       <selfCollide>false</selfCollide>
     </gazebo>

File: sr_description/hand/xacro/finger/distal/distal.gazebo.xacro (robot description, xacro)
@@ -22,5 +22,4 @@
       <kp  value="10000000.0" />
       <kd  value="1.0" />
-      <material>LightGrey</material>
       <selfCollide>true</selfCollide>
     </gazebo>

File: sr_description/hand/xacro/finger/lfmetacarpal/lfmetacarpal.gazebo.xacro (robot description, xacro)
@@ -19,5 +19,4 @@
       </sensor>
       <selfCollide>true</selfCollide>
-      <material>LightGrey</material>
     </gazebo>
   </xacro:macro>

File: sr_description/hand/xacro/finger/middle/middle.gazebo.xacro (robot description, xacro)
@@ -18,5 +18,4 @@
         </plugin>
       </sensor>
-      <material>LightGrey</material>
       <selfCollide>true</selfCollide>
     </gazebo>

File: sr_description/hand/xacro/finger/proximal/proximal.gazebo.xacro (robot description, xacro)
@@ -18,5 +18,4 @@
         </plugin>
       </sensor>
-       <material>LightGrey</material>
       <selfCollide>true</selfCollide>
     </gazebo>

File: sr_description/hand/xacro/forearm/forearm.urdf.xacro (robot description, xacro)
@@ -54,5 +54,4 @@
       </link>
       <gazebo reference="${prefix}forearm">
-        <material>LightGrey</material>
         <selfCollide>false</selfCollide>
       </gazebo>

File: sr_description/hand/xacro/palm/palm.gazebo.xacro (robot description, xacro)
@@ -18,5 +18,4 @@
         </plugin>
       </sensor>
-      <material>LightGrey</material>
     </gazebo>
   </xacro:macro>

File: sr_description/hand/xacro/thumb/thbase.gazebo.xacro (robot description, xacro)
@@ -19,5 +19,4 @@
       </sensor>
       <selfCollide>false</selfCollide>
-      <material>LightGrey</material>
     </gazebo>
   </xacro:macro>

File: sr_description/hand/xacro/thumb/thdistal.gazebo.xacro (robot description, xacro)
@@ -22,5 +22,4 @@
       <kp  value="10000000.0" />
       <kd  value="1.0" />
-      <material>LightGrey</material>
       <selfCollide>true</selfCollide>
     </gazebo>

File: sr_description/hand/xacro/thumb/thhub.gazebo.xacro (robot description, xacro)
@@ -19,5 +19,4 @@
       </sensor>
       <selfCollide>true</selfCollide>
-      <material>LightGrey</material>
     </gazebo>
   </xacro:macro>

File: sr_description/hand/xacro/thumb/thmiddle.gazebo.xacro (robot description, xacro)
@@ -19,5 +19,4 @@
       </sensor>
       <selfCollide>true</selfCollide>
-      <material>LightGrey</material>
     </gazebo>
   </xacro:macro>

File: sr_description/hand/xacro/thumb/thproximal.gazebo.xacro (robot description, xacro)
@@ -19,5 +19,4 @@
       </sensor>
       <selfCollide>false</selfCollide>
-      <material>LightGrey</material>
     </gazebo>
   </xacro:macro>

Commit message: added missing xacro: prefixes

File: sr_description/arm/xacro/base/shadowarm_base.urdf.xacro (robot description, xacro)
@@ -1,4 +1,4 @@
 <robot xmlns:xacro="http://www.ros.org/wiki/xacro">
-  <property name="M_PI" value="3.1415926535897931" />
+  <xacro:property name="M_PI" value="3.1415926535897931" />
   <xacro:macro name="shadowarm_base">
     <link name="shadowarm_base">

File: sr_description/hand/xacro/ff_biotac_hand.urdf.xacro (robot description, xacro)
@@ -8,5 +8,5 @@
   <xacro:include filename="$(find sr_description)/hand/xacro/finger/fingers.urdf.xacro" />
   <xacro:include filename="$(find sr_description)/hand/xacro/thumb/thumb.urdf.xacro" />
-  <property name="M_PI" value="3.1415926535897931" />
+  <xacro:property name="M_PI" value="3.1415926535897931" />
   <!-- muscletrans is true for muscle transmission to be used, false to use motor transmission -->
   <!-- muscle is true for muscle hand or false for motor hand -->

File: sr_description/hand/xacro/finger/fingers.urdf.xacro (robot description, xacro)
@@ -27,5 +27,5 @@
       link_prefix="${link_prefix}" joint_prefix="${joint_prefix}"
       parent="${prefix}lfmetacarpal">
-        <insert_block name="origin" />
+        <xacro:insert_block name="origin" />
       </xacro:knuckle>
     </xacro:if>
@@ -36,5 +36,5 @@
       link_prefix="${link_prefix}" joint_prefix="${joint_prefix}"
       parent="${parent}">
-        <insert_block name="origin" />
+        <xacro:insert_block name="origin" />
       </xacro:knuckle>
     </xacro:unless>

File: sr_description/hand/xacro/finger/knuckle/knuckle.urdf.xacro (robot description, xacro)
@@ -18,5 +18,5 @@
       <inertial>
         <origin xyz="0 0 0" rpy="0 0 0" />
-        <!--<insert_block name="origin" /> -->
+        <!--<xacro:insert_block name="origin" /> -->
         <mass value="0.008" />
         <inertia ixx="0.00000026" ixy="0.0" ixz="0.0"
@@ -42,6 +42,6 @@
       <child link="${prefix}${link_prefix}knuckle" />
       <!--<origin xyz="0.033 0 0.095" rpy="0 0 0" />-->
-      <insert_block name="origin" />
-      <insert_block name="axis" />
+      <xacro:insert_block name="origin" />
+      <xacro:insert_block name="axis" />
       <limit lower="${-20/180*M_PI}" upper="${20/180*M_PI}"
       effort="2" velocity="2.0" />

File: sr_description/hand/xacro/forearm/forearm_lite.urdf.xacro (robot description, xacro)
@@ -3,5 +3,5 @@
   <!-- prefix can be anything but usually is "r_" or  "l_" for right and left hands distinction -->
   <xacro:macro name="forearm" params="muscle prefix">
-    <property name="M_PI" value="3.1415926535897931" />
+    <xacro:property name="M_PI" value="3.1415926535897931" />
     <link name="${prefix}forearm">
       <inertial>

File: sr_description/hand/xacro/full_hand.urdf.xacro (robot description, xacro)
@@ -8,5 +8,5 @@
   <xacro:include filename="$(find sr_description)/hand/xacro/finger/fingers.urdf.xacro" />
   <xacro:include filename="$(find sr_description)/hand/xacro/thumb/thumb.urdf.xacro" />
-  <property name="M_PI" value="3.1415926535897931" />
+  <xacro:property name="M_PI" value="3.1415926535897931" />
   <!-- muscletrans is true for muscle transmission to be used, false to use motor transmission -->
   <!-- muscle is true for muscle hand or false for motor hand -->

File: sr_description/hand/xacro/hand_lite.urdf.xacro (robot description, xacro)
@@ -8,5 +8,5 @@
   <xacro:include filename="$(find sr_description)/hand/xacro/finger/fingers.urdf.xacro" />
   <xacro:include filename="$(find sr_description)/hand/xacro/thumb/thumb.urdf.xacro" />
-  <property name="M_PI" value="3.1415926535897931" />
+  <xacro:property name="M_PI" value="3.1415926535897931" />
   <!-- muscletrans is true for muscle transmission to be used, false to use motor transmission -->
   <!-- muscle is true for muscle hand or false for motor hand -->

File: sr_description/hand/xacro/one_finger_unit.urdf.xacro (robot description, xacro)
@@ -5,5 +5,5 @@
   <xacro:include filename="$(find sr_description)/hand/xacro/forearm/forearm.urdf.xacro" />
   <xacro:include filename="$(find sr_description)/hand/xacro/finger/fingers.urdf.xacro" />
-  <property name="M_PI" value="3.1415926535897931" />
+  <xacro:property name="M_PI" value="3.1415926535897931" />
   <!-- muscletrans is true for muscle transmission to be used, false to use motor transmission -->
   <!-- muscle is true for muscle hand or false for motor hand -->

File: sr_description/hand/xacro/th_ff_rf_ellipsoid_hand.urdf.xacro (robot description, xacro)
@@ -8,5 +8,5 @@
   <xacro:include filename="$(find sr_description)/hand/xacro/finger/fingers.urdf.xacro" />
   <xacro:include filename="$(find sr_description)/hand/xacro/thumb/thumb.urdf.xacro" />
-  <property name="M_PI" value="3.1415926535897931" />
+  <xacro:property name="M_PI" value="3.1415926535897931" />
   <!-- muscletrans is true for muscle transmission to be used, false to use motor transmission -->
   <!-- muscle is true for muscle hand or false for motor hand -->

File: sr_description/hand/xacro/three_biotac_fingers_hand.urdf.xacro (robot description, xacro)
@@ -8,5 +8,5 @@
   <xacro:include filename="$(find sr_description)/hand/xacro/finger/fingers.urdf.xacro" />
   <xacro:include filename="$(find sr_description)/hand/xacro/thumb/thumb.urdf.xacro" />
-  <property name="M_PI" value="3.1415926535897931" />
+  <xacro:property name="M_PI" value="3.1415926535897931" />
   <!-- muscletrans is true for muscle transmission to be used, false to use motor transmission -->
   <!-- muscle is true for muscle hand or false for motor hand -->

File: sr_description/hand/xacro/three_fingers_hand.urdf.xacro (robot description, xacro)
@@ -8,5 +8,5 @@
   <xacro:include filename="$(find sr_description)/hand/xacro/finger/fingers.urdf.xacro" />
   <xacro:include filename="$(find sr_description)/hand/xacro/thumb/thumb.urdf.xacro" />
-  <property name="M_PI" value="3.1415926535897931" />
+  <xacro:property name="M_PI" value="3.1415926535897931" />
   <!-- muscletrans is true for muscle transmission to be used, false to use motor transmission -->
   <!-- muscle is true for muscle hand or false for motor hand -->

File: sr_description/hand/xacro/wrist/wrist.urdf.xacro (robot description, xacro)
@@ -62,5 +62,5 @@
       <parent link="${parent}" />
       <child link="${prefix}wrist" />
-      <insert_block name="origin" />
+      <xacro:insert_block name="origin" />
       <axis xyz="0 ${reflect} 0" />
       <limit lower="${-30/180*M_PI}" upper="${10/180*M_PI}"

File: sr_description/other/xacro/kinect/shadowarm_kinect.urdf.xacro (robot description, xacro)
@@ -1,4 +1,4 @@
 <robot xmlns:xacro="http://ros.org/wiki/xacro">
-  <property name="M_PI" value="3.1415926535" />
+  <xacro:property name="M_PI" value="3.1415926535" />
   <xacro:include filename="$(find sr_description)/other/xacro/kinect/gazebo_kinect.urdf.xacro" />
   <xacro:macro name="shadowarm_side_kinect" params="parent">
