Commit message: adding bt_sp to xacro models

File: sr_description/hand/xacro/ff_biotac_hand.urdf.xacro (robot description, xacro)
@@ -12,4 +12,5 @@
   <!-- muscle is true for muscle hand or false for motor hand -->
   <!-- bio is true for biotac finger or false for standard finger -->
+  <!-- bt_sp is true for BT_SP finger or false for standard finger -->
   <!-- ubi is true for ubi finger or false for standard finger -->
   <!-- eli is true for ellipsoid fingertip or false for standard finger -->
@@ -17,5 +18,5 @@
   <!-- prefix can be anything but usually is "r_" or  "l_" for right and left hands distinction -->
   <xacro:macro name="shadowhand"
-  params="muscletrans muscle bio ubi eli reflect prefix">
+  params="muscletrans muscle bio bt_sp ubi eli reflect prefix">
     <!-- Forearm -->
     <xacro:forearm muscle="${muscle}" prefix="${prefix}" />
@@ -38,5 +39,5 @@
     <!-- First Finger Biotac -->
     <xacro:finger muscletrans="${muscletrans}" lf="false"
-    bio="true" ubi="false" eli="false" prefix="${prefix}"
+    bio="true" bt_sp="false" ubi="false" eli="false" prefix="${prefix}"
     reflect="${reflect}" link_prefix="ff" joint_prefix="FF"
     parent="${prefix}palm">
@@ -46,5 +47,5 @@
     <!-- Middle Finger -->
     <xacro:finger muscletrans="${muscletrans}" lf="false"
-    bio="${bio}" ubi="${ubi}" eli="${eli}" prefix="${prefix}"
+    bio="${bio}" bt_sp="false" ubi="${ubi}" eli="${eli}" prefix="${prefix}"
     reflect="${reflect}" link_prefix="mf" joint_prefix="MF"
     parent="${prefix}palm">
@@ -54,5 +55,5 @@
     <!-- Ring Finger -->
     <xacro:finger muscletrans="${muscletrans}" lf="false"
-    bio="${bio}" ubi="${ubi}" eli="${eli}" prefix="${prefix}"
+    bio="${bio}" bt_sp="${bt_sp}" ubi="${ubi}" eli="${eli}" prefix="${prefix}"
     reflect="${reflect}" link_prefix="rf" joint_prefix="RF"
     parent="${prefix}palm">
@@ -62,5 +63,5 @@
     <!-- Little Finger  -->
     <xacro:finger muscletrans="${muscletrans}" lf="true"
-    bio="${bio}" ubi="${ubi}" eli="${eli}" prefix="${prefix}"
+    bio="${bio}" bt_sp="${bt_sp}" ubi="${ubi}" eli="${eli}" prefix="${prefix}"
     reflect="${reflect}" link_prefix="lf" joint_prefix="LF"
     parent="${prefix}palm">
@@ -69,5 +70,5 @@
     </xacro:finger>
     <!-- Thumb Biotac -->
-    <xacro:thumb muscletrans="${muscletrans}" bio="${bio}"
+    <xacro:thumb muscletrans="${muscletrans}" bio="${bio}" bt_sp="${bt_sp}"
     ubi="${ubi}" eli="${eli}" prefix="${prefix}"
     reflect="${reflect}" is_lite="0" parent="${prefix}palm">

File: sr_description/hand/xacro/finger/distal/distal.urdf.xacro (robot description, xacro)
@@ -10,4 +10,5 @@
   <!-- muscle is true for muscle hand or false for motor hand -->
   <!-- bio is true for biotac finger or false for standard finger -->
+  <!-- bt_sp is true for BT_SP finger or false for standard finger -->
   <!-- ubi is true for ubi finger or false for standard finger -->
   <!-- eli is true for ellipsoid fingertip or false for standard finger -->
@@ -17,5 +18,5 @@
   <!-- parent is the parent link for the joint -->
   <xacro:macro name="distal"
-  params="muscle bio ubi eli prefix link_prefix joint_prefix parent">
+  params="muscle bio bt_sp ubi eli prefix link_prefix joint_prefix parent">
     <link name="${prefix}${link_prefix}distal">
       <inertial>
@@ -23,5 +24,5 @@
         <origin xyz="0 0 0.012" />
         <inertia ixx="0.00000094" ixy="0.0" ixz="0.0"
-        iyy="0.0000011" iyz="0.0" izz="0.00000053" />
+		 iyy="0.0000011" iyz="0.0" izz="0.00000053" />
       </inertial>
       <visual>
@@ -31,5 +32,5 @@
             <!-- Ubi distal -->
             <mesh filename="package://sr_description/hand/model/ubi_tactiles/ubi_tip_visual.dae"
-            scale="0.001 0.001 0.001" />
+		  scale="0.001 0.001 0.001" />
           </xacro:if>
           <xacro:unless value="${ubi}">
@@ -37,5 +38,5 @@
               <!-- Ellispoid distal  -->
               <mesh filename="package://sr_description/hand/model/ellipsoids/distal_ellipsoid_visual.dae"
-              scale="0.001 0.001 0.001" />
+		    scale="0.001 0.001 0.001" />
             </xacro:if>
             <xacro:unless value="${eli}">
@@ -43,10 +44,17 @@
                 <!-- biotac distal  -->
                 <mesh filename="package://sr_description/hand/model/F1.dae"
-                scale="0.001 0.001 0.001" />
+                      scale="0.001 0.001 0.001" />
               </xacro:if>
-              <xacro:unless value="${bio}">
-                <!-- Standard distal  -->
-                <mesh filename="package://sr_description/hand/model/F1.dae"
-                scale="0.001 0.001 0.001" />
+              <xacro:unless value="${bt_sp}">
+		<xacro:if value="${bt_sp}">
+                  <!-- bt_sp distal  -->
+                  <mesh filename="package://sr_description/hand/model/biotacs/sp.dae"
+			scale="0.001 0.001 0.001" />
+		</xacro:if>
+		<xacro:unless value="${bt_sp}">
+                  <!-- Standard distal  -->
+                  <mesh filename="package://sr_description/hand/model/F1.dae"
+			scale="0.001 0.001 0.001" />
+		</xacro:unless>
               </xacro:unless>
             </xacro:unless>

File: sr_description/hand/xacro/finger/fingers.urdf.xacro (robot description, xacro)
@@ -9,4 +9,5 @@
   <!-- lf is true for little finger or false for standard finger -->
   <!-- bio is true for biotac finger or false for standard finger -->
+  <!-- bt_sp is true for BT_SP finger or false for standard finger -->
   <!-- ubi is true for ubi finger or false for standard finger -->
   <!-- eli is true for ellipsoid fingertip or false for standard finger -->
@@ -17,5 +18,5 @@
   <!-- parent is the parent link for the first joint -->
   <xacro:macro name="finger"
-  params="muscletrans lf bio ubi eli reflect prefix link_prefix joint_prefix parent *origin *axis">
+  params="muscletrans lf bio bt_sp ubi eli reflect prefix link_prefix joint_prefix parent *origin *axis">
     <!-- Little finger special case -->
     <xacro:if value="${lf}">
@@ -61,5 +62,5 @@
     <!-- only if finger is not biotac  -->
     <xacro:unless value="${bio}">
-      <xacro:distal muscle="${muscletrans}" bio="${bio}"
+      <xacro:distal muscle="${muscletrans}" bio="${bio}" bt_sp="${bt_sp}"
       ubi="${ubi}" eli="${eli}" prefix="${prefix}"
       link_prefix="${link_prefix}" joint_prefix="${joint_prefix}"

File: sr_description/hand/xacro/full_hand.urdf.xacro (robot description, xacro)
@@ -12,4 +12,5 @@
   <!-- muscle is true for muscle hand or false for motor hand -->
   <!-- bio is true for biotac finger or false for standard finger -->
+  <!-- bt_sp is true for BT_SP finger or false for standard finger -->
   <!-- ubi is true for ubi finger or false for standard finger -->
   <!-- eli is true for ellipsoid fingertip or false for standard finger -->
@@ -17,5 +18,5 @@
   <!-- prefix can be anything but usually is "r_" or  "l_" for right and left hands distinction -->
   <xacro:macro name="shadowhand"
-  params="muscletrans muscle bio ubi eli reflect prefix">
+  params="muscletrans muscle bio bt_sp ubi eli reflect prefix">
     <!-- Forearm -->
     <xacro:forearm muscle="${muscle}" prefix="${prefix}" />
@@ -38,5 +39,5 @@
     <!-- First Finger -->
     <xacro:finger muscletrans="${muscletrans}" lf="false"
-    bio="${bio}" ubi="${ubi}" eli="${eli}" prefix="${prefix}"
+    bio="${bio}" bt_sp="${bt_sp}" ubi="${ubi}" eli="${eli}" prefix="${prefix}"
     reflect="${reflect}" link_prefix="ff" joint_prefix="FF"
     parent="${prefix}palm">
@@ -46,5 +47,5 @@
     <!-- Middle Finger -->
     <xacro:finger muscletrans="${muscletrans}" lf="false"
-    bio="${bio}" ubi="${ubi}" eli="${eli}" prefix="${prefix}"
+    bio="${bio}" bt_sp="${bt_sp}" ubi="${ubi}" eli="${eli}" prefix="${prefix}"
     reflect="${reflect}" link_prefix="mf" joint_prefix="MF"
     parent="${prefix}palm">
@@ -54,5 +55,5 @@
     <!-- Ring Finger -->
     <xacro:finger muscletrans="${muscletrans}" lf="false"
-    bio="${bio}" ubi="${ubi}" eli="${eli}" prefix="${prefix}"
+    bio="${bio}" bt_sp="${bt_sp}" ubi="${ubi}" eli="${eli}" prefix="${prefix}"
     reflect="${reflect}" link_prefix="rf" joint_prefix="RF"
     parent="${prefix}palm">
@@ -62,5 +63,5 @@
     <!-- Little Finger  -->
     <xacro:finger muscletrans="${muscletrans}" lf="true"
-    bio="${bio}" ubi="${ubi}" eli="${eli}" prefix="${prefix}"
+    bio="${bio}" bt_sp="${bt_sp}" ubi="${ubi}" eli="${eli}" prefix="${prefix}"
     reflect="${reflect}" link_prefix="lf" joint_prefix="LF"
     parent="${prefix}palm">
@@ -69,5 +70,5 @@
     </xacro:finger>
     <!-- Thumb  -->
-    <xacro:thumb muscletrans="${muscletrans}" bio="${bio}"
+    <xacro:thumb muscletrans="${muscletrans}" bio="${bio}" bt_sp="${bt_sp}"
     ubi="${ubi}" eli="${eli}" prefix="${prefix}"
     reflect="${reflect}" is_lite="0" parent="${prefix}palm">

File: sr_description/hand/xacro/hand_lite.urdf.xacro (robot description, xacro)
@@ -12,4 +12,5 @@
   <!-- muscle is true for muscle hand or false for motor hand -->
   <!-- bio is true for biotac finger or false for standard finger -->
+  <!-- bt_sp is true for BT_SP finger or false for standard finger -->
   <!-- ubi is true for ubi finger or false for standard finger -->
   <!-- eli is true for ellipsoid fingertip or false for standard finger -->
@@ -17,5 +18,5 @@
   <!-- prefix can be anything but usually is "r_" or  "l_" for right and left hands distinction -->
   <xacro:macro name="shadowhand"
-  params="muscletrans muscle bio ubi eli reflect prefix">
+  params="muscletrans muscle bio bt_sp ubi eli reflect prefix">
     <!-- Forearm -->
     <xacro:forearm muscle="${muscle}" prefix="${prefix}" />
@@ -39,5 +40,5 @@
     <!-- First Finger -->
     <xacro:finger muscletrans="${muscletrans}" lf="false"
-    bio="${bio}" ubi="${ubi}" eli="${eli}" prefix="${prefix}"
+    bio="${bio}" bt_sp="${bt_sp}" ubi="${ubi}" eli="${eli}" prefix="${prefix}"
     reflect="${reflect}" link_prefix="ff" joint_prefix="FF"
     parent="${prefix}palm">
@@ -47,5 +48,5 @@
     <!-- Middle Finger -->
     <xacro:finger muscletrans="${muscletrans}" lf="false"
-    bio="${bio}" ubi="${ubi}" eli="${eli}" prefix="${prefix}"
+    bio="${bio}" bt_sp="${bt_sp}" ubi="${ubi}" eli="${eli}" prefix="${prefix}"
     reflect="${reflect}" link_prefix="mf" joint_prefix="MF"
     parent="${prefix}palm">
@@ -55,5 +56,5 @@
     <!-- Ring Finger -->
     <xacro:finger muscletrans="${muscletrans}" lf="false"
-    bio="${bio}" ubi="${ubi}" eli="${eli}" prefix="${prefix}"
+    bio="${bio}" bt_sp="${bt_sp}" ubi="${ubi}" eli="${eli}" prefix="${prefix}"
     reflect="${reflect}" link_prefix="rf" joint_prefix="RF"
     parent="${prefix}palm">

File: sr_description/hand/xacro/one_finger_unit.urdf.xacro (robot description, xacro)
@@ -9,4 +9,5 @@
   <!-- muscle is true for muscle hand or false for motor hand -->
   <!-- bio is true for biotac finger or false for standard finger -->
+  <!-- bt_sp is true for BT_SP finger or false for standard finger -->
   <!-- ubi is true for ubi finger or false for standard finger -->
   <!-- eli is true for ellipsoid fingertip or false for standard finger -->
@@ -14,5 +15,5 @@
   <!-- prefix can be anything but usually is "r_" or  "l_" for right and left hands distinction -->
   <xacro:macro name="shadowhand"
-  params="muscletrans muscle bio ubi eli reflect prefix">
+  params="muscletrans muscle bio bt_sp ubi eli reflect prefix">
     <!-- Forearm -->
     <xacro:forearm muscle="${muscle}" prefix="${prefix}" />
@@ -49,5 +50,5 @@
     <!-- TODO: Check if offset is the same for muscle hand -->
     <xacro:finger muscletrans="${muscletrans}" lf="false"
-    bio="${bio}" ubi="${ubi}" eli="${eli}" prefix="${prefix}"
+    bio="${bio}" bt_sp="${bt_sp}" ubi="${ubi}" eli="${eli}" prefix="${prefix}"
     reflect="${reflect}" link_prefix="mf" joint_prefix="MF"
     parent="${prefix}dummy_palm">

File: sr_description/hand/xacro/th_ff_rf_ellipsoid_hand.urdf.xacro (robot description, xacro)
@@ -12,4 +12,5 @@
   <!-- muscle is true for muscle hand or false for motor hand -->
   <!-- bio is true for biotac finger or false for standard finger -->
+  <!-- bt_sp is true for BT_SP finger or false for standard finger -->
   <!-- ubi is true for ubi finger or false for standard finger -->
   <!-- eli is true for ellipsoid fingertip or false for standard finger -->
@@ -17,5 +18,5 @@
   <!-- prefix can be anything but usually is "r_" or  "l_" for right and left hands distinction -->
   <xacro:macro name="shadowhand"
-  params="muscletrans muscle bio ubi eli reflect prefix">
+  params="muscletrans muscle bio bt_sp ubi eli reflect prefix">
     <!-- Forearm -->
     <xacro:forearm muscle="${muscle}" prefix="${prefix}" />
@@ -38,5 +39,5 @@
     <!-- First Finger Biotac -->
     <xacro:finger muscletrans="${muscletrans}" lf="false"
-    bio="false" ubi="false" eli="true" prefix="${prefix}"
+    bio="false" bt_sp="false" ubi="false" eli="true" prefix="${prefix}"
     reflect="${reflect}" link_prefix="ff" joint_prefix="FF"
     parent="${prefix}palm">
@@ -46,5 +47,5 @@
     <!-- Middle Finger -->
     <xacro:finger muscletrans="${muscletrans}" lf="false"
-    bio="${bio}" ubi="${ubi}" eli="${eli}" prefix="${prefix}"
+    bio="${bio}" bt_sp="${bt_sp}" ubi="${ubi}" eli="${eli}" prefix="${prefix}"
     reflect="${reflect}" link_prefix="mf" joint_prefix="MF"
     parent="${prefix}palm">
@@ -54,5 +55,5 @@
     <!-- Ring Finger -->
     <xacro:finger muscletrans="${muscletrans}" lf="false"
-    bio="false" ubi="false" eli="true" prefix="${prefix}"
+    bio="false" bt_sp="false" ubi="false" eli="true" prefix="${prefix}"
     reflect="${reflect}" link_prefix="rf" joint_prefix="RF"
     parent="${prefix}palm">
@@ -62,5 +63,5 @@
     <!-- Little Finger  -->
     <xacro:finger muscletrans="${muscletrans}" lf="true"
-    bio="${bio}" ubi="${ubi}" eli="${eli}" prefix="${prefix}"
+    bio="${bio}" bt_sp="${bt_sp}" ubi="${ubi}" eli="${eli}" prefix="${prefix}"
     reflect="${reflect}" link_prefix="lf" joint_prefix="LF"
     parent="${prefix}palm">
@@ -69,5 +70,5 @@
     </xacro:finger>
     <!-- Thumb Biotac -->
-    <xacro:thumb muscletrans="${muscletrans}" bio="false"
+    <xacro:thumb muscletrans="${muscletrans}" bio="false" bt_sp="false"
     ubi="false" eli="true" prefix="${prefix}" reflect="${reflect}"
     is_lite="0" parent="${prefix}palm"></xacro:thumb>

File: sr_description/hand/xacro/three_biotac_fingers_hand.urdf.xacro (robot description, xacro)
@@ -12,4 +12,5 @@
   <!-- muscle is true for muscle hand or false for motor hand -->
   <!-- bio is true for biotac finger or false for standard finger -->
+  <!-- bt_sp is true for BT_SP finger or false for standard finger -->
   <!-- ubi is true for ubi finger or false for standard finger -->
   <!-- eli is true for ellipsoid fingertip or false for standard finger -->
@@ -17,5 +18,5 @@
   <!-- prefix can be anything but usually is "r_" or  "l_" for right and left hands distinction -->
   <xacro:macro name="shadowhand"
-  params="muscletrans muscle bio ubi eli reflect prefix">
+  params="muscletrans muscle bio bt_sp ubi eli reflect prefix">
     <!-- Forearm -->
     <xacro:forearm muscle="${muscle}" prefix="${prefix}" />
@@ -38,5 +39,5 @@
     <!-- First Finger Biotac -->
     <xacro:finger muscletrans="${muscletrans}" lf="false"
-    bio="true" ubi="false" eli="false" prefix="${prefix}"
+    bio="true" bt_sp="false"  ubi="false" eli="false" prefix="${prefix}"
     reflect="${reflect}" link_prefix="ff" joint_prefix="FF"
     parent="${prefix}palm">
@@ -46,5 +47,5 @@
     <!-- Middle Finger Biotac -->
     <xacro:finger muscletrans="${muscletrans}" lf="false"
-    bio="true" ubi="false" eli="false" prefix="${prefix}"
+    bio="true" bt_sp="false" ubi="false" eli="false" prefix="${prefix}"
     reflect="${reflect}" link_prefix="mf" joint_prefix="MF"
     parent="${prefix}palm">
@@ -54,5 +55,5 @@
     <!-- Ring Finger -->
     <xacro:finger muscletrans="${muscletrans}" lf="false"
-    bio="false" ubi="false" eli="false" prefix="${prefix}"
+    bio="false" bt_sp="false" ubi="false" eli="false" prefix="${prefix}"
     reflect="${reflect}" link_prefix="rf" joint_prefix="RF"
     parent="${prefix}palm">
@@ -62,5 +63,5 @@
     <!-- Little Finger  -->
     <xacro:finger muscletrans="${muscletrans}" lf="true"
-    bio="false" ubi="false" eli="false" prefix="${prefix}"
+    bio="false" bt_sp="false" ubi="false" eli="false" prefix="${prefix}"
     reflect="${reflect}" link_prefix="lf" joint_prefix="LF"
     parent="${prefix}palm">
@@ -69,5 +70,5 @@
     </xacro:finger>
     <!-- Thumb Biotac -->
-    <xacro:thumb muscletrans="${muscletrans}" bio="true"
+    <xacro:thumb muscletrans="${muscletrans}" bio="true" bt_sp="false"
     ubi="false" eli="false" prefix="${prefix}" reflect="${reflect}"
     is_lite="0" parent="${prefix}palm"></xacro:thumb>

File: sr_description/hand/xacro/three_fingers_hand.urdf.xacro (robot description, xacro)
@@ -12,4 +12,5 @@
   <!-- muscle is true for muscle hand or false for motor hand -->
   <!-- bio is true for biotac finger or false for standard finger -->
+  <!-- bt_sp is true for BT_SP finger or false for standard finger -->
   <!-- ubi is true for ubi finger or false for standard finger -->
   <!-- eli is true for ellipsoid fingertip or false for standard finger -->
@@ -17,5 +18,5 @@
   <!-- prefix can be anything but usually is "r_" or  "l_" for right and left hands distinction -->
   <xacro:macro name="shadowhand"
-  params="muscletrans muscle bio ubi eli reflect prefix">
+  params="muscletrans muscle bio bt_sp ubi eli reflect prefix">
     <!-- Forearm -->
     <xacro:forearm muscle="${muscle}" prefix="${prefix}" />
@@ -38,5 +39,5 @@
     <!-- First Finger -->
     <xacro:finger muscletrans="${muscletrans}" lf="false"
-    bio="${bio}" ubi="${ubi}" eli="${eli}" prefix="${prefix}"
+    bio="${bio}" bt_sp="${bt_sp}" ubi="${ubi}" eli="${eli}" prefix="${prefix}"
     reflect="${reflect}" link_prefix="ff" joint_prefix="FF"
     parent="${prefix}palm">
@@ -46,5 +47,5 @@
     <!-- Middle Finger -->
     <xacro:finger muscletrans="${muscletrans}" lf="false"
-    bio="${bio}" ubi="${ubi}" eli="${eli}" prefix="${prefix}"
+    bio="${bio}" bt_sp="${bt_sp}" ubi="${ubi}" eli="${eli}" prefix="${prefix}"
     reflect="${reflect}" link_prefix="mf" joint_prefix="MF"
     parent="${prefix}palm">
@@ -53,5 +54,5 @@
     </xacro:finger>
     <!-- Thumb  -->
-    <xacro:thumb muscletrans="${muscletrans}" bio="${bio}"
+    <xacro:thumb muscletrans="${muscletrans}" bio="${bio}" bt_sp="${bt_sp}"
     ubi="${ubi}" eli="${eli}" prefix="${prefix}"
     reflect="${reflect}" is_lite="0" parent="${prefix}palm">

File: sr_description/hand/xacro/thumb/thdistal.urdf.xacro (robot description, xacro)
@@ -10,4 +10,5 @@
   <!-- muscle is true for muscle hand or false for motor hand -->
   <!-- bio is true for biotac finger or false for standard finger -->
+  <!-- bt_sp is true for BT_SP finger or false for standard finger -->
   <!-- ubi is true for ubi finger or false for standard finger -->
   <!-- eli is true for ellipsoid fingertip or false for standard finger -->
@@ -15,5 +16,5 @@
   <!-- parent is the parent link for the first joint -->
   <xacro:macro name="thdistal"
-  params="muscle bio ubi eli prefix parent">
+  params="muscle bio bt_sp ubi eli prefix parent">
     <xacro:if value="${bio}">
       <!--    BIOTAC -->
@@ -137,11 +138,18 @@
                 <!-- Ubi distal -->
                 <mesh filename="package://sr_description/hand/model/TH1_z.dae"
-                scale="0.001 0.001 0.001" />
+                      scale="0.001 0.001 0.001" />
               </xacro:if>
-              <!-- Standard distal  -->
-              <xacro:unless value="${ubi}">
-                <mesh filename="package://sr_description/hand/model/TH1_z.dae"
-                scale="0.001 0.001 0.001" />
-              </xacro:unless>
+	      <xacro:unless value="${ubi}">
+		<xacro:if value="${bt_sp}">
+		  <!-- bt sp distal  -->
+		  <mesh filename="package://sr_description/hand/model/biotacs/sp.dae"
+			scale="0.001 0.001 0.001" />
+		</xacro:if>
+		<xacro:unless value="${bt_sp}">
+		  <!-- Standard distal  -->
+                  <mesh filename="package://sr_description/hand/model/TH1_z.dae"
+			scale="0.001 0.001 0.001" />
+		</xacro:unless>
+	      </xacro:unless>
             </xacro:unless>
           </geometry>
