Commit message: Bring in the new forearm part.
NOTE: Not aligned properly yet!

File: sr_description/hand/xacro/hand_lite.urdf.xacro (robot description, xacro)
@@ -3,7 +3,7 @@
        xmlns:interface="http://playerstage.sourceforge.net/gazebo/xmlschema/#interface"
        xmlns:xacro="http://www.ros.org/wiki/xacro">
-  <xacro:include filename="$(find sr_description)/hand/xacro/forearm/forearm.urdf.xacro" />
+  <xacro:include filename="$(find sr_description)/hand/xacro/forearm/forearm_lite.urdf.xacro" />
   <xacro:include filename="$(find sr_description)/hand/xacro/wrist/wrist.urdf.xacro" />
-  <xacro:include filename="$(find sr_description)/hand/xacro/palm/palm.urdf.xacro" />
+  <xacro:include filename="$(find sr_description)/hand/xacro/palm/palm_lite.urdf.xacro" />
   <xacro:include filename="$(find sr_description)/hand/xacro/finger/fingers.urdf.xacro" />
   <xacro:include filename="$(find sr_description)/hand/xacro/thumb/thumb.urdf.xacro" />
@@ -20,14 +20,17 @@
     <xacro:forearm muscle="${muscle}" prefix="${prefix}" />
     <!-- Wrist -->
-		<xacro:if value="${muscle}">
-			<xacro:wrist muscletrans="${muscletrans}" prefix="${prefix}" reflect="${reflect}" parent="${prefix}forearm">
-			<origin xyz="0 0 0.4096" rpy="0 0 0" />
-			</xacro:wrist>
-		</xacro:if>
-		<xacro:unless value="${muscle}">
-			<xacro:wrist muscletrans="false" prefix="${prefix}" reflect="${reflect}" parent="${prefix}forearm">
-			<origin xyz="0 -0.010 0.213" rpy="0 0 0" />
-			</xacro:wrist>
-		</xacro:unless>
+    <!-- Completely fixed on the lite hand. Bent back at 40 degrees -->
+    <!--
+    <xacro:wrist muscletrans="false" prefix="${prefix}" reflect="${reflect}" parent="${prefix}forearm">
+        <origin xyz="0 -0.010 0.213" rpy="0 0 0" />
+    </xacro:wrist>
+    -->
+    <joint name="${prefix}WRJ1" type="fixed">
+      <parent link="${prefix}forearm"/>
+      <child link="${prefix}palm"/>
+      <!-- <origin xyz="0 -0.010 0.213" rpy="-${M_PI/4} 0 0" /> -->
+      <origin xyz="0 -0.015 0.149" rpy="-${40*M_PI/180} 0 0" />
+      <axis xyz="0 ${reflect} 0" />
+    </joint>
     <!-- Palm -->
     <xacro:palm muscletrans="${muscletrans}" prefix="${prefix}" reflect="${reflect}" parent="${prefix}wrist" />

Commit message: removing commented out xacros from hand lite for tests to work better

File: sr_description/hand/xacro/hand_lite.urdf.xacro (robot description, xacro)
@@ -8,5 +8,4 @@
   <xacro:include filename="$(find sr_description)/hand/xacro/finger/fingers.urdf.xacro" />
   <xacro:include filename="$(find sr_description)/hand/xacro/thumb/thumb.urdf.xacro" />
-  <xacro:property name="M_PI" value="3.1415926535897931" />
   <!-- muscletrans is true for muscle transmission to be used, false to use motor transmission -->
   <!-- muscle is true for muscle hand or false for motor hand -->
@@ -23,13 +22,7 @@
     <!-- Wrist -->
     <!-- Completely fixed on the lite hand. Bent back at 40 degrees -->
-    <!--
-    <xacro:wrist muscletrans="false" prefix="${prefix}" reflect="${reflect}" parent="${prefix}forearm">
-        <origin xyz="0 -0.010 0.213" rpy="0 0 0" />
-    </xacro:wrist>
-    -->
     <joint name="${prefix}WRJ1" type="fixed">
       <parent link="${prefix}forearm" />
       <child link="${prefix}palm" />
-      <!-- <origin xyz="0 -0.010 0.213" rpy="-${M_PI/4} 0 0" /> -->
       <origin xyz="0 -0.015 0.149" rpy="-${40*M_PI/180} 0 0" />
       <axis xyz="0 ${reflect} 0" />
