Commit message: bigger effort limits on wrist joints

File: sr_description/hand/xacro/palm/palm.urdf.xacro (robot description, xacro)
@@ -59,5 +59,5 @@
       <axis xyz="1 0 0" />
       <limit lower="-0.78539816339744828" upper="0.6108652381980153"
-      effort="5" velocity="1.0"/>
+      effort="100" velocity="1.0"/>
       <dynamics damping="100.5"/>
     </joint>

File: sr_description/hand/xacro/wrist/wrist.urdf.xacro (robot description, xacro)
@@ -47,5 +47,5 @@
       <insert_block name="origin" />
       <axis xyz="0 1 0" />
-      <limit lower="-0.52359877559829882" upper="0.17453292519943295" effort="5" velocity="1.0"/>
+      <limit lower="-0.52359877559829882" upper="0.17453292519943295" effort="100" velocity="1.0"/>
       <dynamics damping="100.5"/>
     </joint>

Commit message: Added a wrist mount collision box (motor and muscle hand) Added more precision to the palm collision shape (still using boxes)

File: sr_description/hand/xacro/palm/palm.urdf.xacro (robot description, xacro)
@@ -28,9 +28,37 @@
       </visual>
       <collision>
-        <origin xyz="${reflect*0.011} 0 0.038" rpy="0 0 0" />
+        <origin xyz="${reflect*0.011} 0.0085 0.038" rpy="0 0 0" />
         <geometry name="${prefix}palm_collision_geom">
-          <box size="0.062 0.024 0.098" />
+          <box size="0.062 0.007 0.098" />
         </geometry>
       </collision>
+      <collision>
+        <origin xyz="${reflect*0.0005} -0.0035 0.038" rpy="0 0 0" />
+        <geometry>
+          <box size="0.041 0.017 0.098" />
+        </geometry>
+      </collision>
+      <!-- palm complement below first finger -->
+      <collision>
+        <origin xyz="${reflect*0.0315} -0.0035 0.073" rpy="0 0 0" />
+        <geometry>
+          <box size="0.021 0.017 0.028" />
+        </geometry>
+      </collision>
+      <!-- thumb pulp side -->
+      <collision>
+        <origin xyz="${reflect*0.0315} -0.0085 0.001" rpy="0 0 0" />
+        <geometry>
+          <box size="0.021 0.027 0.024" />
+        </geometry>
+      </collision>
+      <!-- thumb pulp central -->
+      <collision>
+        <origin xyz="${reflect*0.01} -0.017 0.011" rpy="0 0 0" />
+        <geometry>
+          <box size="0.022 0.010 0.044" />
+        </geometry>
+      </collision>
+      <!-- above middle finger-->
       <collision>
         <origin xyz="${reflect*0.011} 0 0.089" rpy="0 0 0" />
@@ -39,4 +67,5 @@
         </geometry>
       </collision>
+      <!-- metacarpal side-->
       <collision>
         <origin xyz="${reflect*-0.030} 0 0.009" rpy="0 0 0" />

Commit message: Fixed self collision between palm and forearm Updated an outdated rviz_motor.launch to use new sr_description loaders, added a joint_state publisher and robot_state_publisher for full interaction with the model

File: sr_description/hand/xacro/palm/palm.urdf.xacro (robot description, xacro)
@@ -36,16 +36,23 @@
       </collision>
       <collision>
-        <origin xyz="${reflect*0.0005} -0.0035 0.038"
+        <origin xyz="${-reflect*0.002} -0.0035 0.038"
         rpy="0 0 0" />
         <geometry>
-          <box size="0.041 0.017 0.098" />
+          <box size="0.036 0.017 0.098" />
         </geometry>
       </collision>
       <!-- palm complement below first finger -->
       <collision>
-        <origin xyz="${reflect*0.0315} -0.0035 0.073"
+        <origin xyz="${reflect*0.029} -0.0035 0.082"
         rpy="0 0 0" />
         <geometry>
-          <box size="0.021 0.017 0.028" />
+          <box size="0.026 0.017 0.010" />
+        </geometry>
+      </collision>
+      <collision>
+        <origin xyz="${reflect*0.0265} -0.001 0.070"
+        rpy="0.2 0 ${reflect*0.25}" />
+        <geometry>
+          <box size="0.026 0.014 0.018" />
         </geometry>
       </collision>
@@ -60,7 +67,7 @@
       <!-- thumb pulp central -->
       <collision>
-        <origin xyz="${reflect*0.01} -0.017 0.011" rpy="0 0 0" />
+        <origin xyz="${reflect*0.0125} -0.015 0.009" rpy="0 0 ${reflect*-0.48}" />
         <geometry>
-          <box size="0.022 0.010 0.044" />
+          <box size="0.022 0.005 0.040" />
         </geometry>
       </collision>
