Commit message: Fixed intend

File: sr_description/hand/xacro/palm/palm.transmission.xacro (robot description, xacro)
@@ -19,10 +19,10 @@
       <transmission name="${prefix}palm_transmission">
         <type>sr_mechanism_model/SimpleTransmission</type>
-      <actuator name="${prefix}WRJ1">
-        <mechanicalReduction>1</mechanicalReduction>
-      </actuator>
-      <joint name="${prefix}WRJ1">
-        <hardwareInterface>EffortJointInterface</hardwareInterface>
-      </joint>
+        <actuator name="${prefix}WRJ1">
+          <mechanicalReduction>1</mechanicalReduction>
+        </actuator>
+        <joint name="${prefix}WRJ1">
+          <hardwareInterface>EffortJointInterface</hardwareInterface>
+        </joint>
       </transmission>
     </xacro:unless>
