Commit message: Corrected xacro to separate muscle transmission parameter from muscle (visual) parameter Corrected the robots xacros to use new hand xacros Added some tests to visualize the resulting urdfs in rviz + move the joints Migrated all the include tags to xacro:include Removed unecessary files

File: sr_description/hand/xacro/finger/biotac/biotac.urdf.xacro (robot description, xacro)
@@ -72,5 +72,5 @@
       <dynamics damping="50.5"/>
     </joint>
-    <xacro:middle_transmission muscle="${muscle}" prefix="${prefix}" joint_prefix="${joint_prefix}"/>
+    <xacro:middle_transmission muscletrans="${muscle}" prefix="${prefix}" joint_prefix="${joint_prefix}"/>
     <link name="${prefix}${link_prefix}biotac">
       <inertial>

File: sr_description/hand/xacro/finger/distal/distal.transmission.xacro (robot description, xacro)
@@ -4,9 +4,9 @@
        xmlns:interface="http://playerstage.sourceforge.net/gazebo/xmlschema/#interface"
        xmlns:xacro="http://ros.org/wiki/xacro">
-  <!-- muscle is true for muscle hand or false for motor hand -->
+  <!-- muscletrans is true for muscle transmission or false for motor transmission -->
   <!-- prefix can be anything but usually is "r_" or  "l_" for right and left hands distinction -->
-  <xacro:macro name="distal_transmission" params="muscle prefix" >
+  <xacro:macro name="distal_transmission" params="muscletrans prefix" >
    <!-- muscle hand -->
-    <xacro:if value="${muscle}">
+    <xacro:if value="${muscletrans}">
       <transmission type="sr_mechanism_model/SimpleTransmissionForMuscle" name="${prefix}distal_transmission">
       <actuator name="${prefix}${joint_prefix}J1" />
@@ -18,5 +18,5 @@
     </xacro:if>
     <!-- motor hand -->
-    <xacro:unless value="${muscle}">
+    <xacro:unless value="${muscletrans}">
       <transmission type="sr_mechanism_model/SimpleTransmission" name="${prefix}distal_transmission">
       <actuator name="${prefix}${joint_prefix}J1" />

File: sr_description/hand/xacro/finger/distal/distal.urdf.xacro (robot description, xacro)
@@ -110,5 +110,5 @@
     </xacro:unless>
     <!-- extensions -->
-    <!--   <xacro:distal_transmission muscle="${muscle}" prefix="${prefix}" /> -->
+    <!--   <xacro:distal_transmission muscletrans="${muscle}" prefix="${prefix}" /> -->
     <xacro:distal_gazebo prefix="${prefix}" />
   </xacro:macro>

File: sr_description/hand/xacro/finger/fingers.urdf.xacro (robot description, xacro)
@@ -6,5 +6,5 @@
   <xacro:include filename="$(find sr_description)/hand/xacro/finger/lfmetacarpal/lfmetacarpal.urdf.xacro" />
   <xacro:include filename="$(find sr_description)/hand/xacro/finger/biotac/biotac.urdf.xacro" />
-  <!-- muscle is true for muscle hand or false for motor hand -->
+  <!-- muscletrans is true for muscle transmission to be used, false to use motor transmission -->
   <!-- lf is true for little finger or false for standard finger -->
   <!-- bio is true for biotac finger or false for standard finger -->
@@ -16,10 +16,10 @@
   <!-- joint_prefix prepends fingername to the joint names -->
   <!-- parent is the parent link for the first joint -->
-  <xacro:macro name="finger" params="muscle lf bio ubi eli reflect prefix link_prefix joint_prefix parent *origin *axis">
+  <xacro:macro name="finger" params="muscletrans lf bio ubi eli reflect prefix link_prefix joint_prefix parent *origin *axis">
     <!-- Little finger special case -->
     <xacro:if value="${lf}">
-      <xacro:lfmetacarpal muscle="${muscle}" prefix="${prefix}" reflect="${reflect}" parent="${parent}" />
+      <xacro:lfmetacarpal muscle="${muscletrans}" prefix="${prefix}" reflect="${reflect}" parent="${parent}" />
       <!-- Knuckle -->
-      <xacro:knuckle muscle="${muscle}" prefix="${prefix}" link_prefix="${link_prefix}" joint_prefix="${joint_prefix}" parent="${prefix}lfmetacarpal" >
+      <xacro:knuckle muscle="${muscletrans}" prefix="${prefix}" link_prefix="${link_prefix}" joint_prefix="${joint_prefix}" parent="${prefix}lfmetacarpal" >
         <insert_block name="origin" />
         <insert_block name="axis"/>
@@ -29,5 +29,5 @@
     <xacro:unless value="${lf}">
       <!-- Knuckle -->
-      <xacro:knuckle muscle="${muscle}" prefix="${prefix}" link_prefix="${link_prefix}" joint_prefix="${joint_prefix}" parent="${parent}" >
+      <xacro:knuckle muscle="${muscletrans}" prefix="${prefix}" link_prefix="${link_prefix}" joint_prefix="${joint_prefix}" parent="${parent}" >
         <insert_block name="origin" />
         <insert_block name="axis"/>
@@ -35,14 +35,14 @@
     </xacro:unless>
     <!-- Proximal -->
-    <xacro:proximal muscle="${muscle}" prefix="${prefix}" link_prefix="${link_prefix}" joint_prefix="${joint_prefix}" parent="${prefix}${link_prefix}knuckle" >
+    <xacro:proximal muscle="${muscletrans}" prefix="${prefix}" link_prefix="${link_prefix}" joint_prefix="${joint_prefix}" parent="${prefix}${link_prefix}knuckle" >
     </xacro:proximal>
     <!-- Biotac Middle -->
     <xacro:if value="${bio}">
-      <xacro:biotac_middle muscle="${muscle}" prefix="${prefix}" link_prefix="${link_prefix}" joint_prefix="${joint_prefix}" parent="${prefix}${link_prefix}proximal">
+      <xacro:biotac_middle muscle="${muscletrans}" prefix="${prefix}" link_prefix="${link_prefix}" joint_prefix="${joint_prefix}" parent="${prefix}${link_prefix}proximal">
       </xacro:biotac_middle>
     </xacro:if>
     <!-- Standard Middle -->
     <xacro:unless value="${bio}">
-      <xacro:middle muscle="${muscle}" prefix="${prefix}" link_prefix="${link_prefix}" joint_prefix="${joint_prefix}" parent="${prefix}${link_prefix}proximal" >
+      <xacro:middle muscle="${muscletrans}" prefix="${prefix}" link_prefix="${link_prefix}" joint_prefix="${joint_prefix}" parent="${prefix}${link_prefix}proximal" >
       </xacro:middle>
     </xacro:unless>
@@ -50,5 +50,5 @@
     <!-- only if finger is not biotac  -->
     <xacro:unless value="${bio}">
-       <xacro:distal muscle="${muscle}" bio="${bio}" ubi="${ubi}" eli="${eli}" prefix="${prefix}" link_prefix="${link_prefix}" joint_prefix="${joint_prefix}" parent="${prefix}${link_prefix}middle" >
+       <xacro:distal muscle="${muscletrans}" bio="${bio}" ubi="${ubi}" eli="${eli}" prefix="${prefix}" link_prefix="${link_prefix}" joint_prefix="${joint_prefix}" parent="${prefix}${link_prefix}middle" >
        </xacro:distal>
     </xacro:unless>

File: sr_description/hand/xacro/finger/knuckle/knuckle.transmission.xacro (robot description, xacro)
@@ -4,9 +4,9 @@
        xmlns:interface="http://playerstage.sourceforge.net/gazebo/xmlschema/#interface"
        xmlns:xacro="http://ros.org/wiki/xacro">
-  <!-- muscle is true for muscle hand or false for motor hand -->
+  <!-- muscletrans is true for muscle transmission or false for motor transmission -->
   <!-- prefix can be anything but usually is "r_" or  "l_" for right and left hands distinction -->
-  <xacro:macro name="knuckle_transmission" params="muscle prefix joint_prefix" >
+  <xacro:macro name="knuckle_transmission" params="muscletrans prefix joint_prefix" >
    <!-- muscle hand -->
-    <xacro:if value="${muscle}">
+    <xacro:if value="${muscletrans}">
       <transmission type="sr_mechanism_model/SimpleTransmissionForMuscle" name="${prefix}knuckle_transmission">
       <actuator name="${prefix}${joint_prefix}J4" />
@@ -18,5 +18,5 @@
     </xacro:if>
     <!-- motor hand -->
-    <xacro:unless value="${muscle}">
+    <xacro:unless value="${muscletrans}">
       <transmission type="sr_mechanism_model/SimpleTransmission" name="${prefix}knuckle_transmission">
       <actuator name="${prefix}${joint_prefix}J4" />

File: sr_description/hand/xacro/finger/knuckle/knuckle.urdf.xacro (robot description, xacro)
@@ -45,5 +45,5 @@
     </joint>
     <!-- extensions -->
-    <xacro:knuckle_transmission muscle="${muscle}" prefix="${prefix}" joint_prefix="${joint_prefix}" />
+    <xacro:knuckle_transmission muscletrans="${muscle}" prefix="${prefix}" joint_prefix="${joint_prefix}" />
     <xacro:knuckle_gazebo prefix="${prefix}" />
   </xacro:macro>

File: sr_description/hand/xacro/finger/lfmetacarpal/lfmetacarpal.transmission.xacro (robot description, xacro)
@@ -4,9 +4,9 @@
        xmlns:interface="http://playerstage.sourceforge.net/gazebo/xmlschema/#interface"
        xmlns:xacro="http://ros.org/wiki/xacro">
-  <!-- muscle is true for muscle hand or false for motor hand -->
+  <!-- muscletrans is true for muscle transmission or false for motor transmission -->
   <!-- prefix can be anything but usually is "r_" or  "l_" for right and left hands distinction -->
-  <xacro:macro name="lfmetacarpal_transmission" params="muscle prefix" >
+  <xacro:macro name="lfmetacarpal_transmission" params="muscletrans prefix" >
    <!-- muscle hand -->
-    <xacro:if value="${muscle}">
+    <xacro:if value="${muscletrans}">
       <transmission type="sr_mechanism_model/SimpleTransmissionForMuscle" name="${prefix}lfmetacarpal_transmission">
       <actuator name="${prefix}LFJ5" />
@@ -18,5 +18,5 @@
     </xacro:if>
     <!-- motor hand -->
-    <xacro:unless value="${muscle}">
+    <xacro:unless value="${muscletrans}">
       <transmission type="sr_mechanism_model/SimpleTransmission" name="${prefix}lfmetacarpal_transmission">
       <actuator name="${prefix}LFJ5" />

File: sr_description/hand/xacro/finger/lfmetacarpal/lfmetacarpal.urdf.xacro (robot description, xacro)
@@ -43,5 +43,5 @@
     </joint>
     <!-- extensions -->
-    <xacro:lfmetacarpal_transmission muscle="${muscle}" prefix="${prefix}" />
+    <xacro:lfmetacarpal_transmission muscletrans="${muscle}" prefix="${prefix}" />
     <xacro:lfmetacarpal_gazebo prefix="${prefix}" />
   </xacro:macro>

File: sr_description/hand/xacro/finger/middle/middle.transmission.xacro (robot description, xacro)
@@ -4,9 +4,9 @@
        xmlns:interface="http://playerstage.sourceforge.net/gazebo/xmlschema/#interface"
        xmlns:xacro="http://ros.org/wiki/xacro">
-  <!-- muscle is true for muscle hand or false for motor hand -->
+  <!-- muscletrans is true for muscle transmission or false for motor transmission -->
   <!-- prefix can be anything but usually is "r_" or  "l_" for right and left hands distinction -->
-  <xacro:macro name="middle_transmission" params="muscle prefix joint_prefix" >
+  <xacro:macro name="middle_transmission" params="muscletrans prefix joint_prefix" >
    <!-- muscle hand -->
-    <xacro:if value="${muscle}">
+    <xacro:if value="${muscletrans}">
       <transmission type="sr_mechanism_model/J0TransmissionForMuscle" name="${prefix}middle_transmission">
       <actuator name="${prefix}${joint_prefix}J0" />
@@ -19,5 +19,5 @@
     </xacro:if>
     <!-- motor hand -->
-    <xacro:unless value="${muscle}">
+    <xacro:unless value="${muscletrans}">
       <transmission type="sr_mechanism_model/J0Transmission" name="${prefix}middle_transmission">
       <actuator name="${prefix}${joint_prefix}J0" />

File: sr_description/hand/xacro/finger/middle/middle.urdf.xacro (robot description, xacro)
@@ -44,5 +44,5 @@
     </joint>
     <!-- extensions -->
-    <xacro:middle_transmission muscle="${muscle}" prefix="${prefix}" joint_prefix="${joint_prefix}"/>
+    <xacro:middle_transmission muscletrans="${muscle}" prefix="${prefix}" joint_prefix="${joint_prefix}"/>
     <xacro:middle_gazebo prefix="${prefix}" />
   </xacro:macro>

File: sr_description/hand/xacro/finger/proximal/proximal.transmission.xacro (robot description, xacro)
@@ -4,9 +4,9 @@
        xmlns:interface="http://playerstage.sourceforge.net/gazebo/xmlschema/#interface"
        xmlns:xacro="http://ros.org/wiki/xacro">
-  <!-- muscle is true for muscle hand or false for motor hand -->
+  <!-- muscletrans is true for muscle transmission or false for motor transmission -->
   <!-- prefix can be anything but usually is "r_" or  "l_" for right and left hands distinction -->
-  <xacro:macro name="proximal_transmission" params="muscle prefix joint_prefix" >
+  <xacro:macro name="proximal_transmission" params="muscletrans prefix joint_prefix" >
    <!-- muscle hand -->
-    <xacro:if value="${muscle}">
+    <xacro:if value="${muscletrans}">
       <transmission type="sr_mechanism_model/SimpleTransmissionForMuscle" name="${prefix}proximal_transmission">
       <actuator name="${prefix}${joint_prefix}J3" />
@@ -18,5 +18,5 @@
     </xacro:if>
     <!-- motor hand -->
-    <xacro:unless value="${muscle}">
+    <xacro:unless value="${muscletrans}">
       <transmission type="sr_mechanism_model/SimpleTransmission" name="${prefix}proximal_transmission">
       <actuator name="${prefix}${joint_prefix}J3" />

File: sr_description/hand/xacro/finger/proximal/proximal.urdf.xacro (robot description, xacro)
@@ -44,5 +44,5 @@
     </joint>
     <!-- extensions -->
-    <xacro:proximal_transmission muscle="${muscle}" prefix="${prefix}" joint_prefix="${joint_prefix}"/>
+    <xacro:proximal_transmission muscletrans="${muscle}" prefix="${prefix}" joint_prefix="${joint_prefix}"/>
     <xacro:proximal_gazebo prefix="${prefix}" />
   </xacro:macro>

File: sr_description/hand/xacro/forearm/forearm.urdf.xacro (robot description, xacro)
@@ -1,3 +1,5 @@
 <robot xmlns:xacro="http://ros.org/wiki/xacro">
+  <!-- muscle is true for muscle hand or false for motor hand -->
+  <!-- prefix can be anything but usually is "r_" or  "l_" for right and left hands distinction -->
   <xacro:macro name="forearm" params="muscle prefix">
       <link name="${prefix}forearm">

File: sr_description/hand/xacro/palm/palm.transmission.xacro (robot description, xacro)
@@ -4,9 +4,9 @@
        xmlns:interface="http://playerstage.sourceforge.net/gazebo/xmlschema/#interface"
        xmlns:xacro="http://ros.org/wiki/xacro">
-  <!-- muscle is true for muscle hand or false for motor hand -->
+  <!-- muscletrans is true for muscle transmission or false for motor transmission -->
   <!-- prefix can be anything but usually is "r_" or  "l_" for right and left hands distinction -->
-  <xacro:macro name="shadowhand_palm_transmission" params="muscle prefix" >
+  <xacro:macro name="shadowhand_palm_transmission" params="muscletrans prefix" >
    <!-- muscle hand -->
-    <xacro:if value="${muscle}">
+    <xacro:if value="${muscletrans}">
       <transmission type="sr_mechanism_model/SimpleTransmissionForMuscle" name="${prefix}palm_transmission">
       <actuator name="${prefix}WRJ1" />
@@ -18,5 +18,5 @@
     </xacro:if>
     <!-- motor hand -->
-    <xacro:unless value="${muscle}">
+    <xacro:unless value="${muscletrans}">
       <transmission type="sr_mechanism_model/SimpleTransmission" name="${prefix}palm_transmission">
       <actuator name="${prefix}WRJ1" />

File: sr_description/hand/xacro/palm/palm.urdf.xacro (robot description, xacro)
@@ -1,4 +1,4 @@
 <robot xmlns:xacro="http://ros.org/wiki/xacro"
-		 xmlns:sensor="http://playerstage.sourceforge.net/gazebo/xmlschema/#sensor"
+       xmlns:sensor="http://playerstage.sourceforge.net/gazebo/xmlschema/#sensor"
        xmlns:controller="http://playerstage.sourceforge.net/gazebo/xmlschema/#controller"
        xmlns:joint="http://playerstage.sourceforge.net/gazebo/xmlschema/#slider"
@@ -8,9 +8,9 @@
   <xacro:include filename="$(find sr_description)/hand/xacro/palm/palm.gazebo.xacro" />
   <xacro:include filename="$(find sr_description)/hand/xacro/palm/palm.transmission.xacro" />
-  <!-- muscle is true for muscle hand or false for motor hand -->
+  <!-- muscletrans is true for muscle transmission or false for motor transmission -->
   <!-- prefix can be anything but usually is "r_" or  "l_" for right and left hands distinction -->
   <!-- reflect is either 1 (for right hand) or -1 (for left hand) -->
   <!-- parent is the parent link for the joint -->
-  <xacro:macro name="palm" params="muscle prefix reflect parent">
+  <xacro:macro name="palm" params="muscletrans prefix reflect parent">
     <link name="${prefix}palm">
       <inertial>
@@ -44,5 +44,5 @@
     </joint>
     <!-- extensions -->
-    <xacro:shadowhand_palm_transmission muscle="${muscle}" prefix="${prefix}" />
+    <xacro:shadowhand_palm_transmission muscletrans="${muscletrans}" prefix="${prefix}" />
     <xacro:shadowhand_palm_gazebo prefix="${prefix}" />
   </xacro:macro>

File: sr_description/hand/xacro/three_biotac_fingers_hand.urdf.xacro (robot description, xacro)
@@ -20,5 +20,5 @@
     <xacro:forearm muscle="${muscle}" prefix="${prefix}" />
     <!-- Wrist -->
-		<xacro:if value="${muscle}">
+    <xacro:if value="${muscle}">
 			<xacro:wrist muscletrans="${muscletrans}" prefix="${prefix}" reflect="${reflect}" parent="${prefix}forearm">
 			<origin xyz="0 0 0.4096" rpy="0 0 0" />
@@ -32,26 +32,26 @@
     <!-- Palm -->
     <xacro:palm muscletrans="${muscletrans}" prefix="${prefix}" reflect="${reflect}" parent="${prefix}wrist" />
-    <!-- First Finger -->
-    <xacro:finger muscletrans="${muscletrans}" lf="false" bio="${bio}" ubi="${ubi}" eli="${eli}" prefix="${prefix}" reflect="${reflect}" link_prefix="ff" joint_prefix="FF" parent="${prefix}palm">
+    <!-- First Finger Biotac -->
+    <xacro:finger muscletrans="${muscletrans}" lf="false" bio="true" ubi="false" eli="false" prefix="${prefix}" reflect="${reflect}" link_prefix="ff" joint_prefix="FF" parent="${prefix}palm">
       <origin xyz="${reflect*0.033} 0 0.095" rpy="0 0 0" />
       <axis xyz="0 ${-1*reflect} 0" />
     </xacro:finger>
-    <!-- Middle Finger -->
-    <xacro:finger muscletrans="${muscletrans}" lf="false" bio="${bio}" ubi="${ubi}" eli="${eli}" prefix="${prefix}" reflect="${reflect}" link_prefix="mf" joint_prefix="MF" parent="${prefix}palm">
+    <!-- Middle Finger Biotac -->
+    <xacro:finger muscletrans="${muscletrans}" lf="false" bio="true" ubi="false" eli="false" prefix="${prefix}" reflect="${reflect}" link_prefix="mf" joint_prefix="MF" parent="${prefix}palm">
       <origin xyz="${reflect*0.011} 0 0.099" rpy="0 0 0" />
       <axis xyz="0 ${-1*reflect} 0" />
     </xacro:finger>
     <!-- Ring Finger -->
-    <xacro:finger muscletrans="${muscletrans}" lf="false" bio="${bio}" ubi="${ubi}" eli="${eli}" prefix="${prefix}" reflect="${reflect}" link_prefix="rf" joint_prefix="RF" parent="${prefix}palm">
+    <xacro:finger muscletrans="${muscletrans}" lf="false" bio="false" ubi="false" eli="false" prefix="${prefix}" reflect="${reflect}" link_prefix="rf" joint_prefix="RF" parent="${prefix}palm">
       <origin xyz="${reflect*-0.011} 0 0.095" rpy="0 0 0" />
       <axis xyz="0 ${reflect} 0" />
     </xacro:finger>
     <!-- Little Finger  -->
-    <xacro:finger muscletrans="${muscletrans}" lf="true" bio="${bio}" ubi="${ubi}" eli="${eli}" prefix="${prefix}" reflect="${reflect}" link_prefix="lf" joint_prefix="LF" parent="${prefix}palm">
+    <xacro:finger muscletrans="${muscletrans}" lf="true" bio="false" ubi="false" eli="false" prefix="${prefix}" reflect="${reflect}" link_prefix="lf" joint_prefix="LF" parent="${prefix}palm">
       <origin xyz="0 0 0.06579" rpy="0 0 0" />
       <axis xyz="0 ${reflect} 0" />
     </xacro:finger>
-		<!-- Thumb  -->
-    <xacro:thumb muscletrans="${muscletrans}" bio="${bio}" ubi="${ubi}" eli="${eli}" prefix="${prefix}" reflect="${reflect}" parent="${prefix}palm">
+		<!-- Thumb Biotac -->
+    <xacro:thumb muscletrans="${muscletrans}" bio="true" ubi="false" eli="false" prefix="${prefix}" reflect="${reflect}" parent="${prefix}palm">
     </xacro:thumb>
   </xacro:macro>

File: sr_description/hand/xacro/three_fingers_hand.urdf.xacro (robot description, xacro)
@@ -20,14 +20,14 @@
     <xacro:forearm muscle="${muscle}" prefix="${prefix}" />
     <!-- Wrist -->
-		<xacro:if value="${muscle}">
+    <xacro:if value="${muscle}">
 			<xacro:wrist muscletrans="${muscletrans}" prefix="${prefix}" reflect="${reflect}" parent="${prefix}forearm">
-			<origin xyz="0 0 0.4096" rpy="0 0 0" />
-			</xacro:wrist>
-		</xacro:if>
-		<xacro:unless value="${muscle}">
-			<xacro:wrist muscletrans="false" prefix="${prefix}" reflect="${reflect}" parent="${prefix}forearm">
-			<origin xyz="0 -0.010 0.213" rpy="0 0 0" />
-			</xacro:wrist>
-		</xacro:unless>
+        <origin xyz="0 0 0.4096" rpy="0 0 0" />
+      </xacro:wrist>
+    </xacro:if>
+    <xacro:unless value="${muscle}">
+			<xacro:wrist muscletrans="${muscletrans}" prefix="${prefix}" reflect="${reflect}" parent="${prefix}forearm">
+        <origin xyz="0 -0.010 0.213" rpy="0 0 0" />
+      </xacro:wrist>
+    </xacro:unless>
     <!-- Palm -->
     <xacro:palm muscletrans="${muscletrans}" prefix="${prefix}" reflect="${reflect}" parent="${prefix}wrist" />
@@ -42,14 +42,4 @@
       <axis xyz="0 ${-1*reflect} 0" />
     </xacro:finger>
-    <!-- Ring Finger -->
-    <xacro:finger muscletrans="${muscletrans}" lf="false" bio="${bio}" ubi="${ubi}" eli="${eli}" prefix="${prefix}" reflect="${reflect}" link_prefix="rf" joint_prefix="RF" parent="${prefix}palm">
-      <origin xyz="${reflect*-0.011} 0 0.095" rpy="0 0 0" />
-      <axis xyz="0 ${reflect} 0" />
-    </xacro:finger>
-    <!-- Little Finger  -->
-    <xacro:finger muscletrans="${muscletrans}" lf="true" bio="${bio}" ubi="${ubi}" eli="${eli}" prefix="${prefix}" reflect="${reflect}" link_prefix="lf" joint_prefix="LF" parent="${prefix}palm">
-      <origin xyz="0 0 0.06579" rpy="0 0 0" />
-      <axis xyz="0 ${reflect} 0" />
-    </xacro:finger>
 		<!-- Thumb  -->
     <xacro:thumb muscletrans="${muscletrans}" bio="${bio}" ubi="${ubi}" eli="${eli}" prefix="${prefix}" reflect="${reflect}" parent="${prefix}palm">

File: sr_description/hand/xacro/thumb/thbase.transmission.xacro (robot description, xacro)
@@ -4,9 +4,9 @@
        xmlns:interface="http://playerstage.sourceforge.net/gazebo/xmlschema/#interface"
        xmlns:xacro="http://ros.org/wiki/xacro">
-  <!-- muscle is true for muscle hand or false for motor hand -->
+  <!-- muscletrans is true for muscle transmission or false for motor transmission -->
   <!-- prefix can be anything but usually is "r_" or  "l_" for right and left hands distinction -->
-  <xacro:macro name="thbase_transmission" params="muscle prefix" >
+  <xacro:macro name="thbase_transmission" params="muscletrans prefix" >
    <!-- muscle hand -->
-    <xacro:if value="${muscle}">
+    <xacro:if value="${muscletrans}">
       <transmission type="sr_mechanism_model/SimpleTransmissionForMuscle" name="${prefix}thbase_transmission">
       <actuator name="${prefix}THJ5" />
@@ -18,5 +18,5 @@
     </xacro:if>
     <!-- motor hand -->
-    <xacro:unless value="${muscle}">
+    <xacro:unless value="${muscletrans}">
       <transmission type="sr_mechanism_model/SimpleTransmission" name="${prefix}thbase_transmission">
       <actuator name="${prefix}THJ5" />

File: sr_description/hand/xacro/thumb/thbase.urdf.xacro (robot description, xacro)
@@ -44,5 +44,5 @@
     </joint>
     <!-- extensions -->
-    <xacro:thbase_transmission muscle="${muscle}" prefix="${prefix}"/>
+    <xacro:thbase_transmission muscletrans="${muscle}" prefix="${prefix}"/>
     <xacro:thbase_gazebo prefix="${prefix}" />
   </xacro:macro>
