Commit message: Corrected xacro to separate muscle transmission parameter from muscle (visual) parameter Corrected the robots xacros to use new hand xacros Added some tests to visualize the resulting urdfs in rviz + move the joints Migrated all the include tags to xacro:include Removed unecessary files

File: sr_description/hand/xacro/thumb/thdistal.transmission.xacro (robot description, xacro)
@@ -4,9 +4,9 @@
        xmlns:interface="http://playerstage.sourceforge.net/gazebo/xmlschema/#interface"
        xmlns:xacro="http://ros.org/wiki/xacro">
-  <!-- muscle is true for muscle hand or false for motor hand -->
+  <!-- muscletrans is true for muscle transmission or false for motor transmission -->
   <!-- prefix can be anything but usually is "r_" or  "l_" for right and left hands distinction -->
-  <xacro:macro name="thdistal_transmission" params="muscle prefix" >
+  <xacro:macro name="thdistal_transmission" params="muscletrans prefix" >
    <!-- muscle hand -->
-    <xacro:if value="${muscle}">
+    <xacro:if value="${muscletrans}">
       <transmission type="sr_mechanism_model/SimpleTransmissionForMuscle" name="${prefix}thdistal_transmission">
       <actuator name="${prefix}THJ1" />
@@ -18,5 +18,5 @@
     </xacro:if>
     <!-- motor hand -->
-    <xacro:unless value="${muscle}">
+    <xacro:unless value="${muscletrans}">
       <transmission type="sr_mechanism_model/SimpleTransmission" name="${prefix}thdistal_transmission">
       <actuator name="${prefix}THJ1" />

Commit message: Corrected transmission xacro ton re-include link_prefix (fixes bug #2453)

File: sr_description/hand/xacro/finger/biotac/biotac.urdf.xacro (robot description, xacro)
@@ -72,5 +72,5 @@
       <dynamics damping="50.5"/>
     </joint>
-    <xacro:middle_transmission muscletrans="${muscle}" prefix="${prefix}" joint_prefix="${joint_prefix}"/>
+    <xacro:middle_transmission muscletrans="${muscle}" prefix="${prefix}" joint_prefix="${joint_prefix}" link_prefix="${link_prefix}"/>
     <link name="${prefix}${link_prefix}biotac">
       <inertial>

File: sr_description/hand/xacro/finger/distal/distal.transmission.xacro (robot description, xacro)
@@ -6,8 +6,10 @@
   <!-- muscletrans is true for muscle transmission or false for motor transmission -->
   <!-- prefix can be anything but usually is "r_" or  "l_" for right and left hands distinction -->
-  <xacro:macro name="distal_transmission" params="muscletrans prefix" >
+  <!-- link_prefix prepends fingername to the link names -->
+  <!-- joint_prefix prepends fingername to the joint names -->
+  <xacro:macro name="distal_transmission" params="muscletrans prefix joint_prefix link_prefix" >
    <!-- muscle hand -->
     <xacro:if value="${muscletrans}">
-      <transmission type="sr_mechanism_model/SimpleTransmissionForMuscle" name="${prefix}distal_transmission">
+      <transmission type="sr_mechanism_model/SimpleTransmissionForMuscle" name="${prefix}${link_prefix}distal_transmission">
       <actuator name="${prefix}${joint_prefix}J1" />
       <joint name="${prefix}${joint_prefix}J1" />
@@ -19,5 +21,5 @@
     <!-- motor hand -->
     <xacro:unless value="${muscletrans}">
-      <transmission type="sr_mechanism_model/SimpleTransmission" name="${prefix}distal_transmission">
+      <transmission type="sr_mechanism_model/SimpleTransmission" name="${prefix}${link_prefix}distal_transmission">
       <actuator name="${prefix}${joint_prefix}J1" />
       <joint name="${prefix}${joint_prefix}J1" />

File: sr_description/hand/xacro/finger/knuckle/knuckle.transmission.xacro (robot description, xacro)
@@ -6,8 +6,10 @@
   <!-- muscletrans is true for muscle transmission or false for motor transmission -->
   <!-- prefix can be anything but usually is "r_" or  "l_" for right and left hands distinction -->
-  <xacro:macro name="knuckle_transmission" params="muscletrans prefix joint_prefix" >
+  <!-- link_prefix prepends fingername to the link names -->
+  <!-- joint_prefix prepends fingername to the joint names -->
+  <xacro:macro name="knuckle_transmission" params="muscletrans prefix joint_prefix link_prefix" >
    <!-- muscle hand -->
     <xacro:if value="${muscletrans}">
-      <transmission type="sr_mechanism_model/SimpleTransmissionForMuscle" name="${prefix}knuckle_transmission">
+      <transmission type="sr_mechanism_model/SimpleTransmissionForMuscle" name="${prefix}${link_prefix}knuckle_transmission">
       <actuator name="${prefix}${joint_prefix}J4" />
       <joint name="${prefix}${joint_prefix}J4" />
@@ -19,5 +21,5 @@
     <!-- motor hand -->
     <xacro:unless value="${muscletrans}">
-      <transmission type="sr_mechanism_model/SimpleTransmission" name="${prefix}knuckle_transmission">
+      <transmission type="sr_mechanism_model/SimpleTransmission" name="${prefix}${link_prefix}knuckle_transmission">
       <actuator name="${prefix}${joint_prefix}J4" />
       <joint name="${prefix}${joint_prefix}J4" />

File: sr_description/hand/xacro/finger/knuckle/knuckle.urdf.xacro (robot description, xacro)
@@ -45,5 +45,5 @@
     </joint>
     <!-- extensions -->
-    <xacro:knuckle_transmission muscletrans="${muscle}" prefix="${prefix}" joint_prefix="${joint_prefix}" />
+    <xacro:knuckle_transmission muscletrans="${muscle}" prefix="${prefix}" joint_prefix="${joint_prefix}" link_prefix="${link_prefix}"/>
     <xacro:knuckle_gazebo prefix="${prefix}" />
   </xacro:macro>

File: sr_description/hand/xacro/finger/middle/middle.transmission.xacro (robot description, xacro)
@@ -6,8 +6,10 @@
   <!-- muscletrans is true for muscle transmission or false for motor transmission -->
   <!-- prefix can be anything but usually is "r_" or  "l_" for right and left hands distinction -->
-  <xacro:macro name="middle_transmission" params="muscletrans prefix joint_prefix" >
+  <!-- link_prefix prepends fingername to the link names -->
+  <!-- joint_prefix prepends fingername to the joint names -->
+  <xacro:macro name="middle_transmission" params="muscletrans prefix joint_prefix link_prefix" >
    <!-- muscle hand -->
     <xacro:if value="${muscletrans}">
-      <transmission type="sr_mechanism_model/J0TransmissionForMuscle" name="${prefix}middle_transmission">
+      <transmission type="sr_mechanism_model/J0TransmissionForMuscle" name="${prefix}${link_prefix}middle_transmission">
       <actuator name="${prefix}${joint_prefix}J0" />
       <joint1 name="${prefix}${joint_prefix}J1" />
@@ -20,5 +22,5 @@
     <!-- motor hand -->
     <xacro:unless value="${muscletrans}">
-      <transmission type="sr_mechanism_model/J0Transmission" name="${prefix}middle_transmission">
+      <transmission type="sr_mechanism_model/J0Transmission" name="${prefix}${link_prefix}middle_transmission">
       <actuator name="${prefix}${joint_prefix}J0" />
       <joint1 name="${prefix}${joint_prefix}J1" />

File: sr_description/hand/xacro/finger/middle/middle.urdf.xacro (robot description, xacro)
@@ -44,5 +44,5 @@
     </joint>
     <!-- extensions -->
-    <xacro:middle_transmission muscletrans="${muscle}" prefix="${prefix}" joint_prefix="${joint_prefix}"/>
+    <xacro:middle_transmission muscletrans="${muscle}" prefix="${prefix}" joint_prefix="${joint_prefix}" link_prefix="${link_prefix}"/>
     <xacro:middle_gazebo prefix="${prefix}" />
   </xacro:macro>

File: sr_description/hand/xacro/finger/proximal/proximal.transmission.xacro (robot description, xacro)
@@ -6,8 +6,10 @@
   <!-- muscletrans is true for muscle transmission or false for motor transmission -->
   <!-- prefix can be anything but usually is "r_" or  "l_" for right and left hands distinction -->
-  <xacro:macro name="proximal_transmission" params="muscletrans prefix joint_prefix" >
+  <!-- link_prefix prepends fingername to the link names -->
+  <!-- joint_prefix prepends fingername to the joint names -->
+  <xacro:macro name="proximal_transmission" params="muscletrans prefix joint_prefix link_prefix" >
    <!-- muscle hand -->
     <xacro:if value="${muscletrans}">
-      <transmission type="sr_mechanism_model/SimpleTransmissionForMuscle" name="${prefix}proximal_transmission">
+      <transmission type="sr_mechanism_model/SimpleTransmissionForMuscle" name="${prefix}${link_prefix}proximal_transmission">
       <actuator name="${prefix}${joint_prefix}J3" />
       <joint name="${prefix}${joint_prefix}J3" />
@@ -19,5 +21,5 @@
     <!-- motor hand -->
     <xacro:unless value="${muscletrans}">
-      <transmission type="sr_mechanism_model/SimpleTransmission" name="${prefix}proximal_transmission">
+      <transmission type="sr_mechanism_model/SimpleTransmission" name="${prefix}${link_prefix}proximal_transmission">
       <actuator name="${prefix}${joint_prefix}J3" />
       <joint name="${prefix}${joint_prefix}J3" />

File: sr_description/hand/xacro/finger/proximal/proximal.urdf.xacro (robot description, xacro)
@@ -44,5 +44,5 @@
     </joint>
     <!-- extensions -->
-    <xacro:proximal_transmission muscletrans="${muscle}" prefix="${prefix}" joint_prefix="${joint_prefix}"/>
+    <xacro:proximal_transmission muscletrans="${muscle}" prefix="${prefix}" joint_prefix="${joint_prefix}" link_prefix="${link_prefix}"/>
     <xacro:proximal_gazebo prefix="${prefix}" />
   </xacro:macro>

File: sr_description/hand/xacro/wrist/wrist.urdf.xacro (robot description, xacro)
@@ -28,5 +28,5 @@
     </link>
     <gazebo reference="${prefix}wrist">
-      <material>Grey2</material>
+      <material>Gazebo/White</material>
       <selfCollide>false</selfCollide>
     </gazebo>

Commit message: Merged F_inertia into hydro

File: sr_description/hand/xacro/finger/biotac/biotac.urdf.xacro (robot description, xacro)
@@ -17,5 +17,6 @@
         <origin xyz="0 0 0.0125" rpy="0 0 0" />
         <mass value="0.012" />
-        <inertia  ixx="0.1" ixy="0.0"  ixz="0.0"  iyy="0.1"  iyz="0.0" izz="0.01" />
+      <inertia  ixx="0.00031" ixy="0.0"  ixz="0.0"  iyy="0.00031"  iyz="0.0"
+        izz="0.000053" />
       </inertial>
       <visual>
@@ -71,6 +72,6 @@
       <origin xyz="0 0 0.02" rpy="0 0 0" />
       <axis xyz="1 0 0" />
-      <limit lower="${20*M_PI/180}" upper="${20.1*M_PI/180}" effort="10" velocity="0.1" />
-      <dynamics damping="50.5"/>
+      <limit lower="${20*M_PI/180}" upper="${20.1*M_PI/180}" effort="2" velocity="0.1" />
+      <dynamics damping="0.1"/>
     </joint>
     <xacro:middle_transmission muscletrans="${muscle}" prefix="${prefix}" joint_prefix="${joint_prefix}" link_prefix="${link_prefix}"/>
@@ -125,5 +126,6 @@
        <mass value="0.001" />
        <origin xyz="0 0 0" rpy="0 0 0" />
-       <inertia  ixx="1" ixy="0"  ixz="0"  iyy="1"  iyz="0" izz="1" />
+        <inertia  ixx="0.00031" ixy="0.0"  ixz="0.0"  iyy="0.00031"  iyz="0.0"
+        izz="0.000053" />
       </inertial>
       <visual>

File: sr_description/hand/xacro/finger/distal/distal.urdf.xacro (robot description, xacro)
@@ -20,7 +20,7 @@
       <inertial>
         <mass value="0.010" />
-        <origin xyz="0 0 0.013" />
-        <inertia  ixx="0.1" ixy="0.0"  ixz="0.0"  iyy="0.1"  iyz="0.0"
-        izz="0.0" />
+        <origin xyz="0 0 0.012" />
+        <inertia  ixx="0.001" ixy="0.0"  ixz="0.0"  iyy="0.001"  iyz="0.0"
+        izz="0.00025" />
       </inertial>
       <visual>
@@ -89,8 +89,8 @@
       <xacro:unless value="${bio}">
 				<!-- standard distal joint -->
-        <limit lower="0" upper="${M_PI/2}" effort="10"
+        <limit lower="0" upper="${M_PI/2}" effort="2"
           velocity="1.0" />
       </xacro:unless>
-      <dynamics damping="50.5"/>
+      <dynamics damping="0.1"/>
     </joint>
     <link name="${prefix}${link_prefix}tip">

File: sr_description/hand/xacro/thumb/thdistal.urdf.xacro (robot description, xacro)
@@ -21,6 +21,7 @@
 					<origin xyz="0 0 0" rpy="0 0 0" />
 					<mass value="0.01" />
-					<inertia  ixx="0.1" ixy="0.0"  ixz="0.0"  iyy="0.1"  iyz="0.0" izz="0.01" />
-				</inertial>
+					 <inertia  ixx="0.0007" ixy="0.0"  ixz="0.0"  iyy="0.0007"  iyz="0.0"
+        izz="0.00010" />
+        </inertial>
 			</link>
 			<joint name="${prefix}THJ1" type="revolute">
@@ -30,5 +31,5 @@
 				<axis xyz="1 0 0" />
 				<limit lower="${20*M_PI/180}" upper="${20.1*M_PI/180}" effort="10" velocity="0.1" />
-				<dynamics damping="50.5"/>
+				<dynamics damping="0.1"/>
 			</joint>
 			<link name="${prefix}thbiotac">
@@ -36,5 +37,6 @@
 					<origin xyz="0 0 0" rpy="0 0 0" />
 					<mass value="0.2" />
-					<inertia  ixx="1" ixy="0.0"  ixz="0.0"  iyy="1"  iyz="0.0" izz="1" />
+					 <inertia  ixx="0.0007" ixy="0.0"  ixz="0.0"  iyy="0.0007"  iyz="0.0"
+        izz="0.00010" />
 				</inertial>
 				<visual>
@@ -83,5 +85,5 @@
 				 <mass value="0.001" />
 				 <origin xyz="0 0 0" rpy="0 0 0" />
-				 <inertia  ixx="1" ixy="0"  ixz="0"  iyy="1"  iyz="0" izz="1" />
+				 <inertia  ixx="0" ixy="0"  ixz="0"  iyy="0"  iyz="0" izz="0" />
 				</inertial>
 				<visual>
@@ -111,6 +113,6 @@
 					<mass value="0.016" />
 					<origin xyz="0 0 0.01375" rpy="0 0 0"/>
-					<inertia  ixx="0.1" ixy="0.0"  ixz="0.0"  iyy="0.1"  iyz="0.0"
-							izz="0.1" />
+					 <inertia  ixx="0.0007" ixy="0.0"  ixz="0.0"  iyy="0.0007"  iyz="0.0"
+        izz="0.00010" />
 				</inertial>
 				<visual>
@@ -163,5 +165,5 @@
 				<axis xyz="1 0 0" />
 				<limit lower="0" upper="${90.0*M_PI/180}" effort="10" velocity="1.0" />
-				<dynamics damping="50.5"/>
+				<dynamics damping="0.1"/>
 			</joint>
 			<link name="${prefix}thtip">

File: sr_description/hand/xacro/wrist/wrist.urdf.xacro (robot description, xacro)
@@ -10,5 +10,5 @@
 		  <origin xyz="0 0 0" rpy="0 0 0" />
 		  <mass value="0.1" />
-		  <inertia  ixx="0.120" ixy="0.0"  ixz="0.0"  iyy="0.148"  iyz="0.0" izz="0.0438" />
+		  <inertia  ixx="0.0120" ixy="0.0"  ixz="0.0"  iyy="0.0148"  iyz="0.0" izz="0.00438" />
       </inertial>
       <visual>
@@ -36,6 +36,6 @@
       <insert_block name="origin" />
       <axis xyz="0 ${reflect} 0" />
-      <limit lower="${-30/180*M_PI}" upper="${10/180*M_PI}" effort="5" velocity="1.0"/>
-      <dynamics damping="100.5"/>
+      <limit lower="${-30/180*M_PI}" upper="${10/180*M_PI}" effort="30" velocity="1.0"/>
+      <dynamics damping="0.1"/>
     </joint>
     <!-- extensions -->

Commit message: Fixed the collision sensors for new gazebo (pending checks)

File: sr_description/hand/xacro/finger/biotac/biotac.urdf.xacro (robot description, xacro)
@@ -39,5 +39,5 @@
         <update_rate>1000.0</update_rate>
         <contact>
-          <collision>${prefix}${link_prefix}adapter_geom</collision>
+          <collision>${prefix}${link_prefix}adapter_collision</collision>
           <topic>${prefix}${link_prefix}adapter_collision</topic>
         </contact>
@@ -102,5 +102,5 @@
         <update_rate>1000.0</update_rate>
         <contact>
-          <collision>${prefix}${link_prefix}biotac_geom</collision>
+          <collision>${prefix}${link_prefix}biotac_collision</collision>
           <topic>${prefix}${link_prefix}biotac_collision</topic>
         </contact>

File: sr_description/hand/xacro/finger/distal/distal.gazebo.xacro (robot description, xacro)
@@ -8,5 +8,5 @@
         <update_rate>1000.0</update_rate>
         <contact>
-          <collision>${prefix}${link_prefix}distal_geom</collision>
+          <collision>${prefix}${link_prefix}distal_collision</collision>
           <topic>${prefix}${link_prefix}distal_collision</topic>
         </contact>

File: sr_description/hand/xacro/finger/knuckle/knuckle.gazebo.xacro (robot description, xacro)
@@ -8,5 +8,5 @@
         <update_rate>1000.0</update_rate>
         <contact>
-          <collision>${prefix}${link_prefix}knuckle_geom</collision>
+          <collision>${prefix}${link_prefix}knuckle_collision</collision>
           <topic>${prefix}${link_prefix}knuckle_collision</topic>
         </contact>

File: sr_description/hand/xacro/finger/lfmetacarpal/lfmetacarpal.gazebo.xacro (robot description, xacro)
@@ -8,5 +8,5 @@
         <update_rate>1000.0</update_rate>
         <contact>
-          <collision>${prefix}lfmetacarpal_geom</collision>
+          <collision>${prefix}lfmetacarpal_collision</collision>
           <topic>${prefix}lfmetacarpal_collision</topic>
         </contact>

File: sr_description/hand/xacro/finger/middle/middle.gazebo.xacro (robot description, xacro)
@@ -8,5 +8,5 @@
         <update_rate>1000.0</update_rate>
         <contact>
-          <collision>${prefix}${link_prefix}middle_geom</collision>
+          <collision>${prefix}${link_prefix}middle_collision</collision>
           <topic>${prefix}${link_prefix}middle_collision</topic>
         </contact>

File: sr_description/hand/xacro/finger/proximal/proximal.gazebo.xacro (robot description, xacro)
@@ -8,5 +8,5 @@
         <update_rate>1000.0</update_rate>
         <contact>
-          <collision>${prefix}${link_prefix}proximal_geom</collision>
+          <collision>${prefix}${link_prefix}proximal_collision</collision>
           <topic>${prefix}${link_prefix}proximal_collision</topic>
         </contact>

File: sr_description/hand/xacro/palm/palm.gazebo.xacro (robot description, xacro)
@@ -8,5 +8,5 @@
         <update_rate>1000.0</update_rate>
         <contact>
-          <collision>${prefix}palm_geom</collision>
+          <collision>${prefix}palm_collision</collision>
           <topic>${prefix}palm_collision</topic>
         </contact>

File: sr_description/hand/xacro/thumb/thbase.gazebo.xacro (robot description, xacro)
@@ -8,5 +8,5 @@
         <update_rate>1000.0</update_rate>
         <contact>
-          <collision>${prefix}thbase_geom</collision>
+          <collision>${prefix}thbase_collision</collision>
           <topic>${prefix}thbase_collision</topic>
         </contact>

File: sr_description/hand/xacro/thumb/thdistal.gazebo.xacro (robot description, xacro)
@@ -8,5 +8,5 @@
         <update_rate>1000.0</update_rate>
         <contact>
-          <collision>${prefix}thdistal_geom</collision>
+          <collision>${prefix}thdistal_collision</collision>
           <topic>${prefix}thdistal_collision</topic>
         </contact>

File: sr_description/hand/xacro/thumb/thhub.gazebo.xacro (robot description, xacro)
@@ -8,5 +8,5 @@
         <update_rate>1000.0</update_rate>
         <contact>
-          <collision>${prefix}thhub_geom</collision>
+          <collision>${prefix}thhub_collision</collision>
           <topic>${prefix}thhub_collision</topic>
         </contact>

File: sr_description/hand/xacro/thumb/thmiddle.gazebo.xacro (robot description, xacro)
@@ -8,5 +8,5 @@
         <update_rate>1000.0</update_rate>
         <contact>
-          <collision>${prefix}thmiddle_geom</collision>
+          <collision>${prefix}thmiddle_collision</collision>
           <topic>${prefix}thmiddle_collision</topic>
         </contact>

File: sr_description/hand/xacro/thumb/thproximal.gazebo.xacro (robot description, xacro)
@@ -8,5 +8,5 @@
         <update_rate>1000.0</update_rate>
         <contact>
-          <collision>${prefix}thproximal_geom</collision>
+          <collision>${prefix}thproximal_collision</collision>
           <topic>${prefix}thproximal_collision</topic>
         </contact>
