Commit message: Fix the other types of hands.

File: sr_description/hand/xacro/finger/biotac/biotac.urdf.xacro (robot description, xacro)
@@ -11,6 +11,6 @@
       <inertial>
         <origin xyz="0 0 0.0125" rpy="0 0 0" />
-        <mass value="0.012" />
-        <inertia  ixx="0.1" ixy="0.0"  ixz="0.0"  iyy="0.1"  iyz="0.0" izz="0.01" />
+        <mass value="0.016" />
+	    <inertia ixx="0.002" ixy="0.0" ixz="0.0" iyy="0.002" iyz="0.0" izz="0.0002" />
       </inertial>
       <visual>
@@ -49,7 +49,6 @@
       <origin xyz="0 0 0.045" rpy="0 0 0" />
       <axis xyz="1 0 0" />
-      <limit lower="0" upper="${M_PI/2}" effort="1000.0"
-      velocity="10.0" />
-      <dynamics damping="10.0"/>
+      <limit lower="0" upper="${M_PI/2}" effort="30" velocity="1.0"/>
+      <dynamics damping="0.1"/>
     </joint>
     <link name="${link_prefix}_J1_dummy">
@@ -57,5 +56,5 @@
         <origin xyz="0 0 0" rpy="0 0 0" />
         <mass value="0.01" />
-        <inertia  ixx="0.1" ixy="0.0"  ixz="0.0"  iyy="0.1"  iyz="0.0" izz="0.01" />
+        <inertia ixx="0.0007" ixy="0.0" ixz="0.0" iyy="0.0007" iyz="0.0" izz="0.00010" />
       </inertial>
     </link>
@@ -65,6 +64,6 @@
       <origin xyz="0 0 0.02" rpy="0 0 0" />
       <axis xyz="1 0 0" />
-      <limit lower="${20*M_PI/180}" upper="${20.1*M_PI/180}" effort="1000.0" velocity="10.0" />
-      <dynamics damping="10.0"/>
+      <limit lower="${20*M_PI/180}" upper="${20.1*M_PI/180}" effort="10" velocity="1.0"/>
+      <dynamics damping="0.1"/>
     </joint>
     <xacro:middle_transmission />
@@ -72,6 +71,6 @@
       <inertial>
         <origin xyz="0 0 0" rpy="0 0 0" />
-        <mass value="0.10" />
-        <inertia  ixx="0.1" ixy="0.0"  ixz="0.0"  iyy="0.1"  iyz="0.0" izz="0.01" />
+        <mass value="0.01" />
+        <inertia ixx="0.0007" ixy="0.0" ixz="0.0" iyy="0.0007" iyz="0.0" izz="0.00010" />
       </inertial>
       <visual>
@@ -118,5 +117,5 @@
        <mass value="0.001" />
        <origin xyz="0 0 0" rpy="0 0 0" />
-       <inertia  ixx="1" ixy="0"  ixz="0"  iyy="1"  iyz="0" izz="1" />
+       <inertia ixx="0" ixy="0" ixz="0" iyy="0" iyz="0" izz="0" />
       </inertial>
       <visual>

File: sr_description/hand/xacro/finger/biotac/edc_muscle_biotac.urdf.xacro (robot description, xacro)
@@ -11,6 +11,6 @@
       <inertial>
         <origin xyz="0 0 0.0125" rpy="0 0 0" />
-        <mass value="0.012" />
-        <inertia  ixx="0.1" ixy="0.0"  ixz="0.0"  iyy="0.1"  iyz="0.0" izz="0.01" />
+        <mass value="0.016" />
+	    <inertia ixx="0.002" ixy="0.0" ixz="0.0" iyy="0.002" iyz="0.0" izz="0.0002" />
       </inertial>
       <visual>
@@ -49,7 +49,6 @@
       <origin xyz="0 0 0.045" rpy="0 0 0" />
       <axis xyz="1 0 0" />
-      <limit lower="0" upper="${M_PI/2}" effort="1000.0"
-      velocity="10.0" />
-      <dynamics damping="10.0"/>
+      <limit lower="0" upper="${M_PI/2}" effort="30" velocity="1.0"/>
+      <dynamics damping="0.1"/>
     </joint>
     <link name="${link_prefix}_J1_dummy">
@@ -57,5 +56,5 @@
         <origin xyz="0 0 0" rpy="0 0 0" />
         <mass value="0.01" />
-        <inertia  ixx="0.1" ixy="0.0"  ixz="0.0"  iyy="0.1"  iyz="0.0" izz="0.01" />
+        <inertia ixx="0.0007" ixy="0.0" ixz="0.0" iyy="0.0007" iyz="0.0" izz="0.00010" />
       </inertial>
     </link>
@@ -65,6 +64,6 @@
       <origin xyz="0 0 0.02" rpy="0 0 0" />
       <axis xyz="1 0 0" />
-      <limit lower="${20*M_PI/180}" upper="${20.1*M_PI/180}" effort="1000.0" velocity="10.0" />
-      <dynamics damping="10.0"/>
+      <limit lower="${20*M_PI/180}" upper="${20.1*M_PI/180}" effort="10" velocity="1.0"/>
+      <dynamics damping="0.1"/>
     </joint>
     <xacro:middle_transmission />
@@ -72,6 +71,6 @@
       <inertial>
         <origin xyz="0 0 0" rpy="0 0 0" />
-        <mass value="0.10" />
-        <inertia  ixx="0.1" ixy="0.0"  ixz="0.0"  iyy="0.1"  iyz="0.0" izz="0.01" />
+        <mass value="0.01" />
+        <inertia ixx="0.0007" ixy="0.0" ixz="0.0" iyy="0.0007" iyz="0.0" izz="0.00010" />
       </inertial>
       <visual>
@@ -118,5 +117,5 @@
        <mass value="0.001" />
        <origin xyz="0 0 0" rpy="0 0 0" />
-       <inertia  ixx="1" ixy="0"  ixz="0"  iyy="1"  iyz="0" izz="1" />
+       <inertia ixx="0" ixy="0" ixz="0" iyy="0" iyz="0" izz="0" />
       </inertial>
       <visual>

File: sr_description/hand/xacro/finger/knuckle/edc_muscle_knuckle.urdf.xacro (robot description, xacro)
@@ -12,7 +12,6 @@
 	<origin xyz="0 0 0" rpy="0 0 0" />
 	<!--<insert_block name="origin" /> -->
-	<mass value="0.008" />
-	<inertia  ixx="0.0" ixy="0.0"  ixz="0.0"  iyy="0.1"  iyz="0.0"
-	izz="0.0" />
+	<mass value="0.08" />
+	<inertia ixx="0.0026" ixy="0.0" ixz="0.0" iyy="0.0026" iyz="0.0" izz="0.0032" />
       </inertial>
       <visual>
@@ -52,7 +51,7 @@
       <insert_block name="origin" />
       <insert_block name="axis"/>
-      <limit lower="-0.43633231299858238" upper="0.43633231299858238"
-      effort="1000.0" velocity="10.0"/>
-      <dynamics damping="10.0"/>
+      <limit lower="${-20/180*M_PI}" upper="${20/180*M_PI}"
+      effort="2" velocity="1.0"/>
+      <dynamics damping="0.1"/>
     </joint>
     <xacro:knuckle_transmission />

File: sr_description/hand/xacro/finger/knuckle/knuckle.urdf.xacro (robot description, xacro)
@@ -51,5 +51,5 @@
       <insert_block name="origin" />
       <insert_block name="axis"/>
-      <limit lower="-0.3491" upper="0.3491"
+      <limit lower="${-20/180*M_PI}" upper="${20/180*M_PI}"
       effort="2" velocity="1.0"/>
       <dynamics damping="0.1"/>

File: sr_description/hand/xacro/finger/lfmetacarpal/edc_muscle_lfmetacarpal.urdf.xacro (robot description, xacro)
@@ -21,6 +21,6 @@
       <inertial>
         <origin xyz="0 0 0.04" rpy="0 0 0" />
-	    <mass value="0.075" />
-	    <inertia  ixx="0.1" ixy="0.0"  ixz="0.0"  iyy="0.1"  iyz="0.0" izz="0.1" />
+	    <mass value="0.030" />
+	    <inertia ixx="0.00545" ixy="0.0" ixz="0.0" iyy="0.0056352" iyz="0.0" izz="0.0004272" />
       </inertial>
       <visual>
@@ -60,7 +60,7 @@
       <origin xyz="${reflect*-0.033} 0 0.02071" rpy="0 0 0" />
       <axis xyz="0.573576436 0 ${reflect*0.819152044}" />
-      <limit lower="0" upper="0.69813170079773179" effort="1000.0"
-      velocity="10.0" />
-      <dynamics damping="10.0"/>
+      <limit lower="0" upper="${45/180*M_PI}" effort="2"
+      velocity="1.0" />
+      <dynamics damping="0.1"/>
     </joint>
     <xacro:lfmetacarpal_transmission />

File: sr_description/hand/xacro/finger/little_finger_ellipsoid.urdf.xacro (robot description, xacro)
@@ -6,71 +6,21 @@
        xmlns:body="http://playerstage.sourceforge.net/gazebo/xmlschema/#body"
        xmlns:geom="http://playerstage.sourceforge.net/gazebo/xmlschema/#geom">
-  <xacro:include filename="$(find sr_description)/hand/xacro/finger/knuckle/knuckle.urdf.xacro" />
-  <xacro:include filename="$(find sr_description)/hand/xacro/finger/proximal/proximal.urdf.xacro" />
-  <xacro:include filename="$(find sr_description)/hand/xacro/finger/middle/middle.urdf.xacro" />
-  <xacro:include filename="$(find sr_description)/hand/xacro/finger/distal/distal_ellipsoid.urdf.xacro" />
   <xacro:include filename="$(find sr_description)/hand/xacro/finger/lfmetacarpal/lfmetacarpal.urdf.xacro" />
-  <xacro:macro name="little_finger_ellipsoid" params="link_prefix joint_prefix parent">
-    <xacro:lfmetacarpal parent="${parent}" >
-    </xacro:lfmetacarpal>
-    <link name="lfknuckle">
-      <inertial>
-	<origin xyz="0 0 0.06579" rpy="0 0 0" />
-	<mass value="0.008" />
-	<inertia  ixx="0.1" ixy="0.0"  ixz="0.0"  iyy="0.1"  iyz="0.0"
-	izz="0.1" />
-      </inertial>
-      <visual>
-	<origin xyz="0 0 0" rpy="0 0 0" />
-	<geometry name="knuckle_visual">
-      <mesh filename="package://sr_description/hand/model/knuckle.dae" scale="0.001 0.001 0.001" />
-      </geometry>
-      <material name="LightGrey" />
-      </visual>
-      <collision>
-	<origin xyz="0 0 0" rpy="0 0 0" />
-	<geometry name="knuckle_collision_geom">
-	  <box size="0.005 0.005 0.005" />
-	</geometry>
-      </collision>
-    </link>
-    <gazebo reference="lfknuckle">
-      <sensor type="contact" name="lfknuckle_contact" >
-        <always_on>1</always_on>
-        <update_rate>1000.0</update_rate>
-        <contact>
-          <collision>lfknuckle_collision</collision>
-          <topic>lfknuckle_collision</topic>
-        </contact>
-        <plugin name="lfknuckle_gazebo_ros_bumper_controller" filename="libgazebo_ros_bumper.so">
-          <updateRate>100.0</updateRate>
-	  <frameName>lfknuckle</frameName>
-	  <bumperTopicName>contacts/lf/knuckle</bumperTopicName>
-        </plugin>
-      </sensor>
-      <material>Gazebo/Grey</material>
-    </gazebo>
-    <joint name="LFJ4" type="revolute">
-      <parent link="lfmetacarpal"/>
-      <child link="lfknuckle"/>
+  <xacro:include filename="$(find sr_description)/hand/xacro/finger/classic_finger_ellipsoid.urdf.xacro" />
+  <!-- Right Handed -->
+  <xacro:macro name="little_finger" params="link_prefix joint_prefix parent">
+    <xacro:lfmetacarpal parent="${parent}" />
+    <xacro:finger_ellipsoid link_prefix="${link_prefix}" joint_prefix="${joint_prefix}" parent="lfmetacarpal">
       <origin xyz="0 0 0.06579" rpy="0 0 0" />
       <axis xyz="0 1 0" />
-      <limit lower="-0.3491" upper="0.3491"
-      effort="1000.0" velocity="10.0"/>
-      <dynamics damping="10.0"/>
-    </joint>
-    <transmission type="sr_mechanism_model/SimpleTransmission" name="lfknuckle_transmission">
-      <actuator name="LFJ4" />
-      <joint name="LFJ4" />
-      <mechanicalReduction>1</mechanicalReduction>
-      <motorTorqueConstant>1</motorTorqueConstant>
-      <pulsesPerRevolution>90000</pulsesPerRevolution>
-    </transmission>
-    <xacro:proximal link_prefix="${link_prefix}" joint_prefix="${joint_prefix}" parent="${link_prefix}knuckle" >
-    </xacro:proximal>
-    <xacro:middle link_prefix="${link_prefix}" joint_prefix="${joint_prefix}" parent="${link_prefix}proximal" >
-    </xacro:middle>
-    <xacro:distal link_prefix="${link_prefix}" joint_prefix="${joint_prefix}" parent="${link_prefix}middle" >
-    </xacro:distal>
+    </xacro:finger_ellipsoid>
+  </xacro:macro>
+  <!-- Left Handed -->
+  <xacro:macro name="little_finger_left" params="link_prefix joint_prefix parent">
+    <xacro:lfmetacarpal_left parent="${parent}" />
+    <xacro:finger_ellipsoid link_prefix="${link_prefix}" joint_prefix="${joint_prefix}" parent="lfmetacarpal">
+      <origin xyz="0 0 0.06579" rpy="0 0 0" />
+      <axis xyz="0 -1 0" />
+    </xacro:finger_ellipsoid>
   </xacro:macro>
 </robot>

File: sr_description/hand/xacro/finger/proximal/edc_muscle_proximal.urdf.xacro (robot description, xacro)
@@ -10,8 +10,7 @@
     <link name="${link_prefix}proximal">
       <inertial>
-	<mass value="0.014" />
-	<origin xyz="0 0 0.0225" />
-	<inertia  ixx="0.1" ixy="0.0"  ixz="0.0"  iyy="0.1"  iyz="0.0"
-	izz="0.0" />
+	    <mass value="0.030" />
+        <origin xyz="0 0 0.0225" />
+        <inertia ixx="0.003" ixy="0.0" ixz="0.0" iyy="0.003" iyz="0.0" izz="0.0003" />
       </inertial>
       <visual>
@@ -51,7 +50,7 @@
       <origin xyz="0 0 0" rpy="0 0 0" />
       <axis xyz="1 0 0" />
-      <limit lower="0" upper="${M_PI/2}" effort="1000.0"
-      velocity="10.0"/>
-      <dynamics damping="10.0"/>
+      <limit lower="0" upper="${M_PI/2}" effort="2"
+      velocity="1.0"/>
+      <dynamics damping="0.1"/>
     </joint>
     <xacro:proximal_transmission />

File: sr_description/hand/xacro/palm/edc_muscle_palm.urdf.xacro (robot description, xacro)
@@ -22,5 +22,5 @@
 	<origin xyz="0 0 0.035" rpy="0 0 0" />
 	<mass value="0.3" />
-	<inertia  ixx="0.5" ixy="0.0"  ixz="0.0"  iyy="0.5"  iyz="0.0"	izz="0.3" />
+	<inertia ixx="0.003581" ixy="0.0" ixz="0.0" iyy="0.005287" iyz="0.0" izz="0.002545" />
       </inertial>
       <visual>
@@ -71,7 +71,7 @@
       <origin xyz="0 0 0.034" rpy="0 0 0" />
       <axis xyz="1 0 0" />
-      <limit lower="-0.78539816339744828" upper="0.6108652381980153"
-      effort="1000.0" velocity="10.0"/>
-      <dynamics damping="30.0"/>
+      <limit lower="${-40/180*M_PI}" upper="${28/180*M_PI}"
+      effort="30" velocity="1.0"/>
+      <dynamics damping="0.1"/>
     </joint>
     <xacro:shadowhand_palm_transmission />

Commit message: Changed inertia and force limits for biotac fingertip

File: sr_description/hand/xacro/finger/biotac/biotac.urdf.xacro (robot description, xacro)
@@ -17,5 +17,6 @@
         <origin xyz="0 0 0.0125" rpy="0 0 0" />
         <mass value="0.012" />
-        <inertia  ixx="0.1" ixy="0.0"  ixz="0.0"  iyy="0.1"  iyz="0.0" izz="0.01" />
+           <inertia  ixx="0.002" ixy="0.0"  ixz="0.0"  iyy="0.002"  iyz="0.0"
+          izz="0.0002" />
       </inertial>
       <visual>
@@ -54,7 +55,7 @@
       <origin xyz="0 0 0.045" rpy="0 0 0" />
       <axis xyz="1 0 0" />
-      <limit lower="0" upper="${M_PI/2}" effort="1000.0"
-      velocity="10.0" />
-      <dynamics damping="10.0"/>
+      <limit lower="0" upper="${M_PI/2}" effort="2.0"
+      velocity="1.0" />
+      <dynamics damping="0.10"/>
     </joint>
     <link name="${prefix}${link_prefix}_J1_dummy">
@@ -62,5 +63,6 @@
         <origin xyz="0 0 0" rpy="0 0 0" />
         <mass value="0.01" />
-        <inertia  ixx="0.1" ixy="0.0"  ixz="0.0"  iyy="0.1"  iyz="0.0" izz="0.01" />
+         <inertia  ixx="0.002" ixy="0.0"  ixz="0.0"  iyy="0.002"  iyz="0.0"
+          izz="0.0002" />
       </inertial>
     </link>
@@ -70,6 +72,6 @@
       <origin xyz="0 0 0.02" rpy="0 0 0" />
       <axis xyz="1 0 0" />
-      <limit lower="${20*M_PI/180}" upper="${20.1*M_PI/180}" effort="1000.0" velocity="10.0" />
-      <dynamics damping="10.0"/>
+      <limit lower="${20*M_PI/180}" upper="${20.1*M_PI/180}" effort="1.0" velocity="1.0" />
+      <dynamics damping="0.1"/>
     </joint>
     <xacro:middle_transmission muscletrans="${muscle}" prefix="${prefix}" joint_prefix="${joint_prefix}" link_prefix="${link_prefix}"/>
@@ -77,6 +79,7 @@
       <inertial>
         <origin xyz="0 0 0" rpy="0 0 0" />
-        <mass value="0.10" />
-        <inertia  ixx="0.1" ixy="0.0"  ixz="0.0"  iyy="0.1"  iyz="0.0" izz="0.01" />
+        <mass value="0.040" />
+        <inertia  ixx="0.001" ixy="0.0"  ixz="0.0"  iyy="0.001"  iyz="0.0"
+        izz="0.00025" />
       </inertial>
       <visual>
@@ -123,5 +126,5 @@
        <mass value="0.001" />
        <origin xyz="0 0 0" rpy="0 0 0" />
-       <inertia  ixx="1" ixy="0"  ixz="0"  iyy="1"  iyz="0" izz="1" />
+       <inertia  ixx="0.0" ixy="0.0"  ixz="0.0"  iyy="0.0"  iyz="0.0" izz="0.0" />
       </inertial>
       <visual>
