Commit message: Inertia now exact values, with inertia tensor at COM (gazebo and ode support the small values now) Removed explicit viscous damping from sr_gazebo_plugin, enabled springDamper in each joint (implicit viscous damping) changed simulation parameters for stability and retuned the controllers, explicitely define friction_deadband for simulated controllers (default is for real hand and is too high)

File: sr_description/hand/xacro/finger/biotac/biotac.urdf.xacro (robot description, xacro)
@@ -16,7 +16,7 @@
       <inertial>
         <origin xyz="0 0 0.0125" rpy="0 0 0" />
-        <mass value="0.012" />
-           <inertia  ixx="0.002" ixy="0.0"  ixz="0.0"  iyy="0.002"  iyz="0.0"
-          izz="0.0002" />
+          <mass value="0.017" />
+        <inertia  ixx="0.0000026" ixy="0.0"  ixz="0.0"  iyy="0.0000027"  iyz="0.0"
+        izz="0.00000087" />
       </inertial>
       <visual>
@@ -28,7 +28,7 @@
       </visual>
       <collision>
-        <origin xyz="0 0 0.0125" rpy="0 0 0" />
+        <origin xyz="0 0 0.005" rpy="0 0 0" />
         <geometry name="${prefix}${link_prefix}adapter_collision_geom">
-          <box size="0.008 0.008 0.03" />
+          <box size="0.001 0.001 0.001" />
         </geometry>
       </collision>
@@ -48,5 +48,5 @@
         </plugin>
       </sensor>
-      <material>Gazebo/Grey</material>
+      <material>Gazebo/FlatBlack</material>
     </gazebo>
     <joint name="${prefix}${joint_prefix}J2" type="revolute">
@@ -56,13 +56,17 @@
       <axis xyz="1 0 0" />
       <limit lower="0" upper="${M_PI/2}" effort="2.0"
-      velocity="1.0" />
-      <dynamics damping="0.001"/>
+      velocity="2.0" />
+      <dynamics damping="0.1"/>
     </joint>
+    <gazebo reference="${prefix}${joint_prefix}J2">
+      <provideFeedback>1</provideFeedback>
+      <implicitSpringDamper>1</implicitSpringDamper>
+    </gazebo>
     <link name="${prefix}${link_prefix}_J1_dummy">
       <inertial>
-        <origin xyz="0 0 0" rpy="0 0 0" />
-        <mass value="0.01" />
-         <inertia  ixx="0.002" ixy="0.0"  ixz="0.0"  iyy="0.002"  iyz="0.0"
-          izz="0.0002" />
+        <origin xyz="0 0 0.012" />
+        <mass value="0.001" />
+             <inertia  ixx="0.00000001" ixy="0.0"  ixz="0.0"  iyy="0.00000001"  iyz="0.0"
+				izz="0.00000001" />
       </inertial>
     </link>
@@ -72,14 +76,18 @@
       <origin xyz="0 0 0.02" rpy="0 0 0" />
       <axis xyz="1 0 0" />
-      <limit lower="${20*M_PI/180}" upper="${20.1*M_PI/180}" effort="1.0" velocity="1.0" />
-      <dynamics damping="0.001"/>
+      <limit lower="${20*M_PI/180}" upper="${20.1*M_PI/180}" effort="0.0" velocity="2.0" />
+      <dynamics damping="0.5"/>
     </joint>
+    <gazebo reference="${prefix}${joint_prefix}J1">
+      <provideFeedback>1</provideFeedback>
+      <implicitSpringDamper>1</implicitSpringDamper>
+    </gazebo>
     <xacro:middle_transmission muscletrans="${muscle}" prefix="${prefix}" joint_prefix="${joint_prefix}" link_prefix="${link_prefix}"/>
     <link name="${prefix}${link_prefix}biotac">
       <inertial>
-        <origin xyz="0 0 0" rpy="0 0 0" />
-        <mass value="0.040" />
-        <inertia  ixx="0.001" ixy="0.0"  ixz="0.0"  iyy="0.001"  iyz="0.0"
-        izz="0.00025" />
+        <origin xyz="0.0 -0.009 0.035" rpy="0 0 0" /> <!-- approximated only FIXME -->
+        <mass value="0.012" />
+        <inertia  ixx="0.00000094" ixy="0.0"  ixz="0.0"  iyy="0.0000011"  iyz="0.0"
+        izz="0.00000053" />
       </inertial>
       <visual>
@@ -89,5 +97,4 @@
           <mesh filename="package://sr_description/hand/model/biotacs/biotac_decimated.dae" scale="0.0254 0.0254 0.0254" />
         </geometry>
-        <material name="BiotacGreen" />
       </visual>
       <collision>
@@ -113,5 +120,4 @@
       </sensor>
       <selfCollide>true</selfCollide>
-      <material>BiotacGreen</material>
     </gazebo>
     <joint name="${prefix}${joint_prefix}_biotac_joint" type="fixed">
@@ -133,9 +139,4 @@
         </geometry>
       </visual>
-      <collision>
-        <geometry>
-          <box size="0.001 0.001 0.001" />
-        </geometry>
-      </collision>
     </link>
     <gazebo reference="${prefix}${link_prefix}tip">

File: sr_description/hand/xacro/thumb/thdistal.urdf.xacro (robot description, xacro)
@@ -19,8 +19,8 @@
 			<link name="${prefix}thbiotac_J1_dummy">
 				<inertial>
-					<origin xyz="0 0 0" rpy="0 0 0" />
-					<mass value="0.01" />
-					 <inertia  ixx="0.0007" ixy="0.0"  ixz="0.0"  iyy="0.0007"  iyz="0.0"
-        izz="0.00010" />
+          <origin xyz="0 0 0" rpy="0 0 0"/>
+          <mass value="0.001" />
+          <inertia  ixx="0.00000001" ixy="0.0"  ixz="0.0"  iyy="0.00000001"  iyz="0.0"
+				izz="0.00000001" />
         </inertial>
 			</link>
@@ -28,15 +28,19 @@
 				<parent link="${parent}"/>
 				<child link="${prefix}thbiotac_J1_dummy"/>
-				<origin xyz="0 0 0.02" rpy="0 0 0" />
+				<origin xyz="0 0 0.02" rpy="0 0 ${-M_PI/2}" />
 				<axis xyz="1 0 0" />
-				<limit lower="${20*M_PI/180}" upper="${20.1*M_PI/180}" effort="10" velocity="0.1" />
-				<dynamics damping="0.001"/>
+				<limit lower="${20*M_PI/180}" upper="${20.1*M_PI/180}" effort="0.0" velocity="2.0" />
+				<dynamics damping="0.5"/>
 			</joint>
+			<gazebo reference="${prefix}THJ1">
+				<provideFeedback>1</provideFeedback>
+				<implicitSpringDamper>1</implicitSpringDamper>
+			</gazebo>
 			<link name="${prefix}thbiotac">
 				<inertial>
-					<origin xyz="0 0 0" rpy="0 0 0" />
-					<mass value="0.2" />
-					 <inertia  ixx="0.0007" ixy="0.0"  ixz="0.0"  iyy="0.0007"  iyz="0.0"
-        izz="0.00010" />
+          <origin xyz="-0.009 0.0 0.035" rpy="0 0 ${-M_PI/2}" /> <!-- approximated only FIXME -->
+					<mass value="0.008" />
+					 <inertia  ixx="0.0000011" ixy="0.0"  ixz="0.0"  iyy="0.0000011"  iyz="0.0"
+        izz="0.0000005" />
 				</inertial>
 				<visual>
@@ -77,5 +81,5 @@
 				<parent link="${prefix}thmiddle"/>
 				<child link="${prefix}thbiotac"/>
-				<origin xyz="0 0.0 0.01" rpy="0 0 -1.571" />
+				<origin xyz="0 0.0 0.01" rpy="0 0 ${-M_PI/2}" />
 			</joint>
 		  <!-- extra link to imaginary sphere in fingertip for FK/IK calculations -->
@@ -92,9 +96,4 @@
 					</geometry>
 				</visual>
-				<collision>
-					<geometry>
-						<box size="0.001 0.001 0.001" />
-					</geometry>
-				</collision>
 			</link>
 			<gazebo reference="${prefix}thtip">
@@ -113,6 +112,6 @@
 					<mass value="0.016" />
 					<origin xyz="0 0 0.01375" rpy="0 0 0"/>
-					 <inertia  ixx="0.0007" ixy="0.0"  ixz="0.0"  iyy="0.0007"  iyz="0.0"
-        izz="0.00010" />
+					 <inertia  ixx="0.0000021" ixy="0.0"  ixz="0.0"  iyy="0.0000022"  iyz="0.0"
+        izz="0.000001" />
 				</inertial>
 				<visual>
@@ -164,7 +163,11 @@
 				<origin xyz="0 0 0.032" rpy="0 0 ${-M_PI/2}" />
 				<axis xyz="1 0 0" />
-				<limit lower="0" upper="${90.0*M_PI/180}" effort="10" velocity="1.0" />
-				<dynamics damping="0.001"/>
+				<limit lower="0" upper="${90.0*M_PI/180}" effort="1.0" velocity="4.0" />
+				<dynamics damping="0.2"/>
 			</joint>
+			<gazebo reference="${prefix}THJ1">
+				<provideFeedback>1</provideFeedback>
+				<implicitSpringDamper>1</implicitSpringDamper>
+			</gazebo>
 			<link name="${prefix}thtip">
 				<inertial>

File: sr_description/hand/xacro/thumb/thhub.urdf.xacro (robot description, xacro)
@@ -16,8 +16,8 @@
     <link name="${prefix}thhub">
       <inertial>
-				<mass value="0.01" />
+				<mass value="0.005" />
 				<origin xyz="0 0 0" rpy="0 0 0"/>
-				<inertia  ixx="0.0003" ixy="0.0"  ixz="0.0"  iyy="0.0003"  iyz="0.0"
-				izz="0.0003" />
+				<inertia  ixx="0.0000001" ixy="0.0"  ixz="0.0"  iyy="0.0000001"  iyz="0.0"
+				izz="0.0000001" />
       </inertial>
       <visual>
@@ -51,8 +51,12 @@
         <origin xyz="0 0 0.038" rpy="0 0 0" />
         <axis xyz="1 0 0" />
-        <limit lower="${-12/180*M_PI}" upper="${12/180*M_PI}" effort="10"
-        velocity="1.0" />
-        <dynamics damping="0.02"/>
+        <limit lower="${-12/180*M_PI}" upper="${12/180*M_PI}" effort="2.0"
+        velocity="4.0" />
+        <dynamics damping="0.2"/>
       </joint>
+      <gazebo reference="${prefix}THJ3">
+        <provideFeedback>1</provideFeedback>
+        <implicitSpringDamper>1</implicitSpringDamper>
+      </gazebo>
     </xacro:unless>
 		<!-- extensions -->

File: sr_description/hand/xacro/thumb/thmiddle.urdf.xacro (robot description, xacro)
@@ -15,7 +15,7 @@
     <link name="${prefix}thmiddle">
       <inertial>
-        <mass value="0.027" />
+        <mass value="0.020" />
         <origin xyz="0 0 0.016" rpy="0 0 0"/>
-          <inertia  ixx="0.0026" ixy="0.0"  ixz="0.0"  iyy="0.0026"  iyz="0.0" izz="0.000169" />
+          <inertia  ixx="0.0000051" ixy="0.0"  ixz="0.0"  iyy="0.0000051"  iyz="0.0" izz="0.00000121" />
       </inertial>
       <visual>
@@ -25,5 +25,4 @@
           <mesh filename="package://sr_description/hand/model/biotacs/biotac_thumb_adapter.dae" scale="0.001 0.001 0.001" />
         </geometry>
-        <material name="BiotacGreen" />
         </xacro:if>
         <xacro:unless value="${bio}">
@@ -37,13 +36,16 @@
       </visual>
       <collision>
-        <origin xyz="0 0 0.012" rpy="0 0 0 " />
-        <geometry name="${prefix}thmiddle_collision_geom">
-          <xacro:if value="${bio}">
-            <box size="0.008 0.008 0.01" />
-          </xacro:if>
-          <xacro:unless value="${bio}">
+        <xacro:if value="${bio}">
+          <origin xyz="0 0 0.005" rpy="0 0 0 " />
+          <geometry name="${prefix}thmiddle_collision_geom">
+            <box size="0.001 0.001 0.001" />
+          </geometry>
+        </xacro:if>
+        <xacro:unless value="${bio}">
+          <origin xyz="0 0 0.012" rpy="0 0 0 " />
+          <geometry name="${prefix}thmiddle_collision_geom">
             <cylinder radius="0.011" length="0.018" />
-          </xacro:unless>
-        </geometry>
+          </geometry>
+        </xacro:unless>
       </collision>
       <xacro:unless value="${bio}">
@@ -66,8 +68,12 @@
 				</xacro:unless>
       <axis xyz="0 -1 0" />
-      <limit lower="${-40/180*M_PI}" upper="${40/180*M_PI}" effort="10"
-      velocity="1.0" />
-      <dynamics damping="0.001"/>
+      <limit lower="${-40/180*M_PI}" upper="${40/180*M_PI}" effort="2.0"
+      velocity="2.0" />
+      <dynamics damping="0.1"/>
     </joint>
+    <gazebo reference="${prefix}THJ2">
+      <provideFeedback>1</provideFeedback>
+      <implicitSpringDamper>1</implicitSpringDamper>
+    </gazebo>
 		<!-- extensions -->
 		<xacro:thmiddle_transmission muscletrans="${muscle}" prefix="${prefix}"/>

Commit message: changing biotacs to have the same link names

File: sr_description/hand/xacro/finger/biotac/biotac.urdf.xacro (robot description, xacro)
@@ -14,5 +14,5 @@
   <xacro:macro name="biotac_middle"
   params="muscle prefix link_prefix joint_prefix parent">
-    <link name="${prefix}${link_prefix}adapter">
+    <link name="${prefix}${link_prefix}middle">
       <inertial>
         <origin xyz="0 0 0.0125" rpy="0 0 0" />
@@ -23,5 +23,5 @@
       <visual>
         <origin xyz="0 0 0" rpy="0 0 1.571" />
-        <geometry name="${prefix}${link_prefix}adapter_visual">
+        <geometry name="${prefix}${link_prefix}middle_visual">
           <mesh filename="package://sr_description/hand/model/biotacs/biotac_finger_adapter.dae"
           scale="1 1 1" />
@@ -31,25 +31,25 @@
       <collision>
         <origin xyz="0 0 0.005" rpy="0 0 0" />
-        <geometry name="${prefix}${link_prefix}adapter_collision_geom">
+        <geometry name="${prefix}${link_prefix}middle_collision_geom">
           <box size="0.001 0.001 0.001" />
         </geometry>
       </collision>
     </link>
-    <gazebo reference="${prefix}${link_prefix}adapter">
+    <gazebo reference="${prefix}${link_prefix}middle">
       <sensor type="contact"
-      name="${prefix}${link_prefix}adapter_contact">
+      name="${prefix}${link_prefix}middle_contact">
         <always_on>1</always_on>
         <update_rate>1000.0</update_rate>
         <contact>
           <collision>
-          ${prefix}${link_prefix}adapter_collision</collision>
-          <topic>${prefix}${link_prefix}adapter_collision</topic>
+          ${prefix}${link_prefix}middle_collision</collision>
+          <topic>${prefix}${link_prefix}middle_collision</topic>
         </contact>
-        <plugin name="${prefix}${link_prefix}adapter_gazebo_ros_bumper_controller"
+        <plugin name="${prefix}${link_prefix}middle_gazebo_ros_bumper_controller"
         filename="libgazebo_ros_bumper.so">
           <updateRate>100.0</updateRate>
-          <frameName>${prefix}${link_prefix}adapter</frameName>
+          <frameName>${prefix}${link_prefix}middle</frameName>
           <bumperTopicName>
-          contacts/${prefix}${link_prefix}/adapter</bumperTopicName>
+          contacts/${prefix}${link_prefix}/middle</bumperTopicName>
         </plugin>
       </sensor>
@@ -58,5 +58,5 @@
     <joint name="${prefix}${joint_prefix}J2" type="revolute">
       <parent link="${parent}" />
-      <child link="${prefix}${link_prefix}adapter" />
+      <child link="${prefix}${link_prefix}middle" />
       <origin xyz="0 0 0.045" rpy="0 0 0" />
       <axis xyz="1 0 0" />
@@ -78,5 +78,5 @@
     </link>
     <joint name="${prefix}${joint_prefix}J1" type="revolute">
-      <parent link="${prefix}${link_prefix}adapter" />
+      <parent link="${prefix}${link_prefix}middle" />
       <child link="${prefix}${link_prefix}_J1_dummy" />
       <origin xyz="0 0 0.02" rpy="0 0 0" />
@@ -93,5 +93,5 @@
     prefix="${prefix}" joint_prefix="${joint_prefix}"
     link_prefix="${link_prefix}" />
-    <link name="${prefix}${link_prefix}biotac">
+    <link name="${prefix}${link_prefix}distal">
       <inertial>
         <origin xyz="0.0 -0.009 0.035" rpy="0 0 0" />
@@ -103,5 +103,5 @@
       <visual>
         <origin xyz="0 0 0" rpy="0 0 0" />
-        <geometry name="${prefix}${link_prefix}biotac_visual">
+        <geometry name="${prefix}${link_prefix}distal_visual">
           <!-- <mesh filename="package://sr_description/hand/model/biotacs/biotac.stl" scale="0.0254 0.0254 0.0254" /> -->
           <mesh filename="package://sr_description/hand/model/biotacs/biotac_decimated.dae"
@@ -110,5 +110,5 @@
       </visual>
       <collision>
-        <geometry name="${prefix}${link_prefix}biotac_collision_geom">
+        <geometry name="${prefix}${link_prefix}distal_collision_geom">
           <!-- <mesh filename="package://sr_description/hand/model/biotacs/biotac.stl" scale="0.0254 0.0254 0.0254" /> -->
           <mesh filename="package://sr_description/hand/model/biotacs/biotac_decimated.dae"
@@ -117,28 +117,28 @@
       </collision>
     </link>
-    <gazebo reference="${prefix}${link_prefix}biotac">
+    <gazebo reference="${prefix}${link_prefix}distal">
       <sensor type="contact"
-      name="${prefix}${link_prefix}biotac_contact">
+      name="${prefix}${link_prefix}distal_contact">
         <always_on>1</always_on>
         <update_rate>1000.0</update_rate>
         <contact>
           <collision>
-          ${prefix}${link_prefix}biotac_collision</collision>
-          <topic>${prefix}${link_prefix}biotac_collision</topic>
+          ${prefix}${link_prefix}distal_collision</collision>
+          <topic>${prefix}${link_prefix}distal_collision</topic>
         </contact>
-        <plugin name="${prefix}${link_prefix}biotac_gazebo_ros_bumper_controller"
+        <plugin name="${prefix}${link_prefix}distal_gazebo_ros_bumper_controller"
         filename="libgazebo_ros_bumper.so">
           <updateRate>100.0</updateRate>
-          <frameName>${prefix}${link_prefix}biotac</frameName>
+          <frameName>${prefix}${link_prefix}distal</frameName>
           <bumperTopicName>
-          contacts/${prefix}${link_prefix}/biotac</bumperTopicName>
+          contacts/${prefix}${link_prefix}/distal</bumperTopicName>
         </plugin>
       </sensor>
       <selfCollide>true</selfCollide>
     </gazebo>
-    <joint name="${prefix}${joint_prefix}_biotac_joint"
+    <joint name="${prefix}${joint_prefix}_distal_joint"
     type="fixed">
-      <parent link="${prefix}${link_prefix}adapter" />
-      <child link="${prefix}${link_prefix}biotac" />
+      <parent link="${prefix}${link_prefix}middle" />
+      <child link="${prefix}${link_prefix}distal" />
       <origin xyz="0 0.0 0.008" rpy="0 0 0" />
     </joint>
@@ -163,5 +163,5 @@
     <joint name="${prefix}${link_prefix}tip_fixed_joint"
     type="fixed">
-      <parent link="${prefix}${link_prefix}adapter" />
+      <parent link="${prefix}${link_prefix}middle" />
       <child link="${prefix}${link_prefix}tip" />
       <origin xyz="0.0 -0.009 ${0.008+0.044}" rpy="0 0 -1.571" />

File: sr_description/hand/xacro/thumb/thdistal.urdf.xacro (robot description, xacro)
@@ -19,5 +19,5 @@
     <xacro:if value="${bio}">
       <!--    BIOTAC -->
-      <link name="${prefix}thbiotac_J1_dummy">
+      <link name="${prefix}thdistal_J1_dummy">
         <inertial>
           <origin xyz="0 0 0" rpy="0 0 0" />
@@ -29,5 +29,5 @@
       <joint name="${prefix}THJ1" type="revolute">
         <parent link="${parent}" />
-        <child link="${prefix}thbiotac_J1_dummy" />
+        <child link="${prefix}thdistal_J1_dummy" />
         <origin xyz="0 0 0.02" rpy="0 0 ${-M_PI/2}" />
         <axis xyz="1 0 0" />
@@ -40,5 +40,5 @@
         <implicitSpringDamper>1</implicitSpringDamper>
       </gazebo>
-      <link name="${prefix}thbiotac">
+      <link name="${prefix}thdistal">
         <inertial>
           <origin xyz="-0.009 0.0 0.035" rpy="0 0 ${-M_PI/2}" />
@@ -50,5 +50,5 @@
         <visual>
           <origin xyz="0 0 0" rpy="0 0 0" />
-          <geometry name="${prefix}th_biotac_visual">
+          <geometry name="${prefix}th_distal_visual">
             <!-- <mesh filename="package://sr_description/hand/model/biotacs/biotac.stl" scale="0.0254 0.0254 0.0254" /> -->
             <mesh filename="package://sr_description/hand/model/biotacs/biotac_decimated.dae"
@@ -58,5 +58,5 @@
         </visual>
         <collision>
-          <geometry name="${prefix}th_biotac_collision_geom">
+          <geometry name="${prefix}th_distal_collision_geom">
             <!-- <box size="0.001 0.001 0.001" /> -->
             <!-- <mesh filename="package://sr_description/hand/model/biotacs/biotac-v5.stl" scale="0.0254 0.0254 0.0254" /> -->
@@ -71,11 +71,11 @@
           <update_rate>1000.0</update_rate>
           <contact>
-            <collision>${prefix}thbiotac_geom</collision>
-            <topic>${prefix}thbiotac_collision</topic>
+            <collision>${prefix}thdistal_geom</collision>
+            <topic>${prefix}thdistal_collision</topic>
           </contact>
-          <plugin name="${prefix}thbiotac_gazebo_ros_bumper_controller"
+          <plugin name="${prefix}thdistal_gazebo_ros_bumper_controller"
           filename="libgazebo_ros_bumper.so">
             <alwaysOn>true</alwaysOn>
-            <frameName>${prefix}thbiotac</frameName>
+            <frameName>${prefix}thdistal</frameName>
             <updateRate>100.0</updateRate>
             <bumperTopicName>
@@ -86,7 +86,7 @@
         <material>BiotacGreen</material>
       </gazebo>
-      <joint name="${prefix}th_biotac_joint" type="fixed">
+      <joint name="${prefix}th_distal_joint" type="fixed">
         <parent link="${prefix}thmiddle" />
-        <child link="${prefix}thbiotac" />
+        <child link="${prefix}thdistal" />
         <origin xyz="0 0.0 0.01" rpy="0 0 ${-M_PI/2}" />
       </joint>

Commit message: unifing names and config between biotac / non biotac hands

File: sr_description/hand/xacro/finger/biotac/biotac.urdf.xacro (robot description, xacro)
@@ -158,8 +158,8 @@
       </visual>
     </link>
-    <gazebo reference="${prefix}${link_prefix}tip">
+    <gazebo reference="${prefix}${joint_prefix}tip">
       <material name="Gazebo/RedGlow" />
     </gazebo>
-    <joint name="${prefix}${link_prefix}tip_fixed_joint"
+    <joint name="${prefix}${joint_prefix}tip"
     type="fixed">
       <parent link="${prefix}${link_prefix}middle" />
