Commit message: Added code to detect joints of the hand.

File: sr_description/hand/xacro/finger/middle/middle.transmission.xacro (robot description, xacro)
@@ -28,4 +28,5 @@
           <hardwareInterface>EffortJointInterface</hardwareInterface>
         </joint>
+        <!--<joint name="${prefix}${joint_prefix}J2" />-->
       </transmission>
     </xacro:unless>

Commit message: Added information about second joint for J0 transmission

File: sr_description/hand/xacro/finger/middle/middle.transmission.xacro (robot description, xacro)
@@ -28,5 +28,5 @@
           <hardwareInterface>EffortJointInterface</hardwareInterface>
         </joint>
-        <!--<joint name="${prefix}${joint_prefix}J2" />-->
+        <secondJoint name="${prefix}${joint_prefix}J2" />
       </transmission>
     </xacro:unless>
